File: S-CPU_kicad/muldiv.kicad_sch (KiCad schematic)
At the start: 0 parts

Commit message: Latch cell identified. Progress in Mul Div section.
Parts:
- added ABVA1 (x2), ABWF1 (x2), ABXH1 (x2), ACBV1 (x2), ACGM1 (x2), ACHJ1 (x2), ACJG1 (x2), ACKH1 (x2): TRI_BUF_IF0, symbol Ricoh_Cells:TRI_BUF_IF0
- added CABL1, CABL2, CABL3, CABL4, CABL5, CABL6, CABL7, CABL8, CABL9: AOI_22, symbol Ricoh_Cells:AOI_22
- added FGKE, HGUU, HHEB, HHFN, HHFN1, HHFN2, HHFN3, HHFN4: INVERTER_A, symbol Ricoh_Cells:INVERTER_A
- added GBEG: OR_3, symbol Ricoh_Cells:OR_3
- added HFJQ, HFPC, HFSC, HFYF, HGDM, HGFS, HGHK, HGRD, HGRD1, HGRQ, HHDH, HHDH1, HHKS, JGON, JGRZ, JGYM, JGYV, JHDZ, JHHT, JHSJ, JHSZ, KFCL: AND_2, symbol Ricoh_Cells:AND_2
- added HGJS, HGJS1: OR_2, symbol Ricoh_Cells:OR_2
- added HHOM, HHXX, HIBF, HIPM: NAND_2, symbol Ricoh_Cells:NAND_2
- added HIBX: NAND_4, symbol Ricoh_Cells:NAND_4
- added HIEP: AND_4, symbol Ricoh_Cells:AND_4
- added IFCU, IFEQ, IFMG, IFMP, IFQQ, IFUF, IFWE, IFXO, IGFF, IGHG, IGKE, IGLE, IGOJ, IGOK, IGST, IGUE, JFCT, JFDF, JFHM, JFKA, JFLO, JFQD, JFRL, JFRP, KFCQ, KFMZ, KFOX, KFYB, KFZV, KGGW, KGHB, KGZD, KHAD, KHRF, KHSS, KHXL, KHYE, KICH, KIDU: AOI_222, symbol Ricoh_Cells:AOI_222
- added JGMY, JGMY1, JGSQ, JGSQ1, JGSQ10, JGSQ11, JGSQ12, JGSQ13, JGSQ2, JGSQ3, JGSQ4, JGSQ5, JGSQ6, JGSQ7, JGSQ8, JGSQ9: D_LATCH_A2, symbol Ricoh_Cells:D_LATCH_A2
- added KBGM (x57): DFFR_B, symbol Ricoh_Cells:DFFR_B
- added KBGM: DFFR_A, symbol Ricoh_Cells:DFFR_A
- added OACG (x22): DELAY_BUF, symbol Ricoh_Cells:DELAY_BUF
- added QABF (x16): XNOR, symbol Ricoh_Cells:XNOR
- added TBUI (x2): NOR_2, symbol Ricoh_Cells:NOR_2
Connections:
- net ~{4203_WR}: now also HGRD.2, HHKS.2
- net ~{4206_WR}: now also HGJS1.2, HGRD1.1, HHKS.1
- net ~{4214_RD}: now also ABVA1.2 (~{ENA}), ABWF1.2 (~{ENA}), ABXH1.2 (~{ENA}), ACBV1.2 (~{ENA}), ACGM1.2 (~{ENA}), ACHJ1.2 (~{ENA}), ACJG1.2 (~{ENA}), ACKH1.2 (~{ENA})
- net ~{4215_RD}: now also ABVA1.2 (~{ENA}), ABWF1.2 (~{ENA}), ABXH1.2 (~{ENA}), ACBV1.2 (~{ENA}), ACGM1.2 (~{ENA}), ACHJ1.2 (~{ENA}), ACJG1.2 (~{ENA}), ACKH1.2 (~{ENA})
- new net: KBGM.1 (~{RESET}), KBGM.5 (~{RESET}) (x39)
- new net: KBGM.2 (D), KFOX.3
- new net: KBGM.3 (CLK), KBGM.3 (CLK), KBGM.3 (CLK), KBGM.3 (CLK), KBGM.3 (CLK), KBGM.3 (CLK), KBGM.3 (CLK), KBGM.3 (CLK), KBGM.3 (CLK), KBGM.3 (CLK), KBGM.3 (CLK), KBGM.3 (CLK), KBGM.3 (CLK), KBGM.3 (CLK), KBGM.3 (CLK), KBGM.4 (~{CLK}), KBGM.4 (~{CLK}), KBGM.4 (~{CLK}), KBGM.4 (~{CLK}), KBGM.4 (~{CLK}), KBGM.4 (~{CLK}), KBGM.4 (~{CLK}), KBGM.4 (~{CLK}), KBGM.4 (~{CLK}), KBGM.4 (~{CLK}), KBGM.4 (~{CLK}), KBGM.4 (~{CLK}), KBGM.4 (~{CLK}), KBGM.4 (~{CLK}), KBGM.4 (~{CLK}), OACG.2, OACG.2
- new net: KBGM.7 (Q), KFMZ.2, KFYB.1, QABF.3 (2)
- new net: KBGM.7 (Q), KHAD.2, KHSS.1, QABF.3 (2)
- new net: KBGM.7 (Q), KHSS.2, KHYE.1, QABF.3 (2)
- new net: KGZD.3, KHAD.3, KHRF.3, KHSS.3, KHXL.3, KHYE.3, KICH.3, KIDU.3, OACG.2
- new net: KBGM.2 (D), KHSS.3
- new net: KGZD.4, KHAD.4, KHRF.4, KHSS.4, KHXL.4, KHYE.4, KICH.4, KIDU.4, OACG.2
- new net: JGYV.3, KHSS.5
- new net: KGZD.6, KHAD.6, KHRF.6, KHSS.6, KHXL.6, KHYE.6, KICH.6, KIDU.6, OACG.2
- new net: KBGM.1 (~{RESET}), KBGM.1 (~{RESET}), KBGM.1 (~{RESET}), KBGM.1 (~{RESET}), KBGM.5 (~{RESET}), KBGM.5 (~{RESET}), KBGM.5 (~{RESET}), KBGM.5 (~{RESET}), KBGM.6 (~{Q})
- new net: KBGM.2 (D), KBGM.3 (CLK), KBGM.4 (~{CLK}), KBGM.6 (~{Q}) (x3)
- new net: HIBX.4, HIEP.3, KBGM.7 (Q)
- new net: IFEQ.3, KBGM.2 (D)
- new net: KBGM.3 (CLK), KBGM.3 (CLK), KBGM.3 (CLK), KBGM.3 (CLK), KBGM.3 (CLK), KBGM.3 (CLK), KBGM.3 (CLK), KBGM.3 (CLK), KBGM.4 (~{CLK}), KBGM.4 (~{CLK}), KBGM.4 (~{CLK}), KBGM.4 (~{CLK}), KBGM.4 (~{CLK}), KBGM.4 (~{CLK}), KBGM.4 (~{CLK}), KBGM.4 (~{CLK}), OACG.2 (x3)
- new net: ACJG1.1 (IN), ACJG1.3 (IN), IFCU.2, IFMG.1, KBGM.7 (Q)
- new net: IGFF.5, JGMY.4 (Q)
- new net: JGON.3, KGZD.5
- new net: HHFN.2, OACG.1, OACG.1, OACG.1, TBUI.2
- new net: QABF.2 (1), QABF.2 (1), QABF.2 (1), QABF.2 (1), QABF.2 (1), QABF.2 (1), QABF.2 (1), QABF.2 (1), QABF.2 (1), QABF.2 (1), QABF.2 (1), QABF.2 (1), QABF.2 (1), QABF.2 (1), QABF.2 (1), QABF.2 (1)
- new net: KBGM.7 (Q), KFZV.2, KGHB.1, QABF.3 (2)
- new net: CABL4.3, JGSQ8.4 (Q)
- new net: OACG.1, OACG.1, OACG.1, TBUI.3
- new net: JFCT.3, JFDF.3, JFHM.3, JFKA.3, JFLO.3, JFQD.3, JFRL.3, JFRP.3, KFCQ.3, KFMZ.3, KFOX.3, KFYB.3, KFZV.3, KGGW.3, KGHB.3, OACG.2, OACG.2
- new net: KBGM.7 (Q), KGGW.2, KGZD.1, QABF.3 (2)
- new net: KBGM.7 (Q), KGZD.2, KHRF.1, QABF.3 (2)
- new net: KBGM.2 (D), KGZD.3
- new net: ACKH1.1 (IN), ACKH1.3 (IN), IFEQ.1, KBGM.7 (Q)
- new net: KBGM.2 (D), KGHB.3
- new net: IFMG.3, KBGM.2 (D)
- new net: ACHJ1.1 (IN), ACHJ1.3 (IN), IFEQ.2, IFMP.1, KBGM.7 (Q)
- new net: IFCU.3, IFEQ.3, IFMG.3, IFMP.3, IFQQ.3, IFUF.3, IFWE.3, IFXO.3, OACG.2
- new net: IFCU.4, IFEQ.4, IFMG.4, IFMP.4, IFQQ.4, IFUF.4, IFWE.4, IFXO.4, OACG.2
- new net: IFCU.6, IFEQ.6, IFMG.6, IFMP.6, IFQQ.6, IFUF.6, IFWE.6, IFXO.6, OACG.2
- new net: KBGM.1 (~{RESET}), KBGM.1 (~{RESET}), KBGM.1 (~{RESET}), KBGM.1 (~{RESET}), KBGM.1 (~{RESET}), KBGM.1 (~{RESET}), KBGM.1 (~{RESET}), KBGM.1 (~{RESET}), KBGM.5 (~{RESET}), KBGM.5 (~{RESET}), KBGM.5 (~{RESET}), KBGM.5 (~{RESET}), KBGM.5 (~{RESET}), KBGM.5 (~{RESET}), KBGM.5 (~{RESET}), KBGM.5 (~{RESET})
- new net: CABL6.3, KBGM.2 (D)
- new net: KBGM.3 (CLK), KBGM.3 (CLK), KBGM.3 (CLK), KBGM.3 (CLK), KBGM.3 (CLK), KBGM.3 (CLK), KBGM.3 (CLK), KBGM.3 (CLK), KBGM.4 (~{CLK}), KBGM.4 (~{CLK}), KBGM.4 (~{CLK}), KBGM.4 (~{CLK}), KBGM.4 (~{CLK}), KBGM.4 (~{CLK}), KBGM.4 (~{CLK}), KBGM.4 (~{CLK})
- new net: CABL9.3, JGSQ13.4 (Q)
- new net: KBGM.7 (Q), KFYB.2, KGGW.1, QABF.3 (2)
- new net: KBGM.2 (D), KFCQ.3
- new net: JFCT.2, KBGM.7 (Q), KFMZ.1, QABF.3 (2)
- new net: HIBF.2, HIEP.5
- new net: HHXX.2, HIBF.3
- new net: JFDF.3, KBGM.2 (D)
- new net: JFCT.1, JFHM.2, KBGM.7 (Q)
- new net: CABL3.3, JGSQ7.4 (Q)
- new net: CABL8.3, JGSQ12.4 (Q)
- new net: ACBV1.1 (IN), ACBV1.3 (IN), IFMP.2, IFUF.1, KBGM.7 (Q)
- new net: IFMP.3, KBGM.2 (D)
- new net: HHDH1.3, OACG.1, OACG.1
- new net: OACG.2, OACG.2
- new net: ABXH1.1 (IN), ABXH1.3 (IN), IFQQ.2, IFWE.1, KBGM.7 (Q)
- new net: ABVA1.1 (IN), ABVA1.3 (IN), IFWE.2, IGFF.1, KBGM.7 (Q)
- new net: IFWE.3, KBGM.2 (D)
- new net: CABL2.3, KBGM.2 (D)
- new net: IGHG.5, JGSQ.4 (Q)
- new net: IGHG.3, KBGM.2 (D)
- new net: ACJG1.1 (IN), ACJG1.3 (IN), IGFF.2, IGKE.1, KBGM.7 (Q)
- new net: ACGM1.1 (IN), ACGM1.3 (IN), IFMG.2, IFQQ.1, KBGM.7 (Q)
- new net: HHDH.3, OACG.1, OACG.1, OACG.1, TBUI.1
- new net: KBGM.7 (Q), KHRF.2, KHXL.1, QABF.3 (2)
- new net: KBGM.2 (D), KHRF.3
- new net: JGYM.3, KHRF.5
- new net: JFCT.5, KFCL.3
- new net: JFDF.2, KBGM.7 (Q), KFCQ.1, QABF.3 (2)
- new net: JFCT.6, JFDF.6, JFHM.6, JFKA.6, JFLO.6, JFQD.6, JFRL.6, JFRP.6, KFCQ.6, KFMZ.6, KFOX.6, KFYB.6, KFZV.6, KGGW.6, KGHB.6, OACG.2, OACG.2
- new net: ABWF1.1 (IN), ABWF1.3 (IN), IFUF.2, IFXO.1, KBGM.7 (Q)
- new net: IFUF.3, KBGM.2 (D)
- new net: ACGM1.1 (IN), ACGM1.3 (IN), IFXO.2, IGHG.1, KBGM.7 (Q)
- new net: KBGM.7 (Q), KHXL.2, KICH.1, QABF.3 (2)
- new net: JFRP.3, KBGM.2 (D)
- new net: JFRL.1, KBGM.7 (Q)
- new net: KBGM.7 (Q), KFCQ.2, KFOX.1, QABF.3 (2)
- new net: KBGM.7 (Q), KFOX.2, KFZV.1, QABF.3 (2)
- new net: JFCT.4, JFDF.4, JFHM.4, JFKA.4, JFLO.4, JFQD.4, JFRL.4, JFRP.4, KFCQ.4, KFMZ.4, KFOX.4, KFYB.4, KFZV.4, KGGW.4, KGHB.4, OACG.2, OACG.2
- new net: HGRD1.3, OACG.1, OACG.1, OACG.1
- new net: HHFN3.2, KBGM.2 (D)
- new net: HHFN2.2, KBGM.3 (CLK), KBGM.4 (~{CLK})
- new net: ABVA1.1 (IN), ABVA1.3 (IN), CABL1.3, IGST.2, KBGM.7 (Q)
- new net: CABL1.3, HHFN3.1
- new net: CABL1.4, HHFN4.2
- new net: KBGM.2 (D), KGGW.3
- new net: HGRQ.3, OACG.1, OACG.1, TBUI.2
- new net: IGOJ.5, JGSQ3.4 (Q)
- new net: JFQD.1, JFRP.2, KBGM.7 (Q)
- new net: KBGM.7 (Q), KICH.2, QABF.3 (2)
- new net: KBGM.2 (D), KICH.3
- new net: JHSJ.3, KICH.5
- new net: ACKH1.1 (IN), ACKH1.3 (IN), IGOJ.2, IGST.1, KBGM.7 (Q)
- new net: IGFF.3, IGHG.3, IGKE.3, IGLE.3, IGOJ.3, IGOK.3, IGST.3, IGUE.3, OACG.2
- new net: IGST.3, KBGM.2 (D)
- new net: IGFF.4, IGHG.4, IGKE.4, IGLE.4, IGOJ.4, IGOK.4, IGST.4, IGUE.4, OACG.2
- new net: IGST.5, JGSQ5.4 (Q)
- new net: IGFF.6, IGHG.6, IGKE.6, IGLE.6, IGOJ.6, IGOK.6, IGST.6, IGUE.6, OACG.2
- new net: JFCT.3, KBGM.2 (D)
- new net: CABL7.3, JGSQ11.4 (Q)
- new net: HGDM.1, HGFS.3
- new net: HFYF.2, HGDM.3
- new net: KBGM.7 (Q), KGHB.2, KHAD.1, QABF.3 (2)
- new net: HGRD.1, HIPM.3, KBGM.3 (CLK), KBGM.4 (~{CLK})
- new net: JFRL.3, KBGM.2 (D)
- new net: JFLO.1, JFRL.2, KBGM.7 (Q)
- new net: JFHM.1, JFLO.2, KBGM.7 (Q)
- new net: JFLO.3, KBGM.2 (D)
- new net: CABL8.3, KBGM.2 (D)
- new net: HHOM.3, KBGM.1 (~{RESET}), KBGM.1 (~{RESET}), KBGM.5 (~{RESET}), KBGM.5 (~{RESET})
- new net: HHKS.3, KBGM.3 (CLK), KBGM.3 (CLK), KBGM.4 (~{CLK}), KBGM.4 (~{CLK})
- new net: ACHJ1.1 (IN), ACHJ1.3 (IN), IGKE.2, IGOJ.1, KBGM.7 (Q)
- new net: IGOJ.3, KBGM.2 (D)
- new net: HFYF.3, HGHK.2
- new net: HGRQ.2, HGUU.2
- new net: CABL2.2, CABL3.2, CABL4.2, CABL5.2, CABL6.2, CABL7.2, CABL8.2, CABL9.2
- new net: CABL7.3, KBGM.2 (D)
- new net: CABL2.4, CABL3.4, CABL4.4, CABL5.4, CABL6.4, CABL7.4, CABL8.4, CABL9.4
- new net: KBGM.2 (D), KBGM.6 (~{Q})
- new net: HIEP.4, KBGM.7 (Q)
- new net: HHEB.2, OACG.1, OACG.1, TBUI.1
- new net: KBGM.2 (D), KFZV.3
- new net: ABXH1.1 (IN), ABXH1.3 (IN), IGLE.2, IGOK.1, KBGM.7 (Q)
- new net: ABWF1.1 (IN), ABWF1.3 (IN), IGOK.2, IGUE.1, KBGM.7 (Q)
- new net: IGUE.2, KBGM.6 (Q)
- new net: IGUE.3, KBGM.2 (D)
- new net: IGUE.5, JGSQ6.4 (Q)
- new net: JFDF.1, JFKA.2, KBGM.7 (Q)
- new net: JFHM.3, KBGM.2 (D)
- new net: IGKE.5, JGSQ1.4 (Q)
- new net: IGLE.3, KBGM.2 (D)
- new net: CABL5.3, KBGM.2 (D)
- new net: HIBX.2, HIEP.1, KBGM.7 (Q)
- new net: CABL9.3, KBGM.2 (D)
- new net: JHDZ.3, KHXL.5
- new net: OACG.1, OACG.1, TBUI.3
- new net: HHXX.1, HIBX.5
- new net: KBGM.2 (D), KIDU.3
- new net: KBGM.2 (D), KFMZ.3
- new net: IGLE.5, JGSQ2.4 (Q)
- new net: HGJS1.1, HHFN1.2
- new net: HGJS1.3, HHDH1.1
- new net: CABL6.3, JGSQ10.4 (Q)
- new net: CABL3.3, KBGM.2 (D)
- new net: CABL2.3, JGMY1.4 (Q)
- new net: KBGM.2 (D), KHXL.3
- new net: JFKA.1, JFQD.2, KBGM.7 (Q)
- new net: FGKE.2, KBGM.1 (~{RESET}), KBGM.3 (CLK), KBGM.4 (~{CLK}), KBGM.5 (~{RESET})
- new net: IGOK.5, JGSQ4.4 (Q)
- new net: IFCU.3, KBGM.2 (D)
- new net: HHOM.1, KBGM.6 (~{Q})
- new net: HHOM.2, KBGM.2 (D), KBGM.7 (Q)
- new net: IGKE.3, KBGM.2 (D)
- new net: ACBV1.1 (IN), ACBV1.3 (IN), IGHG.2, IGLE.1, KBGM.7 (Q)
- new net: KBGM.7 (Q), KHYE.2, KIDU.1, QABF.3 (2)
- new net: JHSZ.3, KIDU.5
- new net: KBGM.2 (D), KHAD.3
- new net: JGRZ.3, KHAD.5
- new net: HFPC.2, HFSC.3
- new net: CABL4.3, KBGM.2 (D)
- new net: JFKA.3, KBGM.2 (D)
- new net: IGOK.3, KBGM.2 (D)
- new net: CABL5.3, JGSQ9.4 (Q)
- new net: JHHT.3, KHYE.5
- new net: HFJQ.3, HFPC.1
- new net: HIBX.3, HIEP.2, KBGM.7 (Q)
- new net: IFXO.3, KBGM.2 (D)
- new net: HFPC.3, HFYF.1
- new net: JFQD.3, KBGM.2 (D)
- new net: IGFF.3, KBGM.2 (D)
- new net: IFQQ.3, KBGM.2 (D)
- new net: KBGM.2 (D), KHYE.3
- new net: KBGM.2 (D), KFYB.3
- new net: GBEG.4, HHDH1.2
- new net: GBEG.1, HHFN2.1
- new net +5V: KBGM.2 (D)
- new net 4202_WR: JGMY.1 (~{ENA}), JGMY.3 (ENA), JGSQ.1 (~{ENA}), JGSQ.3 (ENA), JGSQ1.1 (~{ENA}), JGSQ1.3 (ENA), JGSQ2.1 (~{ENA}), JGSQ2.3 (ENA), JGSQ3.1 (~{ENA}), JGSQ3.3 (ENA), JGSQ4.1 (~{ENA}), JGSQ4.3 (ENA), JGSQ5.1 (~{ENA}), JGSQ5.3 (ENA), JGSQ6.1 (~{ENA}), JGSQ6.3 (ENA)
- new net 4204_WR: JGMY1.1 (~{ENA}), JGMY1.3 (ENA), JGSQ10.1 (~{ENA}), JGSQ10.3 (ENA), JGSQ11.1 (~{ENA}), JGSQ11.3 (ENA), JGSQ12.1 (~{ENA}), JGSQ12.3 (ENA), JGSQ13.1 (~{ENA}), JGSQ13.3 (ENA), JGSQ7.1 (~{ENA}), JGSQ7.3 (ENA), JGSQ8.1 (~{ENA}), JGSQ8.3 (ENA), JGSQ9.1 (~{ENA}), JGSQ9.3 (ENA)
- new net D0: ABVA1.4, ABVA1.4, IFXO.5, JGSQ13.2 (D), JGSQ6.2 (D), JHSZ.2, KFCL.2
- new net D1: ABWF1.4, ABWF1.4, IFWE.5, JFDF.5, JGSQ12.2 (D), JGSQ5.2 (D), JHSJ.2
- new net D2: ABXH1.4, ACKH1.4, IFUF.5, JFHM.5, JGSQ11.2 (D), JGSQ4.2 (D), JHHT.2
- new net D3: ABXH1.4, ACBV1.4, IFQQ.5, JFKA.5, JGSQ10.2 (D), JGSQ3.2 (D), JHDZ.2
- new net D4: ACGM1.4, ACHJ1.4, IFMP.5, JFLO.5, JGSQ2.2 (D), JGSQ9.2 (D), JGYV.2
- new net D5: ACBV1.4, ACHJ1.4, IFMG.5, JFQD.5, JGSQ1.2 (D), JGSQ8.2 (D), JGYM.2
- new net D6: ACJG1.4, ACJG1.4, IFEQ.5, JFRL.5, JGRZ.2, JGSQ.2 (D), JGSQ7.2 (D)
- new net D7: ACGM1.4, ACKH1.4, IFCU.5, JFRP.5, JGMY.2 (D), JGMY1.2 (D), JGON.2
- new net GND: IFCU.1, JFRP.1, KFCQ.5, KFMZ.5, KFOX.5, KFYB.5, KFZV.5, KGGW.5, KGHB.5
- new net MUL_CLK: HGRD.3, HGRD1.2, OACG.1, OACG.1
- new net MUL_OR_DIV_ON: HGJS.3, HGRQ.1, HHDH.1, HHEB.1, HHFN.1, HIPM.2, KBGM.3 (CLK), KBGM.4 (~{CLK})
- new net OAGE: FGKE.1, HIPM.1, KBGM.3 (CLK), KBGM.3 (CLK), KBGM.4 (~{CLK}), KBGM.4 (~{CLK})
- new net wDBJW_wHASI_RST: KBGM.1 (~{RESET}), KBGM.1 (~{RESET}), KBGM.1 (~{RESET}), KBGM.1 (~{RESET}), KBGM.5 (~{RESET}), KBGM.5 (~{RESET}), KBGM.5 (~{RESET}), KBGM.5 (~{RESET})
- new net wHGHK: CABL1.1, HGHK.3, KBGM.2 (D)
- new net wKBNZ: GBEG.2, HHFN1.1
- new net ~{4203}: KBGM.2 (D), KFCL.1
- new net ~{4206}: JGON.1, JGRZ.1, JGYM.1, JGYV.1, JHDZ.1, JHHT.1, JHSJ.1, JHSZ.1, KBGM.2 (D)
- new net ~{MUL_DIV_DONE}: HHXX.3, KBGM.2 (D)
- new net ~{wHGKB}_DIV_ON: HGJS.2, HIBX.1, KBGM.6 (~{Q})
- new net ~{wHHJU}_MUL_ON: CABL1.2, HGJS.1, HGUU.1, HHDH.2, HHFN4.1, HIBF.1, KBGM.6 (~{Q})
- new net ~{wJFDZ}: HFJQ.1, KBGM.6 (~{Q})
- new net ~{wJFGY}: HFJQ.2, KBGM.6 (~{Q})
- new net ~{wJFKL}: HFSC.1, KBGM.6 (~{Q})
- new net ~{wJFLK}: HFSC.2, KBGM.6 (~{Q})
- new net ~{wJFRA}: HGFS.1, KBGM.6 (~{Q})
- new net ~{wJFRC}: HGFS.2, KBGM.6 (~{Q})
- new net ~{wJFRT}: HGDM.2, KBGM.6 (~{Q})
- no-connect marks 0 -> 77
Other:
- note added: "Adder output Sum or Carry?"
- note added: "CLK/8?"
- note added: "MUL takes 16 OAGE cycles TBD? Counter is reset by HIOV when MUL or DIV is started for a couple of cycles. Reset is released on the next OAGE positve level. MUL values are latched by MUL_CLK when writing to 4203 and then anoher 16 times when MUL is ON."
- note added: "Reset when ~{MUL_DIV_DONE} falling edge is detected"

Commit message: MUL DIV section almost done.
Parts:
- added ABVA1 (x2), ABWF1 (x2), ABXH1 (x2), ACBV1 (x2), ACGM1 (x2), ACHJ1 (x2), ACJG1 (x2), ACKH1 (x2): TRI_BUF_IF0, symbol Ricoh_Cells:TRI_BUF_IF0
- added KBGM (x8): DFFR_B, symbol Ricoh_Cells:DFFR_B
- added LFDU, LFFC, LFFN, LFHO, LFNW, LFQZ, LFRR, LFUD: 2BIT_FULL_ADD, symbol Ricoh_Cells:2BIT_FULL_ADD
- added MFGG, MFMC, MFSP, MFUS, MGFY, MGJF, MGQB, MGQS: AOI_22, symbol Ricoh_Cells:AOI_22
- added MGVV, MGZJ: INVERTER_A, symbol Ricoh_Cells:INVERTER_A
- added NFBN, NFFC, NFJJ, NFOI, NFRO, NFSB, NFVQ, NFWE: D_LATCH_A2, symbol Ricoh_Cells:D_LATCH_A2
- added OACG (x8): DELAY_BUF, symbol Ricoh_Cells:DELAY_BUF
- renumbered HHFN3 to LFHS, CABL1 to LFIH, HHFN4 to LFII, HGRD1 to LFJV, CABL2 to MHEA, CABL3 to MHEK, CABL4 to MHMG, CABL5 to MHOU, CABL6 to MHWQ, CABL7 to MHXO, CABL8 to MIDS, CABL9 to MIFC, HHFN2 to NFXH, HHFN1 to NFYD, HGJS1 to NGBH, HHDH1 to NGLG, JGMY1 to NGNU, JGSQ7 to NGQS, JGSQ8 to NGVS, JGSQ9 to NHCN, JGSQ10 to NHHH, JGSQ11 to NHPK, JGSQ12 to NHSH, JGSQ13 to NHUE
Connections:
- net D0: now also ABVA1.4, ABVA1.4, NFWE.2 (D)
- net D1: now also ABWF1.4, ABWF1.4, NFVQ.2 (D)
- net D2: now also ACKH1.4, ACKH1.4, NFSB.2 (D)
- net D3: now also ABXH1.4, ABXH1.4, NFRO.2 (D)
- net D4: now also ACHJ1.4, ACHJ1.4, NFOI.2 (D)
- net D5: now also ACBV1.4, ACBV1.4, NFJJ.2 (D)
- net D6: now also ACJG1.4, ACJG1.4, NFFC.2 (D)
- net D7: now also ACGM1.4, ACGM1.4, NFBN.2 (D)
- net GND: now also KIDU.2
- net ~{4203_WR}: now also OACG.1, OACG.1
- net ~{4206_WR}: now also MGVV.1, OACG.1, OACG.1
- net ~{4216_RD}: now also ABVA1.2 (~{ENA}), ABWF1.2 (~{ENA}), ABXH1.2 (~{ENA}), ACBV1.2 (~{ENA}), ACGM1.2 (~{ENA}), ACHJ1.2 (~{ENA}), ACJG1.2 (~{ENA}), ACKH1.2 (~{ENA})
- net ~{4217_RD}: now also MHEA.2, MHEK.2, MHMG.2, MHOU.2, MHWQ.2, MHXO.2, MIDS.2, MIFC.2, ABVA1.2 (~{ENA}), ABWF1.2 (~{ENA}), ABXH1.2 (~{ENA}), ACBV1.2 (~{ENA}), ACGM1.2 (~{ENA}), ACHJ1.2 (~{ENA}), ACJG1.2 (~{ENA}), ACKH1.2 (~{ENA}), OACG.2
- net MUL_SHL_2: now reaches KGZD.3, KHAD.3, KHRF.3, KHSS.3, KHXL.3, KHYE.3, KICH.3, KIDU.3, OACG.2
- net DIV_SHR_2: now reaches KGZD.4, KHAD.4, KHRF.4, KHSS.4, KHXL.4, KHYE.4, KICH.4, KIDU.4, OACG.2
- net LD_ADDER_BOTTOM: now reaches KGZD.6, KHAD.6, KHRF.6, KHSS.6, KHXL.6, KHYE.6, KICH.6, KIDU.6, OACG.2
- net at QABF.1: now also LFHO.24 (A1)
- net at QABF.2 (1), QABF.2 (1), QABF.2 (1)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: now also OACG.2; no longer QABF.2 (1), QABF.2 (1), QABF.2 (1), QABF.2 (1), QABF.2 (1), QABF.2 (1), QABF.2 (1), QABF.2 (1)
- net MUL_SHL_1: now reaches JFCT.3, JFDF.3, JFHM.3, JFKA.3, JFLO.3, JFQD.3, JFRL.3, JFRP.3, KFCQ.3, KFMZ.3, KFOX.3, KFYB.3, KFZV.3, KGGW.3, KGHB.3, OACG.2, OACG.2
- net DIV_SHL_1: now reaches IFCU.3, IFEQ.3, IFMG.3, IFMP.3, IFQQ.3, IFUF.3, IFWE.3, IFXO.3, OACG.2
- net MUL_SHR_1: now reaches IFCU.4, IFEQ.4, IFMG.4, IFMP.4, IFQQ.4, IFUF.4, IFWE.4, IFXO.4, OACG.2
- net LD_4203: now reaches IFCU.6, IFEQ.6, IFMG.6, IFMP.6, IFQQ.6, IFUF.6, IFWE.6, IFXO.6, OACG.2
- net at KBGM.1 (~{RESET}), KBGM.1 (~{RESET}), KBGM.1 (~{RESET})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: now also OACG.2
- net at KBGM.3 (CLK), KBGM.3 (CLK), KBGM.3 (CLK)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: now also OACG.2
- net at KBGM.7 (Q): now also ABXH1.1 (IN), ABXH1.3 (IN), LFRR.23 (B1)
- net at QABF.1: now also LFFN.13 (A0)
- net DO_ADD_SUB: now reaches NGLG.3, OACG.1, OACG.1
- net at OACG.2: now also KBGM.3 (CLK), KBGM.3 (CLK), KBGM.3 (CLK), KBGM.3 (CLK), KBGM.3 (CLK), KBGM.3 (CLK), KBGM.3 (CLK), KBGM.3 (CLK), KBGM.4 (~{CLK}), KBGM.4 (~{CLK}), KBGM.4 (~{CLK}), KBGM.4 (~{CLK}), KBGM.4 (~{CLK}), KBGM.4 (~{CLK}), KBGM.4 (~{CLK}), KBGM.4 (~{CLK}); no longer OACG.2
- net at KBGM.7 (Q): now also ACGM1.1 (IN), ACGM1.3 (IN), LFNW.23 (B1)
- net at QABF.1: now also LFDU.24 (A1)
- net LD_ADDER_TOP: now reaches JFCT.6, JFDF.6, JFHM.6, JFKA.6, JFLO.6, JFQD.6, JFRL.6, JFRP.6, KFCQ.6, KFMZ.6, KFOX.6, KFYB.6, KFZV.6, KGGW.6, KGHB.6, OACG.2, OACG.2
- net at QABF.1: now also LFRR.13 (A0)
- net DIV_SHR_1: now reaches JFCT.4, JFDF.4, JFHM.4, JFKA.4, JFLO.4, JFQD.4, JFRL.4, JFRP.4, KFCQ.4, KFMZ.4, KFOX.4, KFYB.4, KFZV.4, KGGW.4, KGHB.4, OACG.2, OACG.2
- net at KBGM.7 (Q): now also GBEG.1
- net 4214_D0: now reaches ABVA1.1 (IN), ABVA1.3 (IN), IGST.2, KBGM.7 (Q), LFIH.3
- net at QABF.1: now also LFQZ.24 (A1)
- net DIV_SHL_2: now reaches IGFF.3, IGHG.3, IGKE.3, IGLE.3, IGOJ.3, IGOK.3, IGST.3, IGUE.3, OACG.2
- net MUL_SHR_2: now reaches IGFF.4, IGHG.4, IGKE.4, IGLE.4, IGOJ.4, IGOK.4, IGST.4, IGUE.4, OACG.2
- net LD_4202: now reaches IGFF.6, IGHG.6, IGKE.6, IGLE.6, IGOJ.6, IGOK.6, IGST.6, IGUE.6, OACG.2
- net wHIPM: now reaches HGRD.1, HIPM.3, KBGM.3 (CLK), KBGM.4 (~{CLK})
- net wHIPM: now also GBEG.3, NFXH.1
- net at KBGM.7 (Q): now also ABWF1.1 (IN), ABWF1.3 (IN), LFUD.23 (B1)
- net at HGHK.1: now also LFDU.28 (COUT)
- net at MHXO.1: now also LFRR.4 (SUM0)
- net at MHEA.4, MHEK.4, MHMG.4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: now also OACG.2
- net at QABF.1: now also LFNW.24 (A1)
- net at KBGM.7 (Q): now also ACHJ1.1 (IN), ACHJ1.3 (IN), LFQZ.9 (B0)
- net at MIFC.1: now also LFUD.4 (SUM0)
- net at QABF.1: now also LFQZ.13 (A0)
- net at KBGM.7 (Q): now also ACKH1.1 (IN), ACKH1.3 (IN), LFRR.9 (B0)
- net at MHWQ.1: now also LFRR.17 (SUM1)
- net at KBGM.7 (Q): now also ACJG1.1 (IN), ACJG1.3 (IN), LFNW.9 (B0)
- net at QABF.1: now also LFNW.13 (A0)
- net at MHEA.1: now also LFNW.17 (SUM1)
- net at QABF.1: now also LFRR.24 (A1)
- net at QABF.1: now also LFDU.13 (A0)
- net at QABF.1: now also LFFN.24 (A1)
- net at MHMG.1: now also LFQZ.17 (SUM1)
- net at QABF.1: now also LFHO.13 (A0)
- net at KBGM.7 (Q): now also ACBV1.1 (IN), ACBV1.3 (IN), LFQZ.23 (B1)
- net at MIDS.1: now also LFUD.17 (SUM1)
- net at QABF.1: now also LFUD.24 (A1)
- net at QABF.1: now also LFUD.13 (A0)
- net at QABF.1: now also LFFC.24 (A1)
- net at MHEK.1: now also LFNW.4 (SUM0)
- net at KBGM.7 (Q): now also ABVA1.1 (IN), ABVA1.3 (IN), LFUD.9 (B0)
- net at QABF.1: now also LFFC.13 (A0)
- net at MHOU.1: now also LFQZ.4 (SUM0)
- net MUL_CLK renamed MUL_DIV_CLK
- net wHGHK renamed wHGHK_ZDIV
- net ~{wHGKB}_DIV_ON renamed ~{wHGKB}_MUL_ON
- net ~{wHHJU}_MUL_ON renamed ~{wHHJU}_DIV_ON
- net ~{wHHJU}_DIV_ON: now also LFUD.2 (CIN), MGZJ.1
- net ~{wJFDZ}: no longer names the net of HFJQ.1, KBGM.6 (~{Q})
- net ~{wJFGY}: no longer names the net of HFJQ.2, KBGM.6 (~{Q})
- net ~{wJFKL}: no longer names the net of HFSC.1, KBGM.6 (~{Q})
- net ~{wJFLK}: no longer names the net of HFSC.2, KBGM.6 (~{Q})
- net ~{wJFRA}: no longer names the net of HGFS.1, KBGM.6 (~{Q})
- net ~{wJFRC}: no longer names the net of HGFS.2, KBGM.6 (~{Q})
- net ~{wJFRT}: no longer names the net of HGDM.2, KBGM.6 (~{Q})
- new net: LFFC.4 (SUM0), MFUS.1
- new net: MFGG.2, MFMC.2, MFSP.2, MFUS.2, MGFY.2, MGJF.2, MGQB.2, MGQS.2, OACG.2
- new net: KBGM.2 (D), MFUS.3
- new net: MFUS.3, NFOI.4 (Q)
- new net: MFGG.4, MFMC.4, MFSP.4, MFUS.4, MGFY.4, MGJF.4, MGQB.4, MGQS.4, OACG.2
- new net: MFGG.3, NFBN.4 (Q)
- new net: MGZJ.2, OACG.1, OACG.1
- new net: OACG.2, QABF.2 (1), QABF.2 (1), QABF.2 (1), QABF.2 (1), QABF.2 (1), QABF.2 (1), QABF.2 (1), QABF.2 (1)
- new net: MGVV.2, OACG.1, OACG.1
- new net: LFFN.2 (CIN), LFHO.28 (COUT)
- new net: LFFN.4 (SUM0), MGJF.1
- new net: ACKH1.1 (IN), ACKH1.3 (IN), KBGM.7 (Q), LFFN.9 (B0)
- new net: KBGM.1 (~{RESET}), KBGM.1 (~{RESET}), KBGM.1 (~{RESET}), KBGM.1 (~{RESET}), KBGM.1 (~{RESET}), KBGM.1 (~{RESET}), KBGM.1 (~{RESET}), KBGM.1 (~{RESET}), KBGM.5 (~{RESET}), KBGM.5 (~{RESET}), KBGM.5 (~{RESET}), KBGM.5 (~{RESET}), KBGM.5 (~{RESET}), KBGM.5 (~{RESET}), KBGM.5 (~{RESET}), KBGM.5 (~{RESET}), OACG.2
- new net: ACHJ1.1 (IN), ACHJ1.3 (IN), KBGM.7 (Q), LFFC.9 (B0)
- new net: LFFC.17 (SUM1), MFSP.1
- new net: KBGM.2 (D), MFSP.3
- new net: MFSP.3, NFJJ.4 (Q)
- new net: MGJF.3, NFSB.4 (Q)
- new net: LFHO.17 (SUM1), MGQB.1
- new net: KBGM.2 (D), MGQB.3
- new net: MGQB.3, NFVQ.4 (Q)
- new net: LFDU.17 (SUM1), MFGG.1
- new net: ACGM1.1 (IN), ACGM1.3 (IN), KBGM.7 (Q), LFDU.23 (B1)
- new net: ACBV1.1 (IN), ACBV1.3 (IN), KBGM.7 (Q), LFFC.23 (B1)
- new net: LFQZ.2 (CIN), LFRR.28 (COUT)
- new net: LFNW.2 (CIN), LFQZ.28 (COUT)
- new net: KBGM.2 (D), MFMC.3
- new net: ACJG1.1 (IN), ACJG1.3 (IN), KBGM.7 (Q), LFDU.9 (B0)
- new net: LFDU.2 (CIN), LFFC.28 (COUT)
- new net: LFRR.2 (CIN), LFUD.28 (COUT)
- new net: KBGM.2 (D), MGFY.3
- new net: ABXH1.1 (IN), ABXH1.3 (IN), KBGM.7 (Q), LFFN.23 (B1)
- new net: KBGM.2 (D), MGJF.3
- new net: ABVA1.1 (IN), ABVA1.3 (IN), KBGM.7 (Q), LFHO.9 (B0)
- new net: LFHO.4 (SUM0), MGQS.1
- new net: KBGM.2 (D), MGQS.3
- new net: MGQS.3, NFWE.4 (Q)
- new net: ABWF1.1 (IN), ABWF1.3 (IN), KBGM.7 (Q), LFHO.23 (B1)
- new net: MFMC.3, NFFC.4 (Q)
- new net: LFHO.2 (CIN), LFNW.28 (COUT)
- new net: LFFC.2 (CIN), LFFN.28 (COUT)
- new net: LFDU.4 (SUM0), MFMC.1
- new net: LFFN.17 (SUM1), MGFY.1
- new net: KBGM.2 (D), MFGG.3
- new net: MGFY.3, NFRO.4 (Q)
- new net 4205_WR: NFBN.1 (~{ENA}), NFBN.3 (ENA), NFFC.1 (~{ENA}), NFFC.3 (ENA), NFJJ.1 (~{ENA}), NFJJ.3 (ENA), NFOI.1 (~{ENA}), NFOI.3 (ENA), NFRO.1 (~{ENA}), NFRO.3 (ENA), NFSB.1 (~{ENA}), NFSB.3 (ENA), NFVQ.1 (~{ENA}), NFVQ.3 (ENA), NFWE.1 (~{ENA}), NFWE.3 (ENA)
- no-connect marks 77 -> 93
Other:
- note added: "4202 WRITE MULTIPLICAND"
- note added: "4203 WRITE (MULTIPLIER) OR 4206 WRITE OR SHL/SHR"
- note added: "4203 WRITE (MULTIPLIER) OR SHL/SHR"
- note added: "4204 WRITE"
- note added: "4205 WRITE"
- note added: "4214 READ"
- note added: "4215 READ"
- note added: "4216 READ"
- note added: "4217 READ"
- note added: "DFF15-8 are loaded with data bus and DFF7-0 are loaded with 4202 stored when 4203 is written to while there is no multiplication or division in progress otherwise, data is 1) right shifted and added during multiplication 2) left shifted and subtracted during division"
- note added: "MUL takes 8 OAGE cycles Counter is reset by HIOV when MUL or DIV is started for a couple of cycles. Reset is released on the next OAGE positve level. MUL values are latched by MUL_CLK when writing to 4203 and then anoher 8 times when MUL is ON. DIV takes 16 cycles"
- note added: "Writing to 4203 clears the Product/Remainder Result stored in 4216 and 4217 Writing to 4206 loads values staored in 4204 and 4205 into Product/Remainder."
- note added: "Writing to 4203 will load data bus as multiplier but writing to 4206 will clear it."
- note removed: "Adder output Sum or Carry?"
- note removed: "MUL takes 16 OAGE cycles TBD? Counter is reset by HIOV when MUL or DIV is started for a couple of cycles. Reset is released on the next OAGE positve level. MUL values are latched by MUL_CLK when writing to 4203 and then anoher 16 times when MUL is ON."
- moved on the sheet: ABVA1, ABWF1, ABXH1, ACBV1, ACGM1, ACHJ1, ACJG1, ACKH1, FGKE, GBEG, HFJQ, HFPC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
