File: S-CPU_kicad/addrdatabuses.kicad_sch (KiCad schematic)
At the start: 84 parts

Commit message: More MUL DIV section updates,
Changed lines of the file:
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@@
       (effects (font (size 1.27 1.27)))
     )
-    (property "Value" "TRI_BUF_IF0" (at 266.7 96.925 0)
+    (property "Value" "TRI_BUF_IF0" (at 266.7 97.155 0)
       (effects (font (size 1.27 1.27)))
     )
@@
       (effects (font (size 1.27 1.27)))
     )
-    (property "Value" "TRI_BUF_IF0" (at 542.925 144.6135 0)
+    (property "Value" "TRI_BUF_IF0" (at 542.925 144.78 0)
       (effects (font (size 1.27 1.27)))
     )
@@
       (effects (font (size 1.27 1.27)))
     )
-    (property "Value" "TRI_BUF_IF0" (at 153.67 234.1485 0)
+    (property "Value" "TRI_BUF_IF0" (at 153.67 234.315 0)
       (effects (font (size 1.27 1.27)))
     )
@@
       (effects (font (size 1.27 1.27)))
     )
-    (property "Value" "TRI_BUF_IF0" (at 542.925 177.6335 0)
+    (property "Value" "TRI_BUF_IF0" (at 542.925 177.8 0)
       (effects (font (size 1.27 1.27)))
     )
@@
       (effects (font (size 1.27 1.27)))
     )
-    (property "Value" "TRI_BUF_IF0" (at 153.67 167.4735 0)
+    (property "Value" "TRI_BUF_IF0" (at 153.67 167.64 0)
       (effects (font (size 1.27 1.27)))
     )
@@
       (effects (font (size 1.27 1.27)))
     )
-    (property "Value" "TRI_BUF_IF0" (at 284.48 96.925 0)
+    (property "Value" "TRI_BUF_IF0" (at 284.48 97.155 0)
       (effects (font (size 1.27 1.27)))
     )
@@
       (effects (font (size 1.27 1.27)))
     )
-    (property "Value" "TRI_BUF_IF0" (at 542.925 194.1435 0)
+    (property "Value" "TRI_BUF_IF0" (at 542.925 194.31 0)
       (effects (font (size 1.27 1.27)))
     )
@@
       (effects (font (size 1.27 1.27)))
     )
-    (property "Value" "TRI_BUF_IF0" (at 153.67 80.4785 0)
+    (property "Value" "TRI_BUF_IF0" (at 153.67 80.645 0)
       (effects (font (size 1.27 1.27)))
     )
@@
       (effects (font (size 1.27 1.27)))
     )
-    (property "Value" "TRI_BUF_IF0" (at 271.145 213.8285 0)
+    (property "Value" "TRI_BUF_IF0" (at 271.145 213.995 0)
       (effects (font (size 1.27 1.27)))
     )
@@
       (effects (font (size 1.27 1.27)))
     )
-    (property "Value" "TRI_BUF_IF0" (at 153.67 189.6985 0)
+    (property "Value" "TRI_BUF_IF0" (at 153.67 189.865 0)
       (effects (font (size 1.27 1.27)))
     )
@@
       (effects (font (size 1.27 1.27)))
     )
-    (property "Value" "TRI_BUF_IF0" (at 271.145 169.3785 0)
+    (property "Value" "TRI_BUF_IF0" (at 271.145 169.545 0)
       (effects (font (size 1.27 1.27)))
     )
@@
       (effects (font (size 1.27 1.27)))
     )
-    (property "Value" "TRI_BUF_IF0" (at 271.145 302.7285 0)
+    (property "Value" "TRI_BUF_IF0" (at 271.145 302.895 0)
       (effects (font (size 1.27 1.27)))
     )
@@
       (effects (font (size 1.27 1.27)))
     )
-    (property "Value" "TRI_BUF_IF0" (at 153.67 100.7985 0)
+    (property "Value" "TRI_BUF_IF0" (at 153.67 100.965 0)
       (effects (font (size 1.27 1.27)))
     )
@@
       (effects (font (size 1.27 1.27)))
     )
-    (property "Value" "TRI_BUF_IF0" (at 542.925 111.5935 0)
+    (property "Value" "TRI_BUF_IF0" (at 542.925 111.76 0)
       (effects (font (size 1.27 1.27)))
     )
@@
       (effects (font (size 1.27 1.27)))
     )
-    (property "Value" "TRI_BUF_IF0" (at 542.925 161.1235 0)
+    (property "Value" "TRI_BUF_IF0" (at 542.925 161.29 0)
       (effects (font (size 1.27 1.27)))
     )
@@
       (effects (font (size 1.27 1.27)))
     )
-    (property "Value" "TRI_BUF_IF0" (at 266.7 80.4785 0)
+    (property "Value" "TRI_BUF_IF0" (at 266.7 80.645 0)
       (effects (font (size 1.27 1.27)))
     )
@@
       (effects (font (size 1.27 1.27)))
     )
-    (property "Value" "TRI_BUF_IF0" (at 443.23 127.4685 0)
+    (property "Value" "TRI_BUF_IF0" (at 443.23 127.635 0)
       (effects (font (size 1.27 1.27)))
     )
@@
       (effects (font (size 1.27 1.27)))
     )
-    (property "Value" "TRI_BUF_IF0" (at 443.23 193.5085 0)
+    (property "Value" "TRI_BUF_IF0" (at 443.23 193.675 0)
       (effects (font (size 1.27 1.27)))
     )
@@
       (effects (font (size 1.27 1.27)))
     )
-    (property "Value" "TRI_BUF_IF0" (at 443.23 110.9585 0)
+    (property "Value" "TRI_BUF_IF0" (at 443.23 111.125 0)
       (effects (font (size 1.27 1.27)))
     )
@@
       (effects (font (size 1.27 1.27)))
     )
-    (property "Value" "TRI_BUF_IF0" (at 302.26 96.925 0)
+    (property "Value" "TRI_BUF_IF0" (at 302.26 97.155 0)
       (effects (font (size 1.27 1.27)))
     )
@@
       (effects (font (size 1.27 1.27)))
     )
-    (property "Value" "TRI_BUF_IF0" (at 443.23 210.0185 0)
+    (property "Value" "TRI_BUF_IF0" (at 443.23 210.185 0)
       (effects (font (size 1.27 1.27)))
     )
@@
       (effects (font (size 1.27 1.27)))
     )
-    (property "Value" "TRI_BUF_IF0" (at 542.925 95.0835 0)
+    (property "Value" "TRI_BUF_IF0" (at 542.925 95.25 0)
       (effects (font (size 1.27 1.27)))
     )
@@
       (effects (font (size 1.27 1.27)))
     )
-    (property "Value" "TRI_BUF_IF0" (at 443.23 143.9785 0)
+    (property "Value" "TRI_BUF_IF0" (at 443.23 144.145 0)
       (effects (font (size 1.27 1.27)))
     )
@@
       (effects (font (size 1.27 1.27)))
     )
-    (property "Value" "TRI_BUF_IF0" (at 443.23 160.4885 0)
+    (property "Value" "TRI_BUF_IF0" (at 443.23 160.655 0)
       (effects (font (size 1.27 1.27)))
     )
@@
       (effects (font (size 1.27 1.27)))
     )
-    (property "Value" "TRI_BUF_IF0" (at 443.23 176.9985 0)
+    (property "Value" "TRI_BUF_IF0" (at 443.23 177.165 0)
       (effects (font (size 1.27 1.27)))
     )
@@
       (effects (font (size 1.27 1.27)))
     )
-    (property "Value" "TRI_BUF_IF0" (at 153.67 123.0235 0)
+    (property "Value" "TRI_BUF_IF0" (at 153.67 123.19 0)
       (effects (font (size 1.27 1.27)))
     )
@@
       (effects (font (size 1.27 1.27)))
     )
-    (property "Value" "TRI_BUF_IF0" (at 271.145 191.6035 0)
+    (property "Value" "TRI_BUF_IF0" (at 271.145 191.77 0)
       (effects (font (size 1.27 1.27)))
     )
@@
       (effects (font (size 1.27 1.27)))
     )
-    (property "Value" "TRI_BUF_IF0" (at 153.67 145.2485 0)
+    (property "Value" "TRI_BUF_IF0" (at 153.67 145.415 0)
       (effects (font (size 1.27 1.27)))
     )
@@
       (effects (font (size 1.27 1.27)))
     )
-    (property "Value" "TRI_BUF_IF0" (at 542.925 210.6535 0)
+    (property "Value" "TRI_BUF_IF0" (at 542.925 210.82 0)
       (effects (font (size 1.27 1.27)))
     )
@@
       (effects (font (size 1.27 1.27)))
     )
-    (property "Value" "TRI_BUF_IF0" (at 153.67 211.9235 0)
+    (property "Value" "TRI_BUF_IF0" (at 153.67 212.09 0)
       (effects (font (size 1.27 1.27)))
     )
@@
       (effects (font (size 1.27 1.27)))
     )
-    (property "Value" "TRI_BUF_IF0" (at 271.145 236.0535 0)
+    (property "Value" "TRI_BUF_IF0" (at 271.145 236.22 0)
       (effects (font (size 1.27 1.27)))
     )
@@
       (effects (font (size 1.27 1.27)))
     )
-    (property "Value" "TRI_BUF_IF0" (at 266.7 113.435 0)
+    (property "Value" "TRI_BUF_IF0" (at 266.7 113.665 0)
       (effects (font (size 1.27 1.27)))
     )
@@
       (effects (font (size 1.27 1.27)))
     )
-    (property "Value" "TRI_BUF_IF0" (at 271.145 280.5035 0)
+    (property "Value" "TRI_BUF_IF0" (at 271.145 280.67 0)
       (effects (font (size 1.27 1.27)))
     )
@@
       (effects (font (size 1.27 1.27)))
     )
-    (property "Value" "TRI_BUF_IF0" (at 271.145 258.2785 0)
+    (property "Value" "TRI_BUF_IF0" (at 271.145 258.445 0)
       (effects (font (size 1.27 1.27)))
     )
@@
       (effects (font (size 1.27 1.27)))
     )
-    (property "Value" "TRI_BUF_IF0" (at 542.925 128.1035 0)
+    (property "Value" "TRI_BUF_IF0" (at 542.925 128.27 0)
       (effects (font (size 1.27 1.27)))
     )
@@
       (effects (font (size 1.27 1.27)))
     )
-    (property "Value" "TRI_BUF_IF0" (at 443.23 94.4485 0)
-      (effects (font (size 1.27 1.27)))
-    )
+    (property "Value" "TRI_BUF_IF0" (at 443.23 94.615 0)
+      (effects (font (size 1.27 1.27)))
+    )

Commit message: D latch with reset and tri state output identified
Parts:
- removed HANV1, HANV2, HANV3: TRI_BUF_IF0, symbol Ricoh_Cells:TRI_BUF_IF0
- added DMA? (x3): TRI_BUF_IF0, symbol Ricoh_Cells:TRI_BUF_IF0
- added HANV, HAPY, JBTI, MAOJ: DR_TRI_LATCH, symbol Ricoh_Cells:DR_TRI_LATCH
Connections:
- net 65816_A7: now also HANV.2 (D)
- net A4: now also DMA?.4, JBTI.5 (Q)
- net A5: now also DMA?.4, MAOJ.5 (Q)
- net A6: now also DMA?.4, HAPY.5 (Q)
- net A7: now also HANV.5 (Q)
- net wHAKW: now also HANV.1 (DIS), HAPY.1 (DIS), JBTI.1 (DIS), MAOJ.1 (DIS)
- net wIBEP: now also HANV.4 (~{RESET}), HAPY.4 (~{RESET}), JBTI.4 (~{RESET}), MAOJ.4 (~{RESET})
- net wLCIH: now also HANV.3 (LATCH), HAPY.3 (LATCH), JBTI.3 (LATCH), MAOJ.3 (LATCH)
- net at DMA?.2 (~{ENA}): now also DMA?.2 (~{ENA}), DMA?.2 (~{ENA}), DMA?.2 (~{ENA})
- new net 65816_A4: JBTI.2 (D)
- new net 65816_A5: MAOJ.2 (D)
- new net 65816_A6: HAPY.2 (D)
- new net DMA_A4: DMA?.1 (IN), DMA?.3 (IN)
- new net DMA_A5: DMA?.1 (IN), DMA?.3 (IN)
- new net DMA_A6: DMA?.1 (IN), DMA?.3 (IN)
Other:
- moved on the sheet: AAXI, AAZK, ABEB, ABGY, ABIV, ABNG, ABOH, ABPK, ABVA, ABWF, ABXH, ACBV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

Commit message: ADDR and DAT bus progress
Parts:
- removed AAZK1, ABEB1, ABGY1, ABIV1, ABNG1, ABOH1, ABPK1: TRI_INV_IF2, symbol Ricoh_Cells:TRI_INV_IF2
- removed ABVA1, ABWF1, ABWF3, ABXH1, ABXH2, ABXH3, ACBV1, ACBV2, ACBV3, ACGM1, ACGM2, ACGM3, ACHJ1, ACHJ2, ACHJ3, ACJG1, ACJG2, ACJG3, ACKH1, ACKH2, ACKH3, LADZ: TRI_BUF_IF0, symbol Ricoh_Cells:TRI_BUF_IF0
- removed CA0, CA1, CA10, CA11, CA12, CA13, CA14, CA15, CA2, CA27, CA28, CA29, CA3, CA30, CA31, CA8, CA9, D5, D6: IOBUF_A, symbol Ricoh_Cells:IOBUF_A
- added AAXI (x2), AAXI1 (x7), AAZK (x2), ABEB (x2), ABGY (x2), ABIV (x2), ABNG (x2), ABOH (x2), ABPK (x2), ABRB: TRI_INV_IF2, symbol Ricoh_Cells:TRI_INV_IF2
- added ABVA (x2), ABVA2 (x7), ABWF (x2), ABXH (x2), ACBV (x2), ACGM (x2), ACHJ (x2), ACJG (x2), ACKH (x2), DMA? (x20), IBPD: TRI_BUF_IF0, symbol Ricoh_Cells:TRI_BUF_IF0
- added ABWF2 (x7): TRI_BUF_IF1, symbol Ricoh_Cells:TRI_BUF_IF1
- added ACOU: TRI_INV_IF0, symbol Ricoh_Cells:TRI_INV_IF0
- added CA4 (x9), CA5, CA6, CA7, D7 (x7): IOBUF_A, symbol Ricoh_Cells:IOBUF_A
- added FBTA, FBWK, GBUI, HAQV, HARD, HAXD, IBHO, KBTC, NAUH, OCJG, OCKT, OCTS, OCWB, OCXI, ODKA, ODQZ, ODSH, ODVU, ODWA, ODWF: DR_TRI_LATCH, symbol Ricoh_Cells:DR_TRI_LATCH
- added GBTC, IBPR: INVERTER_A, symbol Ricoh_Cells:INVERTER_A
- added GBTL, LBOP: BUF, symbol Ricoh_Cells:BUF
- added IBSM, OEBY, OEFW, OEHW, OENU, OEPS, OEYB, OFQH, OFXA: D_LATCH_A2, symbol Ricoh_Cells:D_LATCH_A2
- added JBQV, JBRI: AND_2, symbol Ricoh_Cells:AND_2
- added OEFL, OEGK, OEKJ, OEOU, OEUB, OFAD, OFUH, OGBZ: D_LATCH_A, symbol Ricoh_Cells:D_LATCH_A
- added RW: IOBUF_B, symbol Ricoh_Cells:IOBUF_B
- ABWF2: value TRI_BUF_IF0 -> TRI_BUF_IF1; symbol Ricoh_Cells:TRI_BUF_IF0 -> Ricoh_Cells:TRI_BUF_IF1
Connections:
- net A0: now also DMA?.4, HAXD.5 (Q)
- net A1: now also DMA?.4, FBWK.5 (Q)
- net A15: now also AAXI.2, ABVA.4, DMA?.4, ODWA.5 (Q)
- net A16: now also ABOH.2, ACKH.4, DMA?.4, OCJG.5 (Q)
- net A17: now also ABPK.2, ABWF2.4, ACJG.4, DMA?.4, OCWB.5 (Q)
- net A18: now also ABNG.2, ABWF2.4, ACHJ.4, DMA?.4, GBUI.5 (Q)
- net A19: now also ABIV.2, ABWF2.4, ACGM.4, DMA?.4, OCTS.5 (Q)
- net A2: now also DMA?.4, FBTA.5 (Q)
- net A20: now also ABGY.2, ABWF2.4, ACBV.4, DMA?.4, ODVU.5 (Q)
- net A21: now also ABEB.2, ABWF2.4, ABXH.4, DMA?.4, ODWF.5 (Q)
- net A22: now also AAZK.2, ABWF.4, ABWF2.4, DMA?.4, ODQZ.5 (Q)
- net A23: now also AAXI.2, ABVA.4, ABWF2.4, DMA?.4, ODKA.5 (Q)
- net A3: now also DMA?.4, IBHO.5 (Q)
- net A8: now also ABOH.2, ACKH.4, DMA?.4, KBTC.5 (Q)
- net D0: now also ABVA2.4, OFXA.2 (D)
- net D1: now also ABVA2.4, OFQH.2 (D)
- net D2: now also ABVA2.4, OEYB.2 (D)
- net D3: now also ABVA2.4, OEPS.2 (D)
- net D4: now also ABVA2.4, OENU.2 (D)
- net D5: now also ABVA2.4, OEHW.2 (D)
- net D6: now also ABVA2.4, OEFW.2 (D)
- net D7: now also OEBY.2 (D); no longer AAXI1.2
- net IN_CA0: now also CA4.2 (INPUT)
- net IN_CA1: now also CA4.2 (INPUT)
- net IN_CA10: now also ACHJ.1 (IN), ACHJ.3 (IN), CA4.2 (INPUT)
- net IN_CA11: now also ACGM.1 (IN), ACGM.3 (IN), CA4.2 (INPUT)
- net IN_CA12: now also ACBV.1 (IN), ACBV.3 (IN), CA4.2 (INPUT)
- net IN_CA13: now also ABXH.1 (IN), ABXH.3 (IN), CA5.2 (INPUT)
- net IN_CA14: now also ABWF.1 (IN), ABWF.3 (IN), CA6.2 (INPUT)
- net IN_CA15: now also ABVA.1 (IN), ABVA.3 (IN), CA7.2 (INPUT)
- net IN_CA16: now also ACKH.1 (IN), ACKH.3 (IN); no longer ABWF2.1 (IN), ABWF2.3 (IN)
- net IN_CA17: now also ACJG.1 (IN), ACJG.3 (IN)
- net IN_CA18: now also ACHJ.1 (IN), ACHJ.3 (IN)
- net IN_CA19: now also ACGM.1 (IN), ACGM.3 (IN)
- net IN_CA2: now also CA4.2 (INPUT)
- net IN_CA20: now also ACBV.1 (IN), ACBV.3 (IN)
- net IN_CA21: now also ABXH.1 (IN), ABXH.3 (IN)
- net IN_CA22: now also ABWF.1 (IN), ABWF.3 (IN)
- net IN_CA23: now also ABVA.1 (IN), ABVA.3 (IN)
- net IN_CA3: now also CA4.2 (INPUT)
- net IN_CA7: no longer ABVA2.1 (IN), ABVA2.3 (IN), D7.2 (~{INPUT})
- net IN_CA8: now also ACKH.1 (IN), ACKH.3 (IN), CA4.2 (INPUT)
- net IN_CA9: now also ACJG.1 (IN), ACJG.3 (IN), CA4.2 (INPUT)
- net at CA17.1 (DRV_LOW): now also ABPK.3
- net at CA17.3 (~{DRV}_HIGH): now also ABPK.3
- net at ABPK.3: now also CA4.3 (~{DRV}_HIGH)
- net at ABIV.3: now also CA4.3 (~{DRV}_HIGH)
- net at CA21.1 (DRV_LOW): now also ABEB.3
- net at CA21.3 (~{DRV}_HIGH): now also ABEB.3
- net at CA19.1 (DRV_LOW): now also ABIV.3
- net at CA19.3 (~{DRV}_HIGH): now also ABIV.3
- net at CA22.1 (DRV_LOW): now also AAZK.3
- net at CA22.3 (~{DRV}_HIGH): now also AAZK.3
- net at ABOH.3: now also CA4.3 (~{DRV}_HIGH)
- net at ABNG.3: now also CA4.3 (~{DRV}_HIGH)
- net at DMA?.2 (~{ENA}), DMA?.2 (~{ENA}), DMA?.2 (~{ENA})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: now also DMA?.2 (~{ENA}), DMA?.2 (~{ENA}), DMA?.2 (~{ENA}), DMA?.2 (~{ENA}), DMA?.2 (~{ENA}), DMA?.2 (~{ENA}), DMA?.2 (~{ENA}), DMA?.2 (~{ENA}), DMA?.2 (~{ENA}), DMA?.2 (~{ENA}), DMA?.2 (~{ENA}), DMA?.2 (~{ENA}), DMA?.2 (~{ENA}), DMA?.2 (~{ENA}), DMA?.2 (~{ENA}), DMA?.2 (~{ENA}), DMA?.2 (~{ENA}), DMA?.2 (~{ENA}), DMA?.2 (~{ENA}), DMA?.2 (~{ENA})
- net at CA18.1 (DRV_LOW): now also ABNG.3
- net at CA18.3 (~{DRV}_HIGH): now also ABNG.3
- net at CA16.1 (DRV_LOW): now also ABOH.3
- net at CA16.3 (~{DRV}_HIGH): now also ABOH.3
- net at CA20.1 (DRV_LOW): now also ABGY.3
- net at CA20.3 (~{DRV}_HIGH): now also ABGY.3
- net at CA23.1 (DRV_LOW): now also AAXI.3
- net at CA23.3 (~{DRV}_HIGH): now also AAXI.3
- net DIR_OUT_EN renamed ~{INTERNAL_ADDR_EN}
- net ~{INTERNAL_ADDR_EN}: now also AAXI.1 (~{ENA}), AAZK.1 (~{ENA}), ABEB.1 (~{ENA}), ABGY.1 (~{ENA}), ABIV.1 (~{ENA}), ABNG.1 (~{ENA}), ABOH.1 (~{ENA}), ABPK.1 (~{ENA}), ABRB.1 (~{ENA}), JBQV.1
- net wGBTL renamed ~{EXTERNAL _ADDR_EN}
- net ~{EXTERNAL _ADDR_EN}: now also ABVA.2 (~{ENA}), ABWF.2 (~{ENA}), ABXH.2 (~{ENA}), ACBV.2 (~{ENA}), ACGM.2 (~{ENA}), ACHJ.2 (~{ENA}), ACJG.2 (~{ENA}), ACKH.2 (~{ENA}), ACOU.1 (~{ENA}), GBTL.2
- net wHAKW renamed ~{65816_ADDR_EN}
- net ~{65816_ADDR_EN}: now also FBTA.1 (DIS), FBWK.1 (DIS), GBUI.1 (DIS), HAQV.1 (DIS), HARD.1 (DIS), HAXD.1 (DIS), IBHO.1 (DIS), IBPD.2 (~{ENA}), KBTC.1 (DIS), NAUH.1 (DIS), OCJG.1 (DIS), OCKT.1 (DIS), OCTS.1 (DIS), OCWB.1 (DIS), OCXI.1 (DIS), ODKA.1 (DIS), ODQZ.1 (DIS), ODSH.1 (DIS), ODVU.1 (DIS), ODWA.1 (DIS), ODWF.1 (DIS)
- net wIBEP renamed ~{65816_ADDR_RST}
- net ~{65816_ADDR_RST}: now also FBTA.4 (~{RESET}), FBWK.4 (~{RESET}), GBUI.4 (~{RESET}), HAQV.4 (~{RESET}), HARD.4 (~{RESET}), HAXD.4 (~{RESET}), IBHO.4 (~{RESET}), KBTC.4 (~{RESET}), NAUH.4 (~{RESET}), OCJG.4 (~{RESET}), OCKT.4 (~{RESET}), OCTS.4 (~{RESET}), OCWB.4 (~{RESET}), OCXI.4 (~{RESET}), ODKA.4 (~{RESET}), ODQZ.4 (~{RESET}), ODSH.4 (~{RESET}), ODVU.4 (~{RESET}), ODWA.4 (~{RESET}), ODWF.4 (~{RESET})
- net wLCIH renamed 65816_ADDR_LATCH
- net 65816_ADDR_LATCH: now also FBTA.3 (LATCH), FBWK.3 (LATCH), GBUI.3 (LATCH), HAQV.3 (LATCH), HARD.3 (LATCH), HAXD.3 (LATCH), IBHO.3 (LATCH), IBSM.1 (~{ENA}), IBSM.3 (ENA), KBTC.3 (LATCH), NAUH.3 (LATCH), OCJG.3 (LATCH), OCKT.3 (LATCH), OCTS.3 (LATCH), OCWB.3 (LATCH), OCXI.3 (LATCH), ODKA.3 (LATCH), ODQZ.3 (LATCH), ODSH.3 (LATCH), ODVU.3 (LATCH), ODWA.3 (LATCH), ODWF.3 (LATCH)
- net wMBSK: no longer names the net of ABWF2.2 (~{ENA})
- net wMBSK: now also ABWF2.2 (~{ENA}), ABWF2.2 (~{ENA}), ABWF2.2 (~{ENA}), ABWF2.2 (~{ENA}), ABWF2.2 (~{ENA}), ABWF2.2 (~{ENA}), ABWF2.2 (~{ENA}), GBTC.2
- net wODIB renamed DATAIN_EN
- net DATAIN_EN: now also ABVA2.2 (~{ENA}), ABVA2.2 (~{ENA}), ABVA2.2 (~{ENA}), ABVA2.2 (~{ENA}), ABVA2.2 (~{ENA}), ABVA2.2 (~{ENA}), ABVA2.2 (~{ENA})
- net wODQC renamed DATAOUT_EN
- net DATAOUT_EN: now also AAXI1.1 (~{ENA}), AAXI1.1 (~{ENA}), AAXI1.1 (~{ENA}), AAXI1.1 (~{ENA}), AAXI1.1 (~{ENA}), AAXI1.1 (~{ENA}), AAXI1.1 (~{ENA})
- new net: AAXI.3, CA7.1 (DRV_LOW)
- new net: AAXI.3, CA7.3 (~{DRV}_HIGH)
- new net: ABVA2.1 (IN), ABVA2.3 (IN), OFUH.5 (~{Q})
- new net: ABIV.3, CA4.1 (DRV_LOW) (x2)
- new net: ABVA2.1 (IN), ABVA2.3 (IN), OEGK.5 (~{Q})
- new net: OFQH.1 (~{ENA}), OFQH.3 (ENA), OFUH.1 (~{ENA}), OFUH.3 (ENA)
- new net: AAXI1.2, OFQH.4 (Q)
- new net: ABOH.3, CA4.1 (DRV_LOW) (x2)
- new net: ABOH.3, CA4.3 (~{DRV}_HIGH)
- new net: ABNG.3, CA4.1 (DRV_LOW) (x2)
- new net: ABNG.3, CA4.3 (~{DRV}_HIGH)
- new net: OFXA.1 (~{ENA}), OFXA.3 (ENA), OGBZ.1 (~{ENA}), OGBZ.3 (ENA)
- new net: AAXI1.2, OFXA.4 (Q)
- new net: AAZK.3, CA6.1 (DRV_LOW)
- new net: AAZK.3, CA6.3 (~{DRV}_HIGH)
- new net: GBTC.1, IBPR.2, JBQV.2, JBRI.1
- new net: GBTL.1, JBRI.3
- new net: AAXI1.2, OEBY.4 (Q)
- new net: ABVA2.1 (IN), ABVA2.3 (IN), OGBZ.5 (~{Q})
- new net: ABVA2.1 (IN), ABVA2.3 (IN), OEKJ.5 (~{Q})
- new net: ABVA2.1 (IN), ABVA2.3 (IN), OEFL.5 (~{Q})
- new net: AAXI1.2, OEHW.4 (Q)
- new net: AAXI1.3, D7.1 (DRV_LOW) (x7)
- new net: AAXI1.3, D7.3 (~{DRV}_HIGH) (x7)
- new net: ABVA2.1 (IN), ABVA2.3 (IN), OEUB.5 (~{Q})
- new net: ABPK.3, CA4.1 (DRV_LOW) (x2)
- new net: ABEB.3, CA5.1 (DRV_LOW)
- new net: ABEB.3, CA5.3 (~{DRV}_HIGH)
- new net: ABPK.3, CA4.3 (~{DRV}_HIGH)
- new net: OEYB.1 (~{ENA}), OEYB.3 (ENA), OFAD.1 (~{ENA}), OFAD.3 (ENA)
- new net: ABVA2.1 (IN), ABVA2.3 (IN), OFAD.5 (~{Q})
- new net: AAXI1.2, OENU.4 (Q)
- new net: AAXI1.2, OEPS.4 (Q)
- new net: ABGY.3, CA4.1 (DRV_LOW)
- new net: ABGY.3, CA4.3 (~{DRV}_HIGH)
- new net: AAXI1.2, OEYB.4 (Q)
- new net: JBQV.3, LBOP.1
- new net: ABRB.3, RW.1 (DRV_LOW)
- new net: ACOU.2, RW.2 (~{INPUT})
- new net: ABRB.3, RW.4 (~{DRV}_HIGH)
- new net: OEHW.1 (~{ENA}), OEHW.3 (ENA), OEKJ.1 (~{ENA}), OEKJ.3 (ENA)
- new net: OENU.1 (~{ENA}), OENU.3 (ENA), OEOU.1 (~{ENA}), OEOU.3 (ENA)
- new net: OEPS.1 (~{ENA}), OEPS.3 (ENA), OEUB.1 (~{ENA}), OEUB.3 (ENA)
- new net: ABIV.3, CA4.3 (~{DRV}_HIGH)
- new net: ABVA2.1 (IN), ABVA2.3 (IN), OEOU.5 (~{Q})
- new net: OEFW.1 (~{ENA}), OEFW.3 (ENA), OEGK.1 (~{ENA}), OEGK.3 (ENA)
- new net: IBPD.1 (IN), IBPD.3 (IN), IBSM.4 (Q)
- new net: AAXI1.2, OEFW.4 (Q)
- new net 65816_A0: HAXD.2 (D)
- new net 65816_A1: FBWK.2 (D)
- new net 65816_A10: HARD.2 (D)
- new net 65816_A11: HAQV.2 (D)
- new net 65816_A12: NAUH.2 (D)
- new net 65816_A13: OCXI.2 (D)
- new net 65816_A14: ODSH.2 (D)
- new net 65816_A15: ODWA.2 (D)
- new net 65816_A16: OCJG.2 (D)
- new net 65816_A17: OCWB.2 (D)
- new net 65816_A18: GBUI.2 (D)
- new net 65816_A19: OCTS.2 (D)
- new net 65816_A2: FBTA.2 (D)
- new net 65816_A20: ODVU.2 (D)
- new net 65816_A21: ODWF.2 (D)
- new net 65816_A22: ODQZ.2 (D)
- new net 65816_A23: ODKA.2 (D)
- new net 65816_A3: IBHO.2 (D)
- new net 65816_A8: KBTC.2 (D)
- new net 65816_A9: OCKT.2 (D)
- new net 65816_RW: IBSM.2 (D)
- new net A10: ABNG.2, ACHJ.4, DMA?.4, HARD.5 (Q)
- new net A11: ABIV.2, ACGM.4, DMA?.4, HAQV.5 (Q)
- new net A12: ABGY.2, ACBV.4, DMA?.4, NAUH.5 (Q)
- new net A13: ABEB.2, ABXH.4, DMA?.4, OCXI.5 (Q)
- new net A14: AAZK.2, ABWF.4, DMA?.4, ODSH.5 (Q)
- new net A9: ABPK.2, ACJG.4, DMA?.4, OCKT.5 (Q)
- new net DATABUS_LATCH: OEBY.1 (~{ENA}), OEBY.3 (ENA), OEFL.1 (~{ENA}), OEFL.3 (ENA)
- new net DMA_A0: DMA?.1 (IN), DMA?.3 (IN)
- new net DMA_A1: DMA?.1 (IN), DMA?.1 (IN), DMA?.3 (IN), DMA?.3 (IN)
- new net DMA_A10: DMA?.1 (IN), DMA?.3 (IN)
- new net DMA_A11: DMA?.1 (IN), DMA?.3 (IN)
- new net DMA_A12: DMA?.1 (IN), DMA?.3 (IN)
- new net DMA_A13: DMA?.1 (IN), DMA?.3 (IN)
- new net DMA_A14: DMA?.1 (IN), DMA?.3 (IN)
- new net DMA_A15: DMA?.1 (IN), DMA?.3 (IN)
- new net DMA_A16: DMA?.1 (IN), DMA?.3 (IN)
- new net DMA_A17: DMA?.1 (IN), DMA?.3 (IN)
- new net DMA_A18: DMA?.1 (IN), DMA?.3 (IN)
- new net DMA_A19: DMA?.1 (IN), DMA?.3 (IN)
- new net DMA_A2: DMA?.1 (IN), DMA?.3 (IN)
- new net DMA_A20: DMA?.1 (IN), DMA?.3 (IN)
- new net DMA_A21: DMA?.1 (IN), DMA?.3 (IN)
- new net DMA_A22: DMA?.1 (IN), DMA?.3 (IN)
- new net DMA_A23: DMA?.1 (IN), DMA?.3 (IN)
- new net DMA_A3: DMA?.1 (IN), DMA?.3 (IN)
- new net DMA_A8: DMA?.1 (IN), DMA?.3 (IN)
- new net GND: ABWF2.1 (IN), ABWF2.1 (IN), ABWF2.1 (IN), ABWF2.1 (IN), ABWF2.1 (IN), ABWF2.1 (IN), ABWF2.1 (IN), ABWF2.1 (IN), ABWF2.3 (IN), ABWF2.3 (IN), ABWF2.3 (IN), ABWF2.3 (IN), ABWF2.3 (IN), ABWF2.3 (IN), ABWF2.3 (IN), ABWF2.3 (IN)
- new net IN_D0: D7.2 (INPUT), OGBZ.2 (D)
- new net IN_D1: D7.2 (INPUT), OFUH.2 (D)
- new net IN_D2: D7.2 (INPUT), OFAD.2 (D)
- new net IN_D3: D7.2 (INPUT), OEUB.2 (D)
- new net IN_D4: D7.2 (INPUT), OEOU.2 (D)
- new net IN_D5: D7.2 (INPUT), OEKJ.2 (D)
- new net IN_D6: D7.2 (INPUT), OEGK.2 (D)
- new net IN_D7: D7.2 (INPUT), OEFL.2 (D)
- new net MODE2_OR_MODE3: IBPR.1
- new net RW: ABRB.2, ACOU.3, IBPD.4
- new net ~{EXTERNAL_BUS_EN}: ABVA.2 (~{ENA}), ABWF.2 (~{ENA}), ABXH.2 (~{ENA}), ACBV.2 (~{ENA}), ACGM.2 (~{ENA}), ACHJ.2 (~{ENA}), ACJG.2 (~{ENA}), ACKH.2 (~{ENA}), JBRI.2
- new net ~{INTERNAL_BANK_EN}: AAXI.1 (~{ENA}), AAZK.1 (~{ENA}), ABEB.1 (~{ENA}), ABGY.1 (~{ENA}), ABIV.1 (~{ENA}), ABNG.1 (~{ENA}), ABOH.1 (~{ENA}), ABPK.1 (~{ENA}), LBOP.2
- no-connect marks 0 -> 8
Other:
- moved on the sheet: AAXI, AAXI1, AAZK, ABEB, ABGY, ABIV, ABNG, ABOH, ABPK, ABVA, ABVA2, ABWF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
