File: S-CPU_kicad/addrdatabuses.kicad_sch (KiCad schematic)
At the start: 179 parts

Commit message: Schematics update.
Parts:
- removed AAXI1 (x8): TRI_INV_IF2, symbol Ricoh_Cells:TRI_INV_IF2
- removed ABVA2 (x8), DMA? (x24): TRI_BUF_IF0, symbol Ricoh_Cells:TRI_BUF_IF0
- removed D7 (x8): IOBUF_A, symbol Ricoh_Cells:IOBUF_A
- removed OEBY, OEFW, OEHW, OENU, OEPS, OEYB, OFQH, OFXA: D_LATCH_A2, symbol Ricoh_Cells:D_LATCH_A2
- removed OEFL, OEGK, OEKJ, OEOU, OEUB, OFAD, OFUH, OGBZ: D_LATCH_A, symbol Ricoh_Cells:D_LATCH_A
- added OKMN0, OKMN1, OKMN2, OKMN3, OKTR0, OKTR1, OKTR2, OKTR3, OKTY0, OKTY1, OKTY2, OKTY3, OLDU0, OLDU1, OLDU2, OLDU3, OMIG0, OMIG1, OMIG2, OMIG3, OMNC0, OMNC1, OMNC2, OMNC3, QKEL0, QKEL1, QKEL2, QKEL3, QKQM0, QKQM1, QKQM2, QKQM3, RKOE0, RKOE1, RKOE2, RKOE3, RKUL0, RKUL1, RKUL2, RKUL3: TRI_BUF_IF1, symbol Ricoh_Cells:TRI_BUF_IF1
- added OKPW, OKSL, OKUR, OLCW, OMDX, OMMV, QKGG, QKLR, RKPQ, RKPR, RKRK: INVERTER_A, symbol Ricoh_Cells:INVERTER_A
- added QKHU, RKQY: NAND_3, symbol Ricoh_Cells:NAND_3
Connections:
- net A0: now also OKTR3.4, QKQM0.1 (IN), QKQM0.3 (IN)
- net A1: now also OKTR2.4, QKQM1.1 (IN), QKQM1.3 (IN)
- net A10: now also OMNC1.4
- net A11: now also OMNC0.4
- net A12: now also OMIG3.4
- net A13: now also OMIG2.4
- net A14: now also OMIG1.4
- net A15: now also OMIG0.4
- net A16: now also OKTY3.4
- net A17: now also OKTY2.4
- net A18: now also OKTY1.4
- net A19: now also OKTY0.4
- net A2: now also OKTR1.4, QKQM2.1 (IN), QKQM2.3 (IN)
- net A20: now also OLDU3.4
- net A21: now also OLDU2.4
- net A22: now also OLDU1.4
- net A23: now also OLDU0.4
- net A3: now also OKTR0.4, QKQM3.1 (IN), QKQM3.3 (IN)
- net A4: now also OKMN3.4, QKEL0.1 (IN), QKEL0.3 (IN)
- net A5: now also OKMN2.4, QKEL1.1 (IN), QKEL1.3 (IN)
- net A6: now also OKMN1.4, QKEL2.1 (IN), QKEL2.3 (IN)
- net A7: now also OKMN0.4, QKEL3.1 (IN), QKEL3.3 (IN)
- net A8: now also OMNC3.4
- net A9: now also OMNC2.4
- net DMA_A0: now also OKTR3.1 (IN), OKTR3.3 (IN)
- net DMA_A1: now also OKTR2.1 (IN), OKTR2.3 (IN), OMNC2.1 (IN), OMNC2.3 (IN)
- net DMA_A10: now also OMNC1.1 (IN), OMNC1.3 (IN)
- net DMA_A11: now also OMNC0.1 (IN), OMNC0.3 (IN)
- net DMA_A12: now also OMIG3.1 (IN), OMIG3.3 (IN)
- net DMA_A13: now also OMIG2.1 (IN), OMIG2.3 (IN)
- net DMA_A14: now also OMIG1.1 (IN), OMIG1.3 (IN)
- net DMA_A15: now also OMIG0.1 (IN), OMIG0.3 (IN)
- net DMA_A16: now also OKTY3.1 (IN), OKTY3.3 (IN)
- net DMA_A17: now also OKTY2.1 (IN), OKTY2.3 (IN)
- net DMA_A18: now also OKTY1.1 (IN), OKTY1.3 (IN)
- net DMA_A19: now also OKTY0.1 (IN), OKTY0.3 (IN)
- net DMA_A2: now also OKTR1.1 (IN), OKTR1.3 (IN)
- net DMA_A20: now also OLDU3.1 (IN), OLDU3.3 (IN)
- net DMA_A21: now also OLDU2.1 (IN), OLDU2.3 (IN)
- net DMA_A22: now also OLDU1.1 (IN), OLDU1.3 (IN)
- net DMA_A23: now also OLDU0.1 (IN), OLDU0.3 (IN)
- net DMA_A3: now also OKTR0.1 (IN), OKTR0.3 (IN)
- net DMA_A4: now also OKMN3.1 (IN), OKMN3.3 (IN)
- net DMA_A5: now also OKMN2.1 (IN), OKMN2.3 (IN)
- net DMA_A6: now also OKMN1.1 (IN), OKMN1.3 (IN)
- net DMA_A7: now also OKMN0.1 (IN), OKMN0.3 (IN)
- net DMA_A8: now also OMNC3.1 (IN), OMNC3.3 (IN)
- new net: OMMV.2, OMNC0.2 (~{ENA}), OMNC1.2 (~{ENA}), OMNC2.2 (~{ENA}), OMNC3.2 (~{ENA})
- new net: OMDX.2, OMIG0.2 (~{ENA}), OMIG1.2 (~{ENA}), OMIG2.2 (~{ENA}), OMIG3.2 (~{ENA})
- new net: OKSL.2, OKTR0.2 (~{ENA}), OKTR1.2 (~{ENA}), OKTR2.2 (~{ENA}), OKTR3.2 (~{ENA})
- new net: OKMN0.2 (~{ENA}), OKMN1.2 (~{ENA}), OKMN2.2 (~{ENA}), OKMN3.2 (~{ENA}), OKPW.2
- new net: RKRK.2, RKUL0.2 (~{ENA}), RKUL1.2 (~{ENA}), RKUL2.2 (~{ENA}), RKUL3.2 (~{ENA})
- new net: QKLR.2, QKQM0.2 (~{ENA}), QKQM1.2 (~{ENA}), QKQM2.2 (~{ENA}), QKQM3.2 (~{ENA})
- new net: QKEL0.2 (~{ENA}), QKEL1.2 (~{ENA}), QKEL2.2 (~{ENA}), QKEL3.2 (~{ENA}), QKGG.2
- new net: OLCW.2, OLDU0.2 (~{ENA}), OLDU1.2 (~{ENA}), OLDU2.2 (~{ENA}), OLDU3.2 (~{ENA})
- new net: OKTY0.2 (~{ENA}), OKTY1.2 (~{ENA}), OKTY2.2 (~{ENA}), OKTY3.2 (~{ENA}), OKUR.2
- new net: RKPR.2, RKQY.1
- new net: RKPQ.1, RKQY.4, RKRK.1
- new net: QKGG.1, QKHU.4, QKLR.1
- new net: RKOE0.2 (~{ENA}), RKOE1.2 (~{ENA}), RKOE2.2 (~{ENA}), RKOE3.2 (~{ENA}), RKPQ.2
- new net DMA_PA0: RKOE0.1 (IN), RKOE0.3 (IN)
- new net DMA_PA1: RKOE1.1 (IN), RKOE1.3 (IN)
- new net DMA_PA2: RKOE2.1 (IN), RKOE2.3 (IN)
- new net DMA_PA3: RKOE3.1 (IN), RKOE3.3 (IN)
- new net DMA_PA4: RKUL0.1 (IN), RKUL0.3 (IN)
- new net DMA_PA5: RKUL1.1 (IN), RKUL1.3 (IN)
- new net DMA_PA6: RKUL2.1 (IN), RKUL2.3 (IN)
- new net DMA_PA7: RKUL3.1 (IN), RKUL3.3 (IN)
- new net PA0: QKQM0.4, RKOE0.4
- new net PA1: QKQM1.4, RKOE1.4
- new net PA2: QKQM2.4, RKOE2.4
- new net PA3: QKQM3.4, RKOE3.4
- new net PA4: QKEL0.4, RKUL0.4
- new net PA5: QKEL1.4, RKUL1.4
- new net PA6: QKEL2.4, RKUL2.4
- new net PA7: QKEL3.4, RKUL3.4
- new net ~{DMA_BUS_EN}: OKPW.1, OKSL.1, OKUR.1, OLCW.1, OMDX.1, OMMV.1, QKHU.1, RKPR.1
- new net ~{MODE5}: QKHU.3, RKQY.3
- new net ~{MODE6}: QKHU.2, RKQY.2
- no-connect marks 8 -> 0
Other:
- note added: "A-BUS"
- note added: "B-BUS"
- note added: "B_BUS Address coming from DMA banks during DMA or from A bus otherwise"
- company: Regis Galland -> Author: Regis Galland
