File: S-CPU_kicad/productremainder.kicad_sch (KiCad schematic)
At the start: 178 parts

Commit message: ADDR and DAT bus progress
Other:
- company: (none) -> Regis Galland
- title: (none) -> SNES S-CPU Schematics 
Changed lines of the file:
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@@
 (kicad_sch (version 20230121) (generator eeschema)
   (paper "A1")
+  (title_block
+    (title "SNES S-CPU Schematics ")
+    (date "2023-06-14")
+    (rev "0.1")
+    (company "Regis Galland")
+  )
   (junction (at 514.35 306.705) (diameter 0) (color 0 0 0 0)
   )
