File: S-CPU_kicad/productremainder.kicad_sch (KiCad schematic)
At the start: 178 parts

Commit message: Progress in DMA section. Fixed some DFF output issues.
Connections:
- net at ABWF1.1 (IN), ABWF1.3 (IN), LFHO.23 (B1): now also KBGM.6 (~{Q}); no longer KBGM.7 (Q)
- net at KBGM.6 (~{Q}): now also ACBV1.1 (IN), ACBV1.3 (IN), LFFC.23 (B1)
- net at KHRF.2, KHXL.1, QABF.3 (2): now also KBGM.6 (~{Q}); no longer KBGM.7 (Q)
- net at ACBV1.1 (IN), ACBV1.3 (IN), LFQZ.23 (B1): now also KBGM.6 (~{Q}); no longer KBGM.7 (Q)
- net at HFSC.1: now also KBGM.7 (Q); no longer KBGM.6 (~{Q})
- net at HFSC.2: now also KBGM.7 (Q); no longer KBGM.6 (~{Q})
- net at JFHM.1, JFLO.2: now also KBGM.6 (~{Q}); no longer KBGM.7 (Q)
- net at JFCT.1, JFHM.2: now also KBGM.6 (~{Q}); no longer KBGM.7 (Q)
- net at HGDM.2: now also KBGM.7 (Q); no longer KBGM.6 (~{Q})
- net at ABVA1.1 (IN), ABVA1.3 (IN), LFUD.9 (B0): now also KBGM.6 (~{Q}); no longer KBGM.7 (Q)
- net at KFOX.2, KFZV.1, QABF.3 (2): now also KBGM.6 (~{Q}); no longer KBGM.7 (Q)
- net at KBGM.6 (~{Q}): now also KGZD.2, KHRF.1, QABF.3 (2)
- net at KFMZ.2, KFYB.1, QABF.3 (2): now also KBGM.6 (~{Q}); no longer KBGM.7 (Q)
- net at ACHJ1.1 (IN), ACHJ1.3 (IN), LFQZ.9 (B0): now also KBGM.6 (~{Q}); no longer KBGM.7 (Q)
- net at JFCT.2, KFMZ.1, QABF.3 (2): now also KBGM.6 (~{Q}); no longer KBGM.7 (Q)
- net at KHAD.2, KHSS.1, QABF.3 (2): now also KBGM.6 (~{Q}); no longer KBGM.7 (Q)
- net at KHSS.2, KHYE.1, QABF.3 (2): now also KBGM.6 (~{Q}); no longer KBGM.7 (Q)
- net at KBGM.6 (~{Q}): now also ABWF1.1 (IN), ABWF1.3 (IN), LFUD.23 (B1)
- net at ACHJ1.1 (IN), ACHJ1.3 (IN), LFFC.9 (B0): now also KBGM.6 (~{Q}); no longer KBGM.7 (Q)
- net at KBGM.6 (~{Q}): now also ABXH1.1 (IN), ABXH1.3 (IN), LFFN.23 (B1)
- net at JFQD.1, JFRP.2: now also KBGM.6 (~{Q}); no longer KBGM.7 (Q)
- net at ACJG1.1 (IN), ACJG1.3 (IN), LFDU.9 (B0): now also KBGM.6 (~{Q}); no longer KBGM.7 (Q)
- net at ACJG1.1 (IN), ACJG1.3 (IN), LFNW.9 (B0): now also KBGM.6 (~{Q}); no longer KBGM.7 (Q)
- net at KBGM.6 (~{Q}): now also KFCQ.2, KFOX.1, QABF.3 (2)
- net at KGGW.2, KGZD.1, QABF.3 (2): now also KBGM.6 (~{Q}); no longer KBGM.7 (Q)
- net at KBGM.6 (~{Q}): now also ACGM1.1 (IN), ACGM1.3 (IN), LFDU.23 (B1)
- net at KGHB.2, KHAD.1, QABF.3 (2): now also KBGM.6 (~{Q}); no longer KBGM.7 (Q)
- net at HFJQ.1: now also KBGM.7 (Q); no longer KBGM.6 (~{Q})
- net at KFYB.2, KGGW.1, QABF.3 (2): now also KBGM.6 (~{Q}); no longer KBGM.7 (Q)
- net at KBGM.6 (~{Q}): now also KHXL.2, KICH.1, QABF.3 (2)
- net at KFZV.2, KGHB.1, QABF.3 (2): now also KBGM.6 (~{Q}); no longer KBGM.7 (Q)
- net at ACKH1.1 (IN), ACKH1.3 (IN), LFRR.9 (B0): now also KBGM.6 (~{Q}); no longer KBGM.7 (Q)
- net at KICH.2, QABF.3 (2): now also KBGM.6 (~{Q}); no longer KBGM.7 (Q)
- net at JFDF.1, JFKA.2: now also KBGM.6 (~{Q}); no longer KBGM.7 (Q)
- net at JFDF.2, KFCQ.1, QABF.3 (2): now also KBGM.6 (~{Q}); no longer KBGM.7 (Q)
- net at KHYE.2, KIDU.1, QABF.3 (2): now also KBGM.6 (~{Q}); no longer KBGM.7 (Q)
- net at ACGM1.1 (IN), ACGM1.3 (IN), LFNW.23 (B1): now also KBGM.6 (~{Q}); no longer KBGM.7 (Q)
- net at ABXH1.1 (IN), ABXH1.3 (IN), LFRR.23 (B1): now also KBGM.6 (~{Q}); no longer KBGM.7 (Q)
- net at ABVA1.1 (IN), ABVA1.3 (IN), LFHO.9 (B0): now also KBGM.6 (~{Q}); no longer KBGM.7 (Q)
- net at ACKH1.1 (IN), ACKH1.3 (IN), LFFN.9 (B0): now also KBGM.6 (~{Q}); no longer KBGM.7 (Q)
- net at HFJQ.2: now also KBGM.7 (Q); no longer KBGM.6 (~{Q})
- net at JFKA.1, JFQD.2: now also KBGM.6 (~{Q}); no longer KBGM.7 (Q)
- net at JFRL.1: now also KBGM.6 (~{Q}); no longer KBGM.7 (Q)
- net at JFLO.1, JFRL.2: now also KBGM.6 (~{Q}); no longer KBGM.7 (Q)
- net at HGFS.1: now also KBGM.7 (Q); no longer KBGM.6 (~{Q})
- net at HGFS.2: now also KBGM.7 (Q); no longer KBGM.6 (~{Q})
- now unconnected: KBGM.7 (Q), KBGM.7 (Q), KBGM.7 (Q), KBGM.7 (Q), KBGM.7 (Q), KBGM.7 (Q), KBGM.7 (Q)
Other:
- moved on the sheet: ABVA1, ABWF1, ABXH1, ACBV1, ACGM1, ACHJ1, ACJG1, ACKH1, HFJQ, HFPC, HFSC, HFYF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

Commit message: Schematics update.
Other:
- company: Regis Galland -> Author: Regis Galland
Changed lines of the file:
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@@
     (date "2023-06-14")
     (rev "0.1")
-    (company "Regis Galland")
+    (company "Author: Regis Galland")
   )
   (junction (at 514.35 306.705) (diameter 0) (color 0 0 0 0)
