File: S-CPU_kicad/dma.kicad_sch (KiCad schematic)
At the start: 295 parts, among them U1 NOR_2, U10 NAND_2, U11 INVERTER_A, U12 INVERTER_A, U13 INVERTER_A, U14 INVERTER_A, U15 NOR_2, U16 DFFR_B, U17 OR_2, U18 NAND_2, U19 DFFR_B, U2 NAND_2, U20 DFFR_B, U21 DFFR_B, U22 INVERTER_A, U23 NAND_2, U24 INVERTER_A, U25 INVERTER_A, U3 NAND_2, U4 NAND_2, U5 NAND_2, U9 NAND_2

Commit message: More updates in DMA section.
Parts:
- removed PORZ: INVERTER_A, symbol Ricoh_Cells:INVERTER_A
- removed POSD: AND_2, symbol Ricoh_Cells:AND_2
Connections:
- net wOAFI_wOACU_XIN/4 is gone; now on net wOBXZ_wOCHV_XIN/2: ULGF.1
- net wPOSD: now reaches SKCM.1, TKAT.2
- net wNBBM_wNAQE_XIN/2 renamed wNAQE_wNBBM_XIN/2
- net wNBEG_wNBEB_XIN/8 renamed wNBEB_wNBEG_XIN/8
Other:
- moved on the sheet: ULGF
Changed lines of the file:
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@@
     (stroke (width 0) (type default))
   )
+  (wire (pts (xy 488.95 146.05) (xy 496.57 146.05))
+    (stroke (width 0) (type default))
+  )
   (wire (pts (xy 421.64 542.925) (xy 424.18 542.925))
     (stroke (width 0) (type default))
@@
     (stroke (width 0) (type default))
   )
-  (wire (pts (xy 468.63 168.91) (xy 463.55 168.91))
-    (stroke (width 0) (type default))
-  )
   (bus (pts (xy 734.695 212.09) (xy 754.38 212.09))
     (stroke (width 0) (type default))
@@
     (stroke (width 0) (type default))
   )
-  (wire (pts (xy 132.715 464.82) (xy 107.95 464.82))
-    (stroke (width 0) (type default))
-  )
   (wire (pts (xy 295.275 502.92) (xy 276.225 502.92))
     (stroke (width 0) (type default))
@@
     (stroke (width 0) (type default))
   )
-  (wire (pts (xy 463.55 168.91) (xy 463.55 198.12))
-    (stroke (width 0) (type default))
-  )
   (wire (pts (xy 585.47 -19.685) (xy 588.01 -19.685))
     (stroke (width 0) (type default))
@@
     (stroke (width 0) (type default))
   )
+  (wire (pts (xy 107.95 464.82) (xy 132.08 464.82))
+    (stroke (width 0) (type default))
+  )
   (wire (pts (xy 178.435 354.33) (xy 203.835 354.33))
     (stroke (width 0) (type default))
@@
     (stroke (width 0) (type default))
   )
-  (wire (pts (xy 496.57 135.89) (xy 496.57 171.45))
+  (wire (pts (xy 496.57 135.89) (xy 496.57 146.05))
     (stroke (width 0) (type default))
   )
@@
     (stroke (width 0) (type default))
   )
-  (wire (pts (xy 453.39 198.12) (xy 463.55 198.12))
-    (stroke (width 0) (type default))
-  )
   (wire (pts (xy 661.67 81.28) (xy 659.13 81.28))
     (stroke (width 0) (type default))
@@
     (stroke (width 0) (type default))
   )
-  (wire (pts (xy 153.035 467.36) (xy 147.955 467.36))
+  (wire (pts (xy 153.035 467.36) (xy 147.32 467.36))
     (stroke (width 0) (type default))
   )
@@
     (effects (font (size 1.27 1.27)) (justify left bottom))
   )
-  (label "wOAFI_wOACU_XIN{slash}4" (at 107.95 464.82 0) (fields_autoplaced)
-    (effects (font (size 1.27 1.27)) (justify left bottom))
-  )
   (label "A6" (at 775.97 83.82 0) (fields_autoplaced)
     (effects (font (size 1.27 1.27)) (justify left bottom))
@@
     (effects (font (size 1.27 1.27)) (justify left bottom))
   )
+  (label "wOBXZ_wOCHV_XIN{slash}2" (at 107.95 464.82 0) (fields_autoplaced)
+    (effects (font (size 1.27 1.27)) (justify left bottom))
+  )
   (label "PA4" (at 808.99 119.38 180) (fields_autoplaced)
     (effects (font (size 1.27 1.27)) (justify right bottom))
@@
     (effects (font (size 1.27 1.27)) (justify right))
   )
-  (hierarchical_label "wOAFI_wOACU_XIN{slash}4" (shape input) (at 107.95 464.82 180) (fields_autoplaced)
-    (effects (font (size 1.27 1.27)) (justify right))
-  )
   (hierarchical_label "DMA_OFF" (shape input) (at 34.29 38.1 180) (fields_autoplaced)
     (effects (font (size 1.27 1.27)) (justify right))
@@
     (effects (font (size 1.27 1.27)) (justify right))
   )
-  (hierarchical_label "wNBBM_wNAQE_XIN{slash}2" (shape input) (at 558.8 52.07 180) (fields_autoplaced)
+  (hierarchical_label "wNAQE_wNBBM_XIN{slash}2" (shape input) (at 558.8 52.07 180) (fields_autoplaced)
     (effects (font (size 1.27 1.27)) (justify right))
   )
-  (hierarchical_label "wNBEG_wNBEB_XIN{slash}8" (shape input) (at 515.62 107.95 180) (fields_autoplaced)
+  (hierarchical_label "wNBEB_wNBEG_XIN{slash}8" (shape input) (at 515.62 107.95 180) (fields_autoplaced)
+    (effects (font (size 1.27 1.27)) (justify right))
+  )
+  (hierarchical_label "wPOSD" (shape input) (at 488.95 146.05 180) (fields_autoplaced)
     (effects (font (size 1.27 1.27)) (justify right))
   )
@@
     )
   )
-  (symbol (lib_id "Ricoh_Cells:INVERTER_A") (at 474.98 168.91 0) (unit 1)
-    (in_bom yes) (on_board yes) (dnp no) (fields_autoplaced)
-    (property "Reference" "PORZ" (at 474.98 160.9557 0)
-      (effects (font (size 1.27 1.27)))
-    )
-    (property "Value" "INVERTER_A" (at 474.98 163.3799 0)
-      (effects (font (size 1.27 1.27)))
-    )
-    (property "Footprint" "" (at 472.44 168.91 0)
-      (effects (font (size 1.27 1.27)) hide)
-    )
-    (property "Datasheet" "http://iceboy.a-singer.de/doc/dmg_cells.html#inv_a" (at 476.25 176.53 0)
-      (effects (font (size 1.27 1.27)) hide)
-    )
-    (pin "1")
-    (pin "2")
-    (instances
-      (project "S-CPU"
-        (path "/ca9d3ca9-0297-4b98-a109-b7c162ccc5c3/6ab7ea20-bfb3-4f18-94ca-a294126fa0fb"
-          (reference "PORZ") (unit 1)
-        )
-      )
-    )
-  )
   (symbol (lib_id "Ricoh_Cells:TRI_BUF_IF1") (at 611.505 401.32 0) (unit 1)
     (in_bom yes) (on_board yes) (dnp no) (fields_autoplaced)
@@
     )
   )
-  (symbol (lib_id "Ricoh_Cells:OR_2") (at 140.335 467.36 0) (unit 1)
+  (symbol (lib_id "Ricoh_Cells:OR_2") (at 139.7 467.36 0) (unit 1)
     (in_bom yes) (on_board yes) (dnp no)
-    (property "Reference" "ULGF" (at 140.335 460.375 0)
+    (property "Reference" "ULGF" (at 139.7 460.375 0)
       (effects (font (size 1.27 1.27)))
     )
-    (property "Value" "OR_2" (at 140.335 462.28 0)
+    (property "Value" "OR_2" (at 139.7 462.28 0)
       (effects (font (size 1.27 1.27)))
     )
-    (property "Footprint" "" (at 140.081 467.36 0)
+    (property "Footprint" "" (at 139.446 467.36 0)
       (effects (font (size 1.27 1.27)) hide)
     )
-    (property "Datasheet" "http://iceboy.a-singer.de/doc/dmg_cells.html#or2" (at 140.335 474.98 0)
+    (property "Datasheet" "http://iceboy.a-singer.de/doc/dmg_cells.html#or2" (at 139.7 474.98 0)
       (effects (font (size 1.27 1.27)) hide)
     )
@@
         )
       )
-    )
-  )
-  (symbol (lib_id "Ricoh_Cells:AND_2") (at 488.95 171.45 0) (unit 1)
-    (in_bom yes) (on_board yes) (dnp no) (fields_autoplaced)
-    (property "Reference" "POSD" (at 488.9362 163.4957 0)
-      (effects (font (size 1.27 1.27)))
-    )
-    (property "Value" "AND_2" (at 488.9362 165.9199 0)
-      (effects (font (size 1.27 1.27)))
-    )
-    (property "Footprint" "" (at 488.95 171.45 0)
-      (effects (font (size 1.27 1.27)) hide)
-    )
-    (property "Datasheet" "http://iceboy.a-singer.de/doc/dmg_cells.html#and2" (at 488.95 179.07 0)
-      (effects (font (size 1.27 1.27)) hide)
-    )
-    (pin "1")
-    (pin "2")
-    (pin "3")
-    (instances
-      (project "S-CPU"
-        (path "/ca9d3ca9-0297-4b98-a109-b7c162ccc5c3/6ab7ea20-bfb3-4f18-94ca-a294126fa0fb"
-          (reference "POSD") (unit 1)
-        )
-      )

Commit message: Another latch with reset identified. TCKSEL demux cell worked out + notes added to schematics.
Parts:
- added YKDO: INVERTER_A, symbol Ricoh_Cells:INVERTER_A
- renumbered XKQM to YKQM
Connections:
- net A4: now also ZKBA.16; no longer ZKBA.15
- net A5: now also ZKBA.24; no longer ZKBA.25
- net A6: now also ZKBW.4; no longer ZKBW.5
- net at BNVB.5: now also ZKBA.4; no longer ZKBA.5
- net at XKIG.1 (SEL), YKAW.1 (SEL), YKBC.1 (SEL)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: no longer VKBO.1 (SEL0), VKCI.1 (SEL0), XKBP.1 (SEL0), XKDB.1 (SEL0)
- net at YKQD.2: now also YKDO.1
- net at U25.2: now also ZKBA.15; no longer ZKBA.16
- net at U24.2: now also ZKBA.25; no longer ZKBA.24
- net at ZKBA.11: now also BNYC.5
- net at ZKBA.13: no longer BNYC.5
- net at U22.2: now also ZKBW.5; no longer ZKBW.4
- net from_NAND: now reaches YKOE.1
- net wOBXZ_wOCHV_XIN/2 renamed wOBXZ_wOCHV_~{XIN/2}
- new net: VKBO.1 (SEL0), VKCI.1 (SEL0), XKBP.1 (SEL0), XKDB.1 (SEL0), YKDO.2
Other:
- note added: "When DMA is OFF: - Data bus is connected directly to the DMA RAM bank inputs. - DMA RAM addresses come from the CPU A-Bus (with some decoing applied) When DMA is ON: - Data comes from multiplexers holding updated information for addesses and counters - DMA RAM Addresses are based on current DMA channel being executed including configuration register"
- moved on the sheet: U22, U24, U25, VKBOC, VKCIC, WKSNE, WKZCE, XKBPC, XKDBC, XKIGE, YKAWE, YKBCE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
