File: S-CPU_kicad/dma.kicad_sch (KiCad schematic)
At the start: 294 parts, among them U1 NOR_2, U10 NAND_2, U11 INVERTER_A, U12 INVERTER_A, U13 INVERTER_A, U14 INVERTER_A, U15 NOR_2, U16 DFFR_B, U17 OR_2, U18 NAND_2, U19 DFFR_B, U2 NAND_2, U20 DFFR_B, U21 DFFR_B, U22 INVERTER_A, U23 NAND_2, U24 INVERTER_A, U25 INVERTER_A, U3 NAND_2, U4 NAND_2, U5 NAND_2, U9 NAND_2

Commit message: Almost all cells captured in schematicAlmost all cells captured in schematics. Enter the commit message for your changes. Lines starting
Parts:
- removed LFUD1: 2BIT_FULL_ADD, symbol Ricoh_Cells:2BIT_FULL_ADD
- removed POSI, QKAG7, QKAG9, U16, U19, U20, U21: DFFR_B, symbol Ricoh_Cells:DFFR_B
- removed RKMU, SKDK?, U11, U12, U13, U14: INVERTER_A, symbol Ricoh_Cells:INVERTER_A
- removed RKUL4: TRI_BUF_IF1, symbol Ricoh_Cells:TRI_BUF_IF1
- removed TKIB? (x2): AND_2, symbol Ricoh_Cells:AND_2
- removed U1, U15: NOR_2, symbol Ricoh_Cells:NOR_2
- removed U10, U18, U2, U23, U3, U4, U5, U9: NAND_2, symbol Ricoh_Cells:NAND_2
- removed U17: OR_2, symbol Ricoh_Cells:OR_2
- added DSAC: AND_2, symbol Ricoh_Cells:AND_2
- added DSAZ, DSSG, DSSX: NAND_3, symbol Ricoh_Cells:NAND_3
- added DSCS, DSXY, DSYT, DSZC: NAND_2, symbol Ricoh_Cells:NAND_2
- added DSKP: NAND_4, symbol Ricoh_Cells:NAND_4
- added DSLL, DSWN: INVERTER_A, symbol Ricoh_Cells:INVERTER_A
- added ZOOJ: DFFR_B, symbol Ricoh_Cells:DFFR_B
Connections:
- net wQKBI: now also DSLL.1; no longer VKBO.20 (SEL1), VKCI.20 (SEL1), XKBP.20 (SEL1), XKDB.20 (SEL1)
- net wRKNG: now also DSAC.1, DSAZ.1, DSSX.2
- net wSKDA: now also DSAZ.2, DSWN.1, DSZC.2
- net ~{INC}_DEC: now also UKZF.13 (A0), UKZF.24 (A1), ULBK.13 (A0), ULBK.24 (A1), VKID.13 (A0), VKID.24 (A1), VKJK.13 (A0), VKJK.24 (A1)
- net wVOLG: now reaches OMBB.1, QKAI.1, QKAT.1
- net DMA_ON: now reaches EBSG.3 (CLK), EBSG.4 (~{CLK}), EBVQ.3 (CLK), EBVQ.4 (~{CLK}), EBXE.3 (CLK), EBXE.4 (~{CLK}), EBYP.3 (CLK), EBYP.4 (~{CLK}), ECCU.3 (CLK), ECCU.4 (~{CLK}), ECEK.3 (CLK), ECEK.4 (~{CLK}), ECGN.3 (CLK), ECGN.4 (~{CLK}), ECGO.3 (CLK), ECGO.4 (~{CLK})
- net wXKGY: now reaches XKGY.2
- net wUKYL: now reaches UKYL.6 (Q), XKDB.11
- net wDSAC: now reaches TKFI.24 (A1)
- net wDSAC: now also DSAC.3
- net at QKAG6.4 (Q): now also ZOOJ.2 (D)
- net wXKGP: now reaches XKGP.4
- net at WKSN.1 (SEL), WKZC.1 (SEL), YKMY.2: now also VKBO.20 (SEL1), VKCI.20 (SEL1), XKBP.20 (SEL1), XKDB.20 (SEL1)
- net wXOWO: now reaches ULGF.2
- net wXOWO: now also ZOOJ.3 (CLK), ZOOJ.4 (~{CLK})
- net wQKAG4: now reaches QKAG4.4 (Q), TKAT.3
- net wSKDK: now reaches SKDK.2
- net wDSYT: now reaches TKFI.13 (A0)
- net wDSYT: now also DSYT.3
- net wWOCA: now reaches ZKBW.13
- net wXOAO: now reaches ZKBW.25
- net wCSDS: now reaches YKNB.1
- net from_NAND renamed wCSGZ
- new net: DSSG.1, DSSX.1, DSWN.2, DSXY.1
- new net: DSCS.3, DSKP.1
- new net: DSAZ.4, DSKP.2
- new net: DSKP.3, DSSG.4
- new net: DSKP.4, DSSX.4
- new net: DSYT.1, DSZC.3
- new net: DSXY.3, DSYT.2
- new net: DSLL.2, DSSG.3, DSSX.3
- new net: ZOOJ.1 (~{RESET}), ZOOJ.5 (~{RESET})
- new net wDSKP: DSKP.5
- new net wWOVT: DSAZ.3, DSCS.1, DSSG.2, DSXY.2
- new net wWOWE: DSAC.2, DSCS.2, DSZC.1
- new net ~{ZOOJ}: ZOOJ.6 (~{Q})
- no-connect marks 22 -> 24
Other:
- sheet Other DMA gates ports: added CMYW_EN, DMA_CLK?, DMA_FALLING_VBLANK, DMA_OFF, DMA_ON, DMA_RISING_HBLANK, FALLING_VBLANK, INTERNAL_SYSCLK, JPO0, JPO1, JPO2, MODE4_OR_MODE5, VBLANK, wBSEK, wCSDS, wCSGZ, wDBJW_wHASI_RST, wDCBP_NOHDMA_2, wDSKP, wMAGR_wMAGV, wNAGK_wNAJD, wNAQE_wNBBM_XIN/2, wNBEB_wNBEG_XIN/8, wNBKW_wNBPG_~{XIN/4}, wOACU_wOAFI_XIN/4, wOBXZ_wOCHV_~{XIN/2}, wOCRQ_wOCRS_XIN/8, wOORF, wPOSD, wPOSI, wQKAG5, wSKDK, wSODM, wSODT, wSOGE, wTOAY, wUKYL, wUOGG, wVOLG, wWOCA, wWOIX, wWOVT, wWOWE, wXKGP, wXKGY, wXOAO, wXOWO, ~{MODE0_OR_MODE6}, ~{NO_DMA}, ~{NO_HDMA2}, ~{NO_HDMA}, ~{wRDY}; removed none
- note added: "DMA RW signal based on bus direction"
- note added: "DMA_ADDR15-0 /= 0"
- note added: "DMA_ADDR6-0 = 0"
- moved on the sheet: SKDK, TKDG, WKCF, WKNO, WKSNE, WKZCE, XKGP, XKGY, XKIN, XKKB, XKKC, XKKE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

Commit message: Progress in DMA section. Fixed some DFF output issues.
Parts:
- QKBI, RKNG, SKDA: value DFFR_A -> DFFR_B; symbol Ricoh_Cells:DFFR_A -> Ricoh_Cells:DFFR_B
Connections:
- net DMA_BANK1_D0 is gone; now on net DMA_BANK1_DOUT0: QKAG0.2 (D)
- net DMA_BANK1_D1 is gone; now on net DMA_BANK1_DOUT1: QKAG1.2 (D)
- net DMA_BANK1_D2 is gone; now on net DMA_BANK1_DOUT2: QKAG2.2 (D)
- net DMA_BANK1_D3 is gone; now on net DMA_BANK1_DOUT3: QKAG3.2 (D)
- net DMA_BANK1_D4 is gone; now on net DMA_BANK1_DOUT4: QKAG4.2 (D)
- net DMA_BANK1_D6 is gone; now on net DMA_BANK1_DOUT6: QKAG5.2 (D)
- net DMA_BANK1_D7 is gone; now on net DMA_BANK1_DOUT7: QKAG6.2 (D)
- net DMA_BANK2_D0 is gone; now on net DMA_BANK2_DOUT0: OMDK0.2 (D)
- net DMA_BANK2_D1 is gone; now on net DMA_BANK2_DOUT1: OMDK1.2 (D)
- net DMA_BANK2_D2 is gone; now on net DMA_BANK2_DOUT2: OMDK2.2 (D)
- net DMA_BANK2_D3 is gone; now on net DMA_BANK2_DOUT3: OMDK3.2 (D)
- net DMA_BANK2_D4 is gone; now on net DMA_BANK2_DOUT4: OMDK4.2 (D)
- net DMA_BANK2_D5 is gone; now on net DMA_BANK2_DOUT5: OMDK5.2 (D)
- net DMA_BANK2_D6 is gone; now on net DMA_BANK2_DOUT6: OMDK6.2 (D)
- net DMA_BANK2_D7 is gone; now on net DMA_BANK2_DOUT7: OMDK7.2 (D)
- net DMA_CLK? is gone; now on net DMA_OFF: UKBI.1
- net DMARAM_A1: no longer DMA_RAM_BANK1.~ (A4)
- net DMARAM_A3: now also DMA_RAM_BANK1.~ (A4)
- net DMA_BANK1_DOUT0: now also OLCL7.2 (D)
- net DMA_BANK1_DOUT1: now also OLCL6.2 (D)
- net DMA_BANK1_DOUT2: now also OLCL5.2 (D)
- net DMA_BANK1_DOUT3: now also OLCL4.2 (D)
- net DMA_BANK1_DOUT4: now also OLCL3.2 (D)
- net DMA_BANK1_DOUT5: now also OLCL2.2 (D)
- net DMA_BANK1_DOUT6: now also OLCL1.2 (D)
- net DMA_BANK1_DOUT7: now also OLCL0.2 (D)
- net wWOVT: now also DSAZ.2, DSSG.3; no longer DSAZ.3, DSSG.2
- net BSBO_1_A0: now reaches ZKBA.5
- net at DSLL.2, DSSX.3: now also DSSG.2; no longer DSSG.3
- net BSBO_0_A1: now reaches ZKBA.13
- net wSKKT: now reaches OKWN.1, PKBG.1, PKEJ.1
- net wSKKT: now also SKJF.1, SKKT.3
- net DMARAM_BANK1_A3: no longer names the net of DMA_RAM_BANK1.~ (A4), TKAC.3
- net DMA_ON renamed wOCRQ_wOCRS_~{XIN/8}
- net wDSAC renamed PATTERN_OFFSET_B1
- net wDSKP renamed PATTERN_END
- net wDSYT renamed PATTERN_OFFSET_B0
- net wQKBI: no longer names the net of QKBI.6 (~{Q})
- net wQKBI: no longer DSLL.1
- net wRKNG renamed ~{TRANSFER_PATTERN0}
- net wSKDA renamed TRANSFER_PATTERN1
- net TRANSFER_PATTERN1: now also DSAZ.3, SKDA.7 (Q); no longer DSAZ.2, SKDA.6 (Q)
- net wUKYL renamed HDMA_RELOAD_FLAG
- net wWOCA renamed ~{BANK0_WR}
- net wXKGP renamed ~{DMA_LENGTH_IS_ZERO}
- net wXKGY renamed HDMA_EMPTY_SCANLINE_COUNTER
- net wXOAO renamed ~{BANK2_WR}
- net ~{DMA_BANK0_WR}: no longer names the net of DMA_RAM_BANK0.17 (WR), ZKBW.9
- net ~{DMA_BANK1_WR}: no longer names the net of DMA_RAM_BANK1.17 (WR), ZKBW.20
- net ~{DMA_BANK2_WR}: no longer names the net of DMA_RAM_BANK2.17 (WR), ZKBW.22
- net ~{ZOOJ} renamed ~{wZOOJ}
- new net TRANSFER_PATTERN2: DSLL.1, QKBI.7 (Q)
- no-connect marks 24 -> 28
Other:
- sheet Other DMA gates ports: added BSBO_0_A1, BSBO_1_A0, DMA_CLK, HDMA_EMPTY_SCANLINE_COUNTER, HDMA_RELOAD_FLAG, NEXT_CHAN_CLK, PATTERN_END, wOCRQ_wOCRS_~{XIN/8}, ~{DMA_LENGTH_IS_ZERO}, ~{GDMA_CHAN_RST}, ~{STOP_DMA}; removed DMA_CLK?, wDSKP, wOCRQ_wOCRS_XIN/8, wSODM, wSODT, wSOGE, wUKYL, wXKGP, wXKGY
- note added: "BNHI B0_ENB 1 1 0 1 1 0 1 1 0 1 0 1 x x x 1"
- note added: "BNVB A0 0 0 1 1 1 0 0 0 1 1 0 1 x x x 1"
- note added: "BNVB_A0 is low when 0,1,5,6,7,A BNVB = 1xx1 + x100 + 1x0x + 001x"
- note added: "BNYC A1 0 0 0 0 0 1 1 1 1 1 0 1 x x x 1"
- note added: "BNYC_A1 is low when 0,1,2,3,4,A BNYC = x11x + 1xx1 + 1x0x + x1x1"
- note added: "Bank 1 data cannot be written during DMA transfer unlike bank 0 and 2 and furthermore, reading fast memory cannot be done and returns A address bank instead."
- note added: "HDMA Scanline count = 0"
- note removed: "BMHI B0_ENB 1 1 0 1 1 0 1 1 0 1 0 1 x x x 1"
- note removed: "BNVB A4 0 0 1 1 1 0 0 0 1 1 0 1 x x x 1"
- note removed: "BNVB_A4 is low when 0,1,5,6,7,A BNVB = 1xx1 + x100 + 1x0x + 001x"
- note removed: "BNYC A3 0 0 0 0 0 1 1 1 1 1 0 1 x x x 1"
- note removed: "BNYC_A3 is low when 0,1,2,3,4,A BNYC = x11x + 1xx1 + 1x0x + x1x1"
- note removed: "Bank 1 data not altered during DMA transfer unlike bank 0 and 2"
- note removed: "DMA_ADDR6-0 = 0"
- moved on the sheet: DSAC, DSAZ, DSCS, DSKP, DSLL, DSWN, DSXY, DSYT, DSZC

Commit message: Update in DMA sections - most debug signals identified. Error found in SYS clk generation. Simulation show correct 6, 8 and 12 cycle SYSCLK modes.
Connections:
- net D0: now also WKSN.5; no longer WKSN.4
- net D1: now also WKSN.13; no longer WKSN.11
- net D2: now also WKSN.15; no longer WKSN.16
- net D3: now also WKSN.25; no longer WKSN.24
- net D4: now also WKZC.5; no longer WKZC.4
- net D5: now also WKZC.13; no longer WKZC.11
- net D6: now also WKZC.15; no longer WKZC.16
- net D7: now also WKZC.25; no longer WKZC.24
- net DMA_ADDR10: now also WKSN.16; no longer WKSN.15
- net DMA_ADDR11: now also WKSN.24; no longer WKSN.25
- net DMA_ADDR12: now also WKZC.4; no longer WKZC.5
- net DMA_ADDR13: now also WKZC.11; no longer WKZC.13
- net DMA_ADDR14: now also WKZC.16; no longer WKZC.15
- net DMA_ADDR15: now also WKZC.24; no longer WKZC.25
- net DMA_ADDR8: now also WKSN.4; no longer WKSN.5
- net DMA_ADDR9: now also WKSN.11; no longer WKSN.13
- net wPOSD renamed GDMA_TRANSFER
- net ~{DMA_LENGTH_IS_ZERO} renamed ~{GDMA_LENGTH_IS_ZERO}
Other:
- sheet DMA & HDMA Control Registers ports: added FALLING_VBLANK; removed RISING_VBLANK
- sheet Other DMA gates ports: added GDMA_TRANSFER, HDMA_CHAN_RST, HDMA_EN, HDMA_TRANSFER, ~{GDMA_LENGTH_IS_ZERO}, ~{RESTART_DMA}; removed FALLING_VBLANK, MODE4_OR_MODE5, wBSEK, wDCBP_NOHDMA_2, wOORF, wPOSD, wPOSI, wWOCA, wXOAO, ~{DMA_LENGTH_IS_ZERO}, ~{MODE0_OR_MODE6}, ~{NO_DMA}, ~{NO_HDMA2}, ~{NO_HDMA}, ~{STOP_DMA}, ~{wRDY}
- moved on the sheet: OLZN, OLZR0, OLZR1, OLZR2, OLZR3, OLZR4, OLZR5, OLZR6, OLZR7, UKZFA, UKZFB, ULBKA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

Commit message: Schematics update.
Parts:
- removed OKMN0, OKMN1, OKMN2, OKMN3, OKTR0, OKTR1, OKTR2, OKTR3, OKTY0, OKTY1, OKTY2, OKTY3, OLDU0, OLDU1, OLDU2, OLDU3, OMIG0, OMIG1, OMIG2, OMIG3, OMNC0, OMNC1, OMNC2, OMNC3, QKEL0, QKEL1, QKEL2, QKEL3, QKQM0, QKQM1, QKQM2, QKQM3, RKOE0, RKOE1, RKOE2, RKOE3, RKUL0, RKUL1, RKUL2, RKUL3: TRI_BUF_IF1, symbol Ricoh_Cells:TRI_BUF_IF1
- removed OKPW, OKSL, OKUR, OLCW, OMDX, OMMV, QKGG, QKLR, RKPQ, RKPR, RKRK: INVERTER_A, symbol Ricoh_Cells:INVERTER_A
- removed QKHU, RKQY: NAND_3, symbol Ricoh_Cells:NAND_3
- added OCLC, OCLX: DFFR_A, symbol Ricoh_Cells:DFFR_A
- added OMRS: INVERTER_A, symbol Ricoh_Cells:INVERTER_A
Connections:
- net DMA_PA4: now reaches SKKP4.4 (Q)
- net DMA_PA5: now reaches SKKP5.4 (Q)
- net DMA_A12: now reaches PKEM3.4 (Q)
- net DMA_A4: now reaches PKBB3.4 (Q)
- net DMA_PA0: now reaches SKKP0.4 (Q)
- net DMA_A19: now reaches OLCL4.4 (Q)
- net DMA_A3: now reaches PKBB4.4 (Q)
- net DMA_PA1: now reaches SKKP1.4 (Q)
- net DMA_A10: now reaches PKEM5.4 (Q)
- net DMA_A7: now reaches PKBB0.4 (Q)
- net DMA_A1: now reaches PKBB6.4 (Q)
- net DMA_A11: now reaches PKEM4.4 (Q)
- net DMA_A2: now reaches PKBB5.4 (Q)
- net DMA_A0: now reaches PKBB7.4 (Q)
- net DMA_A5: now reaches PKBB2.4 (Q)
- net DMA_PA2: now reaches SKKP2.4 (Q)
- net DMA_A21: now reaches OLCL2.4 (Q)
- net DMA_A23: now reaches OLCL0.4 (Q)
- net DMA_A22: now reaches OLCL1.4 (Q)
- net DMA_PA3: now reaches SKKP3.4 (Q)
- net DMA_A16: now reaches OLCL7.4 (Q)
- net DMA_A9: now reaches PKEM6.4 (Q)
- net DMA_A17: now reaches OLCL6.4 (Q)
- net DMA_A14: now reaches PKEM1.4 (Q)
- net DMA_A8: now reaches PKEM7.4 (Q)
- net DMA_A20: now reaches OLCL3.4 (Q)
- net DMA_A15: now reaches PKEM0.4 (Q)
- net DMA_A6: now reaches PKBB1.4 (Q)
- net DMA_PA7: now reaches SKKP7.4 (Q)
- net DMA_PA6: now reaches SKKP6.4 (Q)
- net DMA_A18: now reaches OLCL5.4 (Q)
- net DMA_A13: now reaches PKEM2.4 (Q)
- net wSKKT renamed LATCH_NEXT_DMA_ADDR_BUS
- net ~{wZOOJ}: no longer names the net of ZOOJ.6 (~{Q})
- net ~{wZOOJ}: now also OMRS.1
- new net: OCLX.1 (~{RESET}), OCLX.5 (~{RESET})
- new net: OCLC.1 (~{RESET}), OCLC.5 (~{RESET})
- new net: OCLC.2 (D), OMRS.2
- new net DMA_B->A: OCLC.6 (Q)
- new net wNBHJ_wNBHM_XIN/2: OCLC.3 (CLK), OCLC.4 (~{CLK}), OCLX.3 (CLK), OCLX.4 (~{CLK})
- new net wUOGG: OCLX.2 (D)
- new net ~{DMA_BUS_ON}: OCLX.6 (Q)
- no-connect marks 28 -> 30
Other:
- sheet Other DMA gates ports: added CPU_CLK, DISABLE_HDMA_CHANNEL, DMA_TO_BE_SERVICED, ENABLE_HDMA_CHANNELS, GDMA, HBLANK, HDMA, LONG_FALLING_VBLANK, ~{BANK0_WR}, ~{BANK2_WR}; removed CMYW_EN, DMA_CLK, DMA_FALLING_VBLANK, DMA_RISING_HBLANK, wTOAY, wWOIX
- note added: "0= A->B, 1= B->A"
- note added: "0= Direct HDMA, 1= Indirect HDMA"
- note added: "Address Decoding"
- note added: "B-BUS offset based on pattern"
- note added: "DMA B-BUS"
- note added: "DMA Configuration"
- note removed: "B_BUS Address coming from DMA banks during DMA or from A bus otherwise"
- note removed: "JBQK = '0' when DMA is active"
- company: (none) -> Author: Regis Galland
- title: (none) -> SNES S-CPU Schematics 
- moved on the sheet: AMCK, AMEV, AMEX, AMGY, AMLH, AMMZ, AMQL, AMZL, ANAY, BNAP, BNBV, BNHI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

Commit message: Schematics tidying in progress.
Parts:
- removed DSAC, RKLP, SKCM, TKIB: AND_2, symbol Ricoh_Cells:AND_2
- removed DSAZ, DSSG, DSSX: NAND_3, symbol Ricoh_Cells:NAND_3
- removed DSCS, DSXY, DSYT, DSZC: NAND_2, symbol Ricoh_Cells:NAND_2
- removed DSKP: NAND_4, symbol Ricoh_Cells:NAND_4
- removed DSLL, DSWN, OLHT, OLMD, OLOZ, OLRW, OLUQ, OLWK, OMRS, QKAT, SKPA, TKAS: INVERTER_A, symbol Ricoh_Cells:INVERTER_A
- removed OCLC, OCLX: DFFR_A, symbol Ricoh_Cells:DFFR_A
- removed OKWN, OMBB, PKBG, PKEJ, QKAI, SKJF: BUF_DIFF, symbol Ricoh_Cells:BUF_DIFF
- removed OLCL0, OLCL1, OLCL2, OLCL3, OLCL4, OLCL5, OLCL6, OLCL7, OMDK0, OMDK1, OMDK2, OMDK3, OMDK4, OMDK5, OMDK6, OMDK7, PKBB0, PKBB1, PKBB2, PKBB3, PKBB4, PKBB5, PKBB6, PKBB7, PKEM0, PKEM1, PKEM2, PKEM3, PKEM4, PKEM5, PKEM6, PKEM7, QKAG0, QKAG1, QKAG2, QKAG3, QKAG4, QKAG5, QKAG6, SKKP0, SKKP1, SKKP2, SKKP3, SKKP4, SKKP5, SKKP6, SKKP7: D_LATCH_ARRAY, symbol Ricoh_Cells:D_LATCH_ARRAY
- removed OLCO0, OLCO1, OLCO2, OLCO3, OLGV0, OLGV1, OLGV2, OLGV3, OLNC0, OLNC1, OLNC2, OLNC3, OLSH0, OLSH1, OLSH2, OLSH3, OLWI0, OLWI1, OLWI2, OLWI3, OLXX0, OLXX1, OLXX2, OLXX3: TRI_BUF_IF1, symbol Ricoh_Cells:TRI_BUF_IF1
- removed QKBI, RKNG, SKDA, TKGB, ZOOJ: DFFR_B, symbol Ricoh_Cells:DFFR_B
- removed QKCI, RKNZ, TKFI, TKFN: 2BIT_FULL_ADD, symbol Ricoh_Cells:2BIT_FULL_ADD
- removed SKKT, TKAY, TKHG: OR_2, symbol Ricoh_Cells:OR_2
- removed TKAT: AND_3, symbol Ricoh_Cells:AND_3
Connections:
- no-connect marks 30 -> 17
Other:
- added sheet DMA CONFIG AND ADDRESS BUSES (dmaconfig_addr.kicad_sch)
- sheet DMA & HDMA Control Registers ports: added DISABLE_HDMA_CHANNEL, DMA_TO_BE_SERVICED, ENABLE_HDMA_CHANNELS, GDMA, HDMA, HDMA_CHAN_RST, HDMA_EN, HDMA_TRANSFER, NEXT_CHAN_CLK, wDBJW_wHASI_~{RST}, wNBEB_wNBEG_XIN/8, wXOWO, ~{GDMA_CHAN_RST}, ~{RESTART_DMA}; removed wNBEG_wNBEB_XIN/8
- sheet Other DMA gates ports: added wDBJW_wHASI_~{RST}; removed wDBJW_wHASI_RST
- note removed: "0= A->B, 1= B->A"
- note removed: "0= Direct HDMA, 1= Indirect HDMA"
- note removed: "0= INC or DEC, 1= Fixed"
- note removed: "0= INC, 1= DEC"
- note removed: "A_BUS Address coming from DMA banks"
- note removed: "B-BUS offset based on pattern"
- note removed: "DMA B-BUS"
- note removed: "DMA Configuration"
- note removed: "DMA RW signal based on bus direction"
- moved on the sheet: OLYP0, OLYP1, OLYP2, OLYP3, OLYP4, OLYP5, OLYP6, OLYP7, OLYU, OLZN, OLZR0, OLZR1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

Commit message: Big update on the hierarchical sheet. DMA section update too.
Parts:
- added OMNN: INVERTER_A, symbol Ricoh_Cells:INVERTER_A
- added OMVB, PKFR: OR_2, symbol Ricoh_Cells:OR_2
Connections:
- net DMA_OFF: now also OMNN.1
- net ~{DMA_RD}: now also OMVB.3
- net ~{DMA_WR}: now also PKFR.3
- net wNBKW_wNBPG_XIN/4 renamed wNBKW_wNBPG_~{XIN/4}
- net wSKDK renamed ~{DATA_IS_ZERO}
- new net: OMNN.2, OMVB.1, PKFR.1
- new net ~{CPU_RD}: OMVB.2
- new net ~{MAWK_WR}: PKFR.2
Other:
- sheet DMA & HDMA Control Registers ports: added none; removed ~{NO_DMA}, ~{NO_HDMA}
- sheet DMA CONFIG AND ADDRESS BUSES ports: added BUS_DIRECTION_FLAG, CYCLE_COUNTER[0..1], INDIRECT_HDMA_FLAG; removed DMA_B->A, wNBHJ_wNBHM_XIN/2, wQKAG5, wUOGG, wWOVT, wWOWE, ~{DMA_BUS_ON}
- sheet Other DMA gates ports: added BUS_DIRECTION_FLAG, CYCLE_COUNTER[0..1], DMA_B->A, INDIRECT_HDMA_FLAG, wHBLANK, wJPOUT[0..2], wNBHJ_wNBHM_XIN/2, wVBLANK, ~{DATA_IS_ZERO}, ~{DMA_BUS_ON}, ~{MODE5}; removed HBLANK, JPO0, JPO1, JPO2, VBLANK, wQKAG5, wSKDK, wUOGG, wWOVT, wWOWE
- moved on the sheet: RKMW, SKDK, TKDG, WKCF, WKNO, XKGP, XKGY, XKIN, XKKB, XKKC, XKKE

Commit message: DMA section update. Fixed gate related to INC/DEC and BORROW/CARRY FLAG
Connections:
- net wXOWO renamed ~{DMA_STEP2}
Other:
- sheet DMA & HDMA Control Registers ports: added ~{DMA_STEP2}; removed wXOWO
- sheet DMA CONFIG AND ADDRESS BUSES ports: added DMA_STEP1; removed wVOLG
- sheet Other DMA gates ports: added DMA_STEP1, ~{DMA_STEP2}; removed wVOLG, wXOWO
Changed lines of the file:
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@@
     (stroke (width 0) (type default))
   )
-  (wire (pts (xy 330.2 447.675) (xy 341.63 447.675))
+  (wire (pts (xy 323.85 447.675) (xy 341.63 447.675))
     (stroke (width 0) (type default))
   )
@@
     (effects (font (size 1.27 1.27)) (justify left bottom))
   )
-  (label "wXOWO" (at 533.4 299.72 0) (fields_autoplaced)
+  (label "~{DMA_STEP2}" (at 533.4 299.72 0) (fields_autoplaced)
     (effects (font (size 1.27 1.27)) (justify left bottom))
   )
@@
     (effects (font (size 1.27 1.27)) (justify left bottom))
   )
-  (label "wXOWO" (at 330.2 447.675 0) (fields_autoplaced)
+  (label "~{DMA_STEP2}" (at 323.85 447.675 0) (fields_autoplaced)
     (effects (font (size 1.27 1.27)) (justify left bottom))
   )
@@
     (effects (font (size 1.27 1.27)) (justify left bottom))
   )
-  (label "wXOWO" (at 635 195.58 180) (fields_autoplaced)
+  (label "~{DMA_STEP2}" (at 635 195.58 180) (fields_autoplaced)
     (effects (font (size 1.27 1.27)) (justify right bottom))
   )
@@
       (effects (font (size 1.27 1.27)) (justify right))
     )
-    (pin "wXOWO" input (at 546.1 299.72 180)
+    (pin "~{DMA_STEP2}" input (at 546.1 299.72 180)
       (effects (font (size 1.27 1.27)) (justify left))
     )
@@
       (effects (font (size 1.27 1.27)) (justify left))
     )
-    (pin "wVOLG" output (at 622.3 193.04 0)
+    (pin "DMA_STEP1" output (at 622.3 193.04 0)
       (effects (font (size 1.27 1.27)) (justify right))
     )
@@
       (effects (font (size 1.27 1.27)) (justify right))
     )
-    (pin "wXOWO" output (at 622.3 195.58 0)
+    (pin "~{DMA_STEP2}" output (at 622.3 195.58 0)
       (effects (font (size 1.27 1.27)) (justify right))
     )
@@
       (effects (font (size 1.27 1.27)) (justify left))
     )
-    (pin "wVOLG" input (at 711.2 193.04 180)
+    (pin "DMA_STEP1" input (at 711.2 193.04 180)
       (effects (font (size 1.27 1.27)) (justify left))
     )

Commit message: DMA section update. Found errors between some MUX and MUXI gates.
Parts:
- renumbered U22 to EMAU, U24 to EMCQ, U25 to EMGX
Other:
- sheet Other DMA gates ports: added HDMA_TABLE_RD; removed ~{DMA_BUS_ON}
- note added: "During DMA, A1-0 = - "00" will read DMA parameters from bank 1, B-bus address from bank 2 and Number of lines to transfer from bank 0 (only during HDMA). - "01" will read A-BUS address (16 bits) from bank 0 and 2 and A-BUS bank from bank 1. Bank does not get incremented when 16-bit address over spills. - "10" will read number of GDMA bytes to be transfered (16-bit) from bank 0 and 2 and HDMA data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"
