File: S-CPU_kicad/DMAothers.kicad_sch (KiCad schematic)
At the start: 37 parts

Commit message: More updates in DMA section.
Parts:
- removed FMKL: DFFR_A, symbol Ricoh_Cells:DFFR_A
- removed PORE: NOR_2, symbol Ricoh_Cells:NOR_2
- removed QOMK: DFFSR, symbol Ricoh_Cells:DFFSR
- removed ROHW: AND_3, symbol Ricoh_Cells:AND_3
- added CMVK, CMVW, LNZS, OOZO, POGD?, PORZ, SODT, SOLZ, SOOS, UOFS: INVERTER_A, symbol Ricoh_Cells:INVERTER_A
- added FMKL (x17): DFFR_B, symbol Ricoh_Cells:DFFR_B
- added OBEE (x2), POUO, ROLZ, SODM, SONJ, SOPE, TOAY, UOCE, UOFY, UOGG, UOKI, UONJ: AND_2, symbol Ricoh_Cells:AND_2
- added PORE, QOHV, RODU, SOQC, TODR: OR_2, symbol Ricoh_Cells:OR_2
- added ROBA: NOR_2, symbol Ricoh_Cells:NOR_2
- added ROMA: NAND_2, symbol Ricoh_Cells:NAND_2
- added SBRW (x3): DFFSR, symbol Ricoh_Cells:DFFSR
- added SOGE: AND_3, symbol Ricoh_Cells:AND_3
- added SOQE?: AOI_22, symbol Ricoh_Cells:AOI_22
Connections:
- net +5V: now also SBRW.2 (D), FMKL.2 (D), FMKL.2 (D), SBRW.2 (D), SBRW.2 (D)
- net DMA_ON: now also PORE.3
- net wDCBP_NOHDMA_2: now also OBEE.1; no longer ROMP.1
- net wMAGR_wMAGV: now also FMKL.3 (CLK), FMKL.3 (CLK), FMKL.3 (CLK), FMKL.4 (~{CLK}), FMKL.4 (~{CLK}), FMKL.4 (~{CLK}), SBRW.7 (CLK)
- net wNAGK_wNAJD: now also FMKL.3 (CLK), FMKL.4 (~{CLK})
- net wOCRQ_wOCRS_XIN/8: now also FMKL.3 (CLK), FMKL.4 (~{CLK})
- net ~{DMA_RESET}: now reaches FMKL.1 (~{RESET}), FMKL.1 (~{RESET}), FMKL.1 (~{RESET}), FMKL.1 (~{RESET}), FMKL.1 (~{RESET}), FMKL.1 (~{RESET}), FMKL.5 (~{RESET}), FMKL.5 (~{RESET}), FMKL.5 (~{RESET}), FMKL.5 (~{RESET}), FMKL.5 (~{RESET}), FMKL.5 (~{RESET}), OOBX.1 (~{RESET}), OOBX.5 (~{RESET}), POPB.2
- net ~{DMA_RESET}: now also FMKL.1 (~{RESET}), FMKL.1 (~{RESET}), FMKL.1 (~{RESET}), FMKL.1 (~{RESET}), FMKL.1 (~{RESET}), FMKL.1 (~{RESET}), FMKL.1 (~{RESET}), FMKL.1 (~{RESET}), FMKL.5 (~{RESET}), FMKL.5 (~{RESET}), FMKL.5 (~{RESET}), FMKL.5 (~{RESET}), FMKL.5 (~{RESET}), FMKL.5 (~{RESET}), FMKL.5 (~{RESET}), FMKL.5 (~{RESET}), FMKL.7 (Q), SBRW.1 (~{SET}), SBRW.1 (~{SET}), SBRW.3 (~{SET}), SBRW.3 (~{SET}), SOGE.2
- net at FMKL.2 (D): now also SONJ.3
- net at FMKL.3 (CLK), FMKL.4 (~{CLK}), OOBX.3 (CLK)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: now also FMKL.3 (CLK), FMKL.4 (~{CLK})
- net at FMKL.7 (Q): now also SBRW.7 (CLK)
- net at QOUI.1: now also SBRW.5 (Q)
- net at QOUI.2: now also ROHW.3, SBRW.2 (D), SBRW.4 (~{Q})
- net NO_DMA: now reaches FMKL.2 (D), FMKL.6 (~{Q}), OOIW.2, ROHW.1
- net at FMKL.1 (~{RESET}), FMKL.5 (~{RESET}), ROMP.3: now also SBRW.6 (~{RESET}), FMKL.2 (D)
- net wUOTI: now reaches FMKL.3 (CLK), FMKL.4 (~{CLK})
- net wUOTI: now also FMKL.7 (Q), PORE.1, PORZ.1, TOAY.1, TODR.1, UOCE.2, UOFY.2, UOGG.2
- net at FMKL.2 (D), FMKL.7 (Q): now also OOLO.1
- net at SOGW.3: now also ROMP.1; no longer ROMP.2
- net wPOSD: now reaches FMKL.2 (D), OOSR.1, POSD.3
- net wPOSD: now also SOOS.1
- net at OOSR.2: now also FMKL.6 (~{Q}); no longer FMKL.7 (Q)
- net at POSD.1: now also PORZ.2
- net at POSD.2: now also FMKL.7 (Q), PORE.2
- net at FMKL.7 (Q), POOO.2: now also FMKL.2 (D)
- net at ROHL.1: now also FMKL.6 (~{Q})
- net at ROHL.2: now also FMKL.2 (D), RODU.3
- net at ROHL.3, SOGW.2, SOJJ.2: now also SBRW.7 (CLK)
- net wOORF: now reaches OORF.3
- net wOORF: now also FMKL.2 (D), ROBA.2, SOGE.3
- net ?: now reaches ROME.1
- net at FMKL.6 (~{Q}): no longer OOLO.1
- net at SOGW.1: now also SBRW.4 (~{Q})
- net at SBRW.1 (~{SET}), SBRW.3 (~{SET}): now also SBRW.1 (~{SET}), SBRW.3 (~{SET}), SBRW.6 (~{RESET})
- net at SBRW.5 (Q): now also FMKL.2 (D), FMKL.2 (D)
- net at POOO.1: now also FMKL.6 (~{Q})
- net at SOJJ.1: now also SBRW.5 (Q)
- net at SOJJ.3: now also LNZS.1, SOGE.1
- net SYSCLK renamed wUOTW
- net wUOTW: now also FMKL.7 (Q), OBEE.2
- net wNBEG_wNBEB_XIN/8 renamed wNBEB_wNBEG_XIN/8
- new net: UOCE.1, UOFS.1, UOGG.3
- new net: UOFS.2, UOFY.1
- new net: OBEE.2, QOHV.3
- new net: FMKL.1 (~{RESET}), FMKL.5 (~{RESET}) (x5)
- new net: FMKL.3 (CLK), FMKL.4 (~{CLK}) (x2)
- new net: FMKL.3 (CLK), FMKL.3 (CLK), FMKL.3 (CLK), FMKL.3 (CLK), FMKL.3 (CLK), FMKL.3 (CLK), FMKL.4 (~{CLK}), FMKL.4 (~{CLK}), FMKL.4 (~{CLK}), FMKL.4 (~{CLK}), FMKL.4 (~{CLK}), FMKL.4 (~{CLK})
- new net: FMKL.2 (D), SONJ.1, SOPE.3
- new net: FMKL.2 (D), FMKL.7 (Q), FMKL.7 (Q), OBEE.1
- new net: FMKL.3 (CLK), FMKL.4 (~{CLK}), OBEE.3
- new net: OOZO.2, UONJ.1
- new net: POUO.1, UOKI.3, UONJ.2
- new net: ROLZ.1, ROMA.3
- new net: FMKL.2 (D), FMKL.7 (Q) (x2)
- new net: FMKL.2 (D), FMKL.7 (Q), QOHV.2
- new net: CMVK.1, CMVW.2
- new net: CMVK.2, FMKL.2 (D)
- new net: OOZO.1, POUO.2
- new net: FMKL.7 (Q), RODU.1
- new net: ROBA.3, RODU.2, SOLZ.1
- new net: SOPE.1, SOQC.3
- new net: SBRW.6 (~{RESET}), SOLZ.2
- new net: FMKL.6 (~{Q}), ROBA.1
- new net: SOQC.1, SOQE?.3
- new net: FMKL.1 (~{RESET}), FMKL.2 (D), FMKL.5 (~{RESET})
- new net: FMKL.7 (Q), SBRW.6 (~{RESET})
- new net: LNZS.2, TOAY.2
- new net: FMKL.3 (CLK), FMKL.4 (~{CLK}), SBRW.4 (~{Q})
- new net: POGD?.2, ROMA.1
- new net: FMKL.6 (~{Q}), QOHV.1
- new net: SONJ.2, SOOS.2
- new net: FMKL.7 (Q), SBRW.7 (CLK)
- new net CMYW: CMVW.1
- new net DMA_FALLING_VBLANK: SOQC.2
- new net DMA_RISING_HBLANK: SOQE?.1
- new net MODE4_OR_MODE5: ROMA.2
- new net VBLANK: SOQE?.4
- new net wDBJW_wHASI_RST: FMKL.1 (~{RESET}), FMKL.1 (~{RESET}), FMKL.1 (~{RESET}), FMKL.5 (~{RESET}), FMKL.5 (~{RESET}), FMKL.5 (~{RESET})
- new net wOACU_wOAFI_XIN/4: FMKL.3 (CLK), FMKL.4 (~{CLK})
- new net wPOSI: UOKI.2
- new net wSODM: SODM.3
- new net wSODT: SODM.1, SODT.2
- new net wSOGE: SODM.2, SOGE.4
- new net ~{MODE0_OR_MODE6}: ROLZ.2
- new net ~{NO_HDMA2}: ROMP.2
- new net ~{NO_HDMA}: SOPE.2
- new net ~{wRDY}: POGD?.1
- no-connect marks 12 -> 37
Other:
- note added: "to DMA"
- note removed: "Some HDMA channels are enabled"
- moved on the sheet: FMKL, OOIW, OOLO, OORC, OORF, OOSR, POGD, POOO, POPB, POSD, POUL, QOUI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

Commit message: Fixed reset signal in DMA section.
Connections:
- net +5V: now also FMKL.2 (D)
- net wDBJW_wHASI_RST: now also FMKL.1 (~{RESET}), FMKL.1 (~{RESET}), FMKL.1 (~{RESET}), FMKL.1 (~{RESET}), FMKL.1 (~{RESET}), FMKL.1 (~{RESET}), FMKL.1 (~{RESET}), FMKL.1 (~{RESET}), FMKL.1 (~{RESET}), FMKL.1 (~{RESET}), FMKL.1 (~{RESET}), FMKL.1 (~{RESET}), FMKL.1 (~{RESET}), FMKL.1 (~{RESET}), FMKL.5 (~{RESET}), FMKL.5 (~{RESET}), FMKL.5 (~{RESET}), FMKL.5 (~{RESET}), FMKL.5 (~{RESET}), FMKL.5 (~{RESET}), FMKL.5 (~{RESET}), FMKL.5 (~{RESET}), FMKL.5 (~{RESET}), FMKL.5 (~{RESET}), FMKL.5 (~{RESET}), FMKL.5 (~{RESET}), FMKL.5 (~{RESET}), FMKL.5 (~{RESET}), OBEE.2, OOBX.1 (~{RESET}), OOBX.5 (~{RESET}), POPB.2, SBRW.1 (~{SET}), SBRW.1 (~{SET}), SBRW.3 (~{SET}), SBRW.3 (~{SET}), SOGE.2
- net wOCRQ_wOCRS_XIN/8: now also FMKL.3 (CLK), FMKL.4 (~{CLK})
- net wPOSD: now also FMKL.3 (CLK), FMKL.4 (~{CLK})
- net wPOSI: now also FMKL.2 (D), FMKL.7 (Q), OORC.2
- net at FMKL.1 (~{RESET}), FMKL.5 (~{RESET}): now also FMKL.7 (Q), OBEE.1
- net wOBXZ_wOCHV_~{XIN/2}: now reaches FMKL.3 (CLK), FMKL.3 (CLK), FMKL.3 (CLK), FMKL.3 (CLK), FMKL.3 (CLK), FMKL.3 (CLK), FMKL.4 (~{CLK}), FMKL.4 (~{CLK}), FMKL.4 (~{CLK}), FMKL.4 (~{CLK}), FMKL.4 (~{CLK}), FMKL.4 (~{CLK})
- net at FMKL.2 (D), FMKL.7 (Q): no longer FMKL.7 (Q), OBEE.1
- net at OOZO.1, POUO.2: now also SBRW.5 (Q), SOJJ.1
- removed net wUOTW: FMKL.7 (Q), OBEE.2, OOLO.2
- removed net ~{DMA_RESET}: FMKL.1 (~{RESET}), FMKL.1 (~{RESET}), FMKL.1 (~{RESET}), FMKL.1 (~{RESET}), FMKL.1 (~{RESET}), FMKL.1 (~{RESET}), FMKL.1 (~{RESET}), FMKL.1 (~{RESET}), FMKL.1 (~{RESET}), FMKL.1 (~{RESET}), FMKL.1 (~{RESET}), FMKL.1 (~{RESET}), FMKL.1 (~{RESET}), FMKL.1 (~{RESET}), FMKL.5 (~{RESET}), FMKL.5 (~{RESET}), FMKL.5 (~{RESET}), FMKL.5 (~{RESET}), FMKL.5 (~{RESET}), FMKL.5 (~{RESET}), FMKL.5 (~{RESET}), FMKL.5 (~{RESET}), FMKL.5 (~{RESET}), FMKL.5 (~{RESET}), FMKL.5 (~{RESET}), FMKL.5 (~{RESET}), FMKL.5 (~{RESET}), FMKL.5 (~{RESET}), FMKL.7 (Q), OOBX.1 (~{RESET}), OOBX.5 (~{RESET}), POPB.2, SBRW.1 (~{SET}), SBRW.1 (~{SET}), SBRW.3 (~{SET}), SBRW.3 (~{SET}), SOGE.2
- new net: FMKL.7 (Q), OOLO.2
- now unconnected: FMKL.6 (~{Q})
Other:
- moved on the sheet: FMKL, OBEE, OOIW, OOLO, OOZO, POGD?, POUL, POUO, QOUI, ROHW, ROLZ, ROMA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

Commit message: Another latch with reset identified. TCKSEL demux cell worked out + notes added to schematics.
Parts:
- removed FMKL: DFFR_B, symbol Ricoh_Cells:DFFR_B
- removed SBRW: DFFSR, symbol Ricoh_Cells:DFFSR
- removed SOQE?: AOI_22, symbol Ricoh_Cells:AOI_22
- added FMKL (x2): DFFR_B, symbol Ricoh_Cells:DFFR_B
- added OBEE, SOUV: AND_2, symbol Ricoh_Cells:AND_2
- added ODNR: TRI_BUF_IF0, symbol Ricoh_Cells:TRI_BUF_IF0
- added RONY, SOVA: INVERTER_A, symbol Ricoh_Cells:INVERTER_A
- added SOXY, SOZA: NAND_3, symbol Ricoh_Cells:NAND_3
Connections:
- net +5V: now also FMKL.2 (D)
- net DMA_RISING_HBLANK: now also SOUV.2
- net VBLANK: now also SOVA.1
- net wDBJW_wHASI_RST: now also FMKL.1 (~{RESET}), FMKL.5 (~{RESET})
- net wOACU_wOAFI_XIN/4: now also FMKL.3 (CLK), FMKL.4 (~{CLK})
- net wPOSD: now also SOXY.1, SOZA.2; no longer FMKL.3 (CLK), FMKL.4 (~{CLK})
- net wUOTI: now also FMKL.7 (Q)
- net at OBEE.3: now also OBEE.2
- net wSOXO: now reaches FMKL.7 (Q)
- net wSOXO: now also FMKL.1 (~{RESET}), FMKL.2 (D), FMKL.5 (~{RESET}), SOXY.3
- net wROLX: now reaches FMKL.7 (Q)
- net wROLX: now also FMKL.3 (CLK), FMKL.4 (~{CLK})
- net at OBEE.3: now also FMKL.1 (~{RESET}), FMKL.5 (~{RESET})
- net at SOQC.1: now also SOUV.3
- net wTOAY: now reaches TOAY.3
- net wQOXN: now reaches FMKL.7 (Q), OOLO.2
- net wQOXN: now also FMKL.2 (D)
- net at FMKL.7 (Q): now also FMKL.3 (CLK), FMKL.4 (~{CLK})
- net at SBRW.1 (~{SET}), SBRW.1 (~{SET}), SBRW.3 (~{SET})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: now also OBEE.3
- net at LNZS.1, SOGE.1, SOJJ.3: now also ODNR.1 (IN), ODNR.3 (IN)
- net CMYW renamed CMYW_EN
- new net: RONY.2, SOXY.2
- new net: SOXY.4, SOZA.1
- new net: FMKL.7 (Q), SOZA.3
- new net: SOUV.1, SOVA.2
- new net DFF?: RONY.1
- new net PA1: ODNR.4
- new net wSOZA: OBEE.1, SOZA.4
- new net ~{MODE5}: ODNR.2 (~{ENA})
- no-connect marks 37 -> 39
Other:
- note added: "SOPE goes high for a few cycles when HDMA is enabled at: - the end of VBLANK (falling edge) - the rising edge of HBLANK when VBLANK is low (i.e. during rendering)"
- note removed: "to DMA"
- moved on the sheet: CMVK, CMVW, FMKL, LNZS, OBEE, ROBA, RODU, ROHL, ROMP, SBRW, SODM, SODT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

Commit message: Almost all cells captured in schematicAlmost all cells captured in schematics. Enter the commit message for your changes. Lines starting
Parts:
- added ASAK (x2), ASEA, XOAO, XOKS, XONF: NAND_2, symbol Ricoh_Cells:NAND_2
- added ASAR, ASBC, ASIK, CSDS, CSGZ, VOLG, XOFV, XPDE, YOLV (x6): AND_2, symbol Ricoh_Cells:AND_2
- added ASBG, ASDD (x4), ASFK, BSHU, CTBB (x2), RKMU, WOCA, WOEK, WOZE, XOAP, XOIL, XOMS, XOWO, YOXQ, ZONT, ZORE: INVERTER_A, symbol Ricoh_Cells:INVERTER_A
- added ASCU, ASDM (x6), FMKL (x22), XOGA, YOJQ, ZOED: DFFR_B, symbol Ricoh_Cells:DFFR_B
- added ASGB, YOOX: AND_3, symbol Ricoh_Cells:AND_3
- added BSBO: MUX_2x4:1, symbol Ricoh_Cells:MUX_2x4{colon}1
- added BSEK, WOWY: AND_2, symbol Ricoh_Cells:AND_3
- added BSQD (x2), BSSO (x2), CSZL (x2): DELAY_BUF, symbol Ricoh_Cells:DELAY_BUF
- added CSFL, CSLQ, DTHT, DTSJ: XNOR, symbol Ricoh_Cells:XNOR
- added DTBB, WODN, YORL, ZOQW: OR_2, symbol Ricoh_Cells:OR_2
- added DTEF, YOCE: NOR_3, symbol Ricoh_Cells:NOR_3
- added HAUU0, HAUU1: MUX, symbol Ricoh_Cells:MUX
- added ODNR (x12): TRI_BUF_IF0, symbol Ricoh_Cells:TRI_BUF_IF0
- added PAWC (x2): NOR_LATCH, symbol Ricoh_Cells:NOR_LATCH
- added RKUL4: TRI_BUF_IF1, symbol Ricoh_Cells:TRI_BUF_IF1
- added VOJL: NAND_4, symbol Ricoh_Cells:NAND_4
- added XOTJ: DR_LATCH, symbol Ricoh_Cells:DR_LATCH
- added YOXF (x4), ZODY (x3), ZONY: NOR_2, symbol Ricoh_Cells:NOR_2
- added ZOJK: NAND_3, symbol Ricoh_Cells:NAND_3
Connections:
- net DFF? is gone; now on net wYOYP: RONY.1
- net +5V: now also XOGA.2 (D)
- net DMA_ON: now also FMKL.1 (~{RESET}), FMKL.5 (~{RESET}), YOLV.2
- net wDBJW_wHASI_RST: now also FMKL.1 (~{RESET}), FMKL.1 (~{RESET}), FMKL.1 (~{RESET}), FMKL.1 (~{RESET}), FMKL.1 (~{RESET}), FMKL.1 (~{RESET}), FMKL.1 (~{RESET}), FMKL.5 (~{RESET}), FMKL.5 (~{RESET}), FMKL.5 (~{RESET}), FMKL.5 (~{RESET}), FMKL.5 (~{RESET}), FMKL.5 (~{RESET}), FMKL.5 (~{RESET}), WOWY.1, XOFV.1, XOTJ.4 (~{RESET}), ZORE.1
- net wNBEB_wNBEG_XIN/8: now also ASAK.2, ASDD.1, DTSJ.3 (2), FMKL.2 (D), FMKL.3 (CLK), FMKL.4 (~{CLK}), VOJL.1, YOXF.2, ZOED.3 (CLK), ZOED.4 (~{CLK})
- net wOACU_wOAFI_XIN/4: now also DTEF.1, DTSJ.2 (1), FMKL.3 (CLK), FMKL.3 (CLK), FMKL.3 (CLK), FMKL.4 (~{CLK}), FMKL.4 (~{CLK}), FMKL.4 (~{CLK}), VOJL.2, YOOX.3; no longer FMKL.3 (CLK), FMKL.4 (~{CLK})
- net wOBXZ_wOCHV_~{XIN/2}: now also ASDM.3 (CLK), ASDM.3 (CLK), ASDM.3 (CLK), ASDM.3 (CLK), ASDM.3 (CLK), ASDM.4 (~{CLK}), ASDM.4 (~{CLK}), ASDM.4 (~{CLK}), ASDM.4 (~{CLK}), ASDM.4 (~{CLK}), FMKL.3 (CLK), FMKL.3 (CLK), FMKL.3 (CLK), FMKL.3 (CLK), FMKL.3 (CLK), FMKL.3 (CLK), FMKL.3 (CLK), FMKL.3 (CLK), FMKL.3 (CLK), FMKL.3 (CLK), FMKL.4 (~{CLK}), FMKL.4 (~{CLK}), FMKL.4 (~{CLK}), FMKL.4 (~{CLK}), FMKL.4 (~{CLK}), FMKL.4 (~{CLK}), FMKL.4 (~{CLK}), FMKL.4 (~{CLK}), FMKL.4 (~{CLK}), FMKL.4 (~{CLK}), YOCE.3
- net wOCRQ_wOCRS_XIN/8: now also ASAR.2, YOLV.1, YOLV.1, YOOX.1
- net wOORF: now also WOEK.1, XOFV.2
- net wPOSD: now also VOJL.4, XPDE.1
- net wPOSI: now also FMKL.2 (D)
- net wSODM: now also FMKL.2 (D), ODNR.1 (IN), ODNR.3 (IN), VOLG.2
- net ~{MODE5}: now also ODNR.2 (~{ENA}), ODNR.2 (~{ENA}), ODNR.2 (~{ENA}), ODNR.2 (~{ENA}), ODNR.2 (~{ENA}), ODNR.2 (~{ENA}), ODNR.2 (~{ENA}), ODNR.2 (~{ENA}), ODNR.2 (~{ENA}), RKUL4.2 (~{ENA})
- net wUOGG: now reaches UOCE.1, UOFS.1, UOGG.3
- net wUOGG: now also ASBC.2, CSDS.2, CSGZ.2, YOLV.2
- net at UOGG.1: now also FMKL.7 (Q)
- net wROMP: now reaches FMKL.1 (~{RESET}), FMKL.2 (D), FMKL.5 (~{RESET}), ROMP.3, SBRW.6 (~{RESET})
- net at UONJ.3: now also FMKL.2 (D)
- net wSOKC: now reaches OOZO.1, POUO.2, SBRW.5 (Q), SOJJ.1
- net wSOKC: now also FMKL.2 (D)
- net wUOFY: now reaches UOFY.3
- net wUOFY: now also BSBO.1 (SEL0), HAUU1.1
- net at UOKI.1: now also FMKL.7 (Q)
- net at TODR.2: now also XOFV.3, XOGA.1 (~{RESET}), XOGA.5 (~{RESET})
- net at TODR.3: now also ASCU.1 (~{RESET}), ASCU.5 (~{RESET}), YOJQ.1 (~{RESET}), YOJQ.5 (~{RESET})
- net wSOJJ: now reaches LNZS.1, ODNR.1 (IN), ODNR.3 (IN), SOGE.1, SOJJ.3
- net at SODT.1: now also ODNR.1 (IN), ODNR.3 (IN), ODNR.4, ODNR.4, ODNR.4
- net wVOJF: now reaches FMKL.2 (D)
- net wVOJF: now also FMKL.7 (Q), VOJL.3
- net at POUO.3: now also FMKL.2 (D)
- net wUOCE: now reaches UOCE.3
- net wUOCE: now also BSBO.20 (SEL1), HAUU0.1
- net ? renamed wYOYP
- net wYOYP: now also FMKL.7 (Q), ODNR.1 (IN), ODNR.3 (IN)
- new net: ASDM.1 (~{RESET}), ASDM.5 (~{RESET}) (x6)
- new net: ASDM.2 (D), DTBB.3
- new net: ASDM.7 (Q), YOLV.1
- new net: FMKL.7 (Q), VOLG.1
- new net: FMKL.2 (D), FMKL.7 (Q) (x2)
- new net: FMKL.2 (D), FMKL.2 (D), FMKL.7 (Q), ZOQW.2
- new net: FMKL.1 (~{RESET}), FMKL.5 (~{RESET}) (x12)
- new net: FMKL.2 (D), PAWC.3 (Q)
- new net: ASCU.2 (D), YOJQ.2 (D), ZODY.3
- new net: ASCU.3 (CLK), ASCU.4 (~{CLK}), XOGA.3 (CLK), XOGA.4 (~{CLK}), YOJQ.3 (CLK), YOJQ.4 (~{CLK}), YOLV.3
- new net: ASCU.7 (Q), YOOX.2
- new net: ASGB.4, YOLV.1
- new net: FMKL.7 (Q), XOIL.1
- new net: FMKL.7 (Q), XOMS.1, XONF.1
- new net: ODNR.1 (IN), ODNR.3 (IN), WODN.3, YOCE.2
- new net: WOCA.1, XOAO.1, YOCE.4
- new net: ASDM.2 (D), ZODY.3
- new net: BSEK.2, FMKL.7 (Q)
- new net: ASDM.2 (D), RKMU.2
- new net: ASDD.2, ASDM.3 (CLK), ASDM.4 (~{CLK}), ASEA.2, BSBO.11
- new net: BSQD.2, CSZL.1 (x2)
- new net: CSZL.2, CTBB.1 (x2)
- new net: ASAK.1, ASAR.1, XPDE.2, YOJQ.7 (Q), YOXF.1, ZOED.2 (D)
- new net: XPDE.3, YOXF.2
- new net: CSDS.1, CSFL.1
- new net: ASDM.2 (D), YOLV.3
- new net: ASDM.7 (Q), YOLV.2
- new net: ODNR.2 (~{ENA}), XOIL.2, XOKS.2, XONF.2
- new net: ODNR.2 (~{ENA}), XONF.3
- new net: FMKL.6 (~{Q}), WODN.2
- new net: FMKL.3 (CLK), FMKL.4 (~{CLK}), FMKL.7 (Q)
- new net: XOTJ.2 (D), YORL.3
- new net: ASAK.3, BSBO.3
- new net: ZODY.1, ZOED.7 (Q)
- new net: DTEF.2, DTHT.1
- new net: ASDD.2, DTEF.3
- new net: DTBB.1, DTEF.4
- new net: HAUU1.3, YOXF.3
- new net: VOJL.5, WOWY.3
- new net: ASIK.2, BSHU.1, FMKL.2 (D), FMKL.7 (Q)
- new net: ASIK.3, CSFL.3 (2), CSLQ.3 (2)
- new net: BSQD.1, BSSO.2 (x2)
- new net: XOKS.1, XOMS.2
- new net: ODNR.2 (~{ENA}), XOKS.3
- new net: BSBO.12, BSBO.14, CTBB.2
- new net: ZOJK.1, ZONT.2
- new net: ASEA.3, BSBO.5
- new net: BSBO.29, ODNR.1 (IN), ODNR.3 (IN), YOXF.2
- new net: ASDD.2, YOLV.1
- new net: ASDD.1, ASDM.2 (D), DTBB.2, DTSJ.1, YOLV.2, ZODY.2
- new net: HAUU1.2, YOXF.3
- new net: ASBC.3, FMKL.2 (D)
- new net: BSHU.2, FMKL.3 (CLK), FMKL.4 (~{CLK})
- new net: BSEK.1, FMKL.7 (Q)
- new net: ZODY.1, ZODY.3
- new net: BSSO.1, YOLV.3
- new net: XOAO.2, XOAP.2
- new net: YOLV.1, ZOJK.4
- new net: PAWC.1 (SET), ZONY.3
- new net: PAWC.1 (SET), PAWC.4 (RESET), ZOQW.3
- new net: BSBO.6, BSBO.8, CTBB.2
- new net: FMKL.2 (D), YOXF.3
- new net: ASAR.3, BSBO.9
- new net: ASBC.1, ASBG.2
- new net: ZOQW.1, ZORE.2
- new net: FMKL.1 (~{RESET}), FMKL.1 (~{RESET}), FMKL.5 (~{RESET}), FMKL.5 (~{RESET}), WOWY.4
- new net: FMKL.2 (D), FMKL.3 (CLK), FMKL.4 (~{CLK}), FMKL.6 (~{Q})
- new net: CSGZ.1, CSLQ.1
- new net: ZOED.1 (~{RESET}), ZOED.5 (~{RESET})
- new net: ASFK.2, ASGB.1
- new net: ASGB.2, FMKL.6 (~{Q})
- new net: ASGB.3, FMKL.7 (Q)
- new net: WOWY.2, WOZE.2
- new net: ASDM.7 (Q), BSSO.1
- new net: FMKL.2 (D), FMKL.6 (~{Q})
- new net: FMKL.2 (D), HAUU0.4
- new net: ASAK.3, YOLV.2
- new net: BSBO.24, ODNR.1 (IN), ODNR.3 (IN), YOXF.1
- new net: YOXQ.2, ZONY.2
- new net: ASDD.2, ASDM.2 (D)
- new net: HAUU0.2, HAUU1.4
- new net: XOAP.1, YOXF.3
- new net FALLING_VBLANK: ASAK.1, YORL.2
- new net JPO0: ODNR.4
- new net JPO1: ODNR.4
- new net JPO2: ODNR.4
- new net PA0: ODNR.4
- new net PA2: ODNR.4
- new net PA3: ODNR.4
- new net PA4: RKUL4.4
- new net PA5: ODNR.4
- new net PA6: ODNR.4
- new net PA7: ODNR.4
- new net wASLJ: HAUU0.3, PAWC.3 (Q)
- new net wBSEK: BSEK.4, ODNR.1 (IN), ODNR.3 (IN)
- new net wCSDS: CSDS.3
- new net wCSGZ: CSGZ.3
- new net wDSKP: FMKL.2 (D), YOLV.2
- new net wNAQE_wNBBM_XIN/2: FMKL.3 (CLK), FMKL.3 (CLK), FMKL.3 (CLK), FMKL.3 (CLK), FMKL.3 (CLK), FMKL.4 (~{CLK}), FMKL.4 (~{CLK}), FMKL.4 (~{CLK}), FMKL.4 (~{CLK}), FMKL.4 (~{CLK})
- new net wNBKW_wNBPG_~{XIN/4}: FMKL.3 (CLK), FMKL.4 (~{CLK}), YOCE.1
- new net wQKAG5: RKMU.1
- new net wSKDK: ASBG.1
- new net wUKYL: ASFK.1
- new net wVOLG: ASDD.1, FMKL.2 (D), VOLG.3
- new net wWOCA: WOCA.2
- new net wWOEK: ODNR.1 (IN), ODNR.3 (IN), WODN.1, WOEK.2
- new net wWOIX: ODNR.1 (IN), ODNR.3 (IN), YOLV.3
- new net wWOVT: ASDD.1, DTHT.3 (2), FMKL.7 (Q), ZODY.1
- new net wWOWE: DTHT.2 (1), FMKL.7 (Q), ZODY.2
- new net wWPAI: FMKL.2 (D), FMKL.7 (Q), WOZE.1, XOTJ.1 (~{ENA}), XOTJ.3 (ENA), XOWO.1
- new net wXKGP: ZODY.2
- new net wXKGY: RKUL4.1 (IN), RKUL4.3 (IN), YORL.1
- new net wXOAO: XOAO.3
- new net wXOPA: ODNR.1 (IN), ODNR.3 (IN), YOLV.3
- new net wXOTJ: FMKL.2 (D), XOTJ.6 (~{Q}), ZOJK.3, ZONY.1
- new net wXOWO: PAWC.4 (RESET), XOWO.2
- new net wXPHM: ASAK.2, FMKL.2 (D), FMKL.7 (Q), YOXQ.1
- new net wYOOX: ODNR.1 (IN), ODNR.3 (IN), YOOX.4
- new net wYOWZ: FMKL.7 (Q), ZOJK.2
- new net wZOGE: ASIK.1, BSEK.3, FMKL.7 (Q)
- new net wZOGY: ODNR.1 (IN), ODNR.3 (IN), YOLV.3
- new net ~{INDIRECT_HDMA}: ASDM.7 (Q), ASEA.1, ZONT.1
- new net ~{wCSMZ}: ASDM.6 (~{Q}), CSFL.2 (1)
- new net ~{wCSQI}: ASDM.6 (~{Q}), CSLQ.2 (1)
- new net ~{wXOGA}: XOGA.6 (~{Q}), YOXF.1, YOXF.1, YOXF.2
- no-connect marks 39 -> 88
Other:
- note added: "Indirect HDMA transfer when set to 1"
- note added: "WOVT and WOWE is a 2 bit counter for DMA transfers that deals with different patterns"
- moved on the sheet: CMVK, CMVW, FMKL, LNZS, OBEE, ODNR, OOZO, POGD?, POUO, ROBA, RODU, ROHL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

Commit message: Progress in DMA section. Fixed some DFF output issues.
Parts:
- removed HAUU0, HAUU1: MUX, symbol Ricoh_Cells:MUX
- added ZOAA, ZOBY: MUXI, symbol Ricoh_Cells:MUXI
- added ZOAV: INVERTER_A, symbol Ricoh_Cells:INVERTER_A
- ASAK: value NAND_2 -> NOR_2; symbol Ricoh_Cells:NAND_2 -> Ricoh_Cells:NOR_2
Connections:
- net wASLJ: now also ZOAV.1
- net wUOCE: now also ZOAA.1
- net wUOFY: now also ZOBY.1
- net at YOXF.3: now also ZOBY.2
- net BSBO_0_A1: now reaches BSBO.29, ODNR.1 (IN), ODNR.3 (IN), YOXF.2
- net at YOXF.3: now also ZOBY.3
- net at FMKL.2 (D): now also ZOAA.4
- net BSBO_1_A0: now reaches BSBO.24, ODNR.1 (IN), ODNR.3 (IN), YOXF.1
- net DMA_CLK? renamed DMA_CLK
- net wDSKP renamed PATTERN_END
- net wOCRQ_wOCRS_XIN/8 renamed wOCRQ_wOCRS_~{XIN/8}
- net wSODM renamed NEXT_CHAN_CLK
- net wSODT renamed ~{GDMA_CHAN_RST}
- net wSOGE renamed ~{STOP_DMA}
- net wUKYL renamed HDMA_RELOAD_FLAG
- net wWOCA renamed ~{BANK0_WR}
- net wXKGP renamed ~{DMA_LENGTH_IS_ZERO}
- net wXKGY renamed HDMA_EMPTY_SCANLINE_COUNTER
- net wXOAO renamed ~{BANK2_WR}
- new net: ZOAA.3, ZOBY.4
- new net: ZOAA.2, ZOAV.2
Other:
- note added: "POSI 0 0 1 1"
- note added: "SODT (~{GDMA_CHAN_RST} ~{wYOOX} On for 2 XIN cycles when GDMA length becomes 0 ~{wYOOX} On for 2 XIN cycles when GDMA length becomes 0 ~{wXOPA} ~{wYOGY}"
- note added: "SOKC 0 1 0 1"
- note added: "UOCE & UOFY can only be "00", "10" or "01" but never "11""
- note added: "When A1-0 = "00" BANK2 WR is not allowed as it corresponds to B Bus address but it allows BANK0 WR to update the HDMA line counter BANK0 WR and BANK2 WR are active together to update: - the A-bus 16-bit address when A1-0 = "01" - the GDMA byte counter when A1-0 = "10" - the HDMA table address when A1-0 = "11""
- note added: "negative pulse on falling edge"
- note added: "positive pulse on falling edge"
- moved on the sheet: ASAK, ASCU, ASDD, ASDM, ASEA, BSBOA, BSBOB, BSBOC, BSQD, BSSO, CSZL, CTBB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

Commit message: Update in DMA sections - most debug signals identified. Error found in SYS clk generation. Simulation show correct 6, 8 and 12 cycle SYSCLK modes.
Parts:
- removed ASAR, ROLZ: AND_2, symbol Ricoh_Cells:AND_2
- removed ASEA, ROMA: NAND_2, symbol Ricoh_Cells:NAND_2
- removed CMVK, CMVW, POGD?: INVERTER_A, symbol Ricoh_Cells:INVERTER_A
- added ASAK: NOR_2, symbol Ricoh_Cells:NOR_2
- added XPDE: AND_2, symbol Ricoh_Cells:AND_2
Connections:
- net ~{NO_HDMA2} is gone; now on net HDMA_EN: ROMP.2
- net wOCRQ_wOCRS_~{XIN/8}: now also ASAK.2
- net ~{INDIRECT_HDMA}: now also XPDE.1
- net at VOLG.1: now also FMKL.6 (~{Q}); no longer FMKL.7 (Q)
- net NO_HDMA: now reaches QOUI.2, ROHW.3, SBRW.2 (D), SBRW.4 (~{Q})
- net at ASDD.2, ASDM.3 (CLK), ASDM.4 (~{CLK})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: now also XPDE.2
- net GDMA_LENGTH_IS_ZERO_PULSE: now reaches ASAK.1, XPDE.2, YOJQ.7 (Q), YOXF.1, ZOED.2 (D)
- net GDMA_LENGTH_IS_ZERO_PULSE: now also ASAK.1
- net DMA_TO_BE_SERVICED: now reaches FMKL.2 (D)
- net GDMA_ON: now reaches FMKL.7 (Q), PORE.2, POSD.2
- net at BSBO.5: now also XPDE.3
- net at BSBO.9: now also ASAK.3
- net FALLING_VBLANK renamed LONG_FALLING_VBLANK
- net NO_DMA renamed NO_GDMA
- net wBSEK renamed HDMA_CHAN_RST
- net wDCBP_NOHDMA_2 renamed HDMA_EN
- net wOORF renamed ~{DMA_START_PULSE}
- net ~{DMA_START_PULSE}: now also ODNR.1 (IN), ODNR.3 (IN)
- net wPOSD renamed GDMA_TRANSFER
- net wPOSI renamed HDMA_TRANSFER
- net wROMP renamed END_HDMA
- net wSOJJ renamed ~{DMA_START_SHORT_PULSE}
- net wSOKC: no longer names the net of FMKL.2 (D), OOZO.1, POUO.2, SBRW.5 (Q), SOJJ.1
- net wTOAY renamed ENABLE_HDMA_CHANNELS
- net wUOTI renamed HDMA_ON
- net wWOEK: no longer names the net of WODN.1, WOEK.2
- net wWOEK: no longer ODNR.1 (IN), ODNR.3 (IN)
- net wWOIX renamed DISABLE_HDMA_CHANNEL
- net ~{DMA_LENGTH_IS_ZERO} renamed ~{GDMA_LENGTH_IS_ZERO}
- net ~{NO_DMA} renamed GDMA
- net ~{NO_HDMA} renamed HDMA
- net ~{STOP_DMA} renamed ~{RESTART_DMA}
- net ~{wXOGA} renamed ~{DMA_ON}
- no-connect marks 88 -> 87
Other:
- note added: "CSVJ_Q = 1 on cycle 1 or 3 during patterns that are 2 or 4 cycles long for 2 clock cycles"
- note added: "HDMA won't actually start if 420C register content is changed to 0"
- note added: "In MODE5 DMA bedugging mode: - PA0 = ~{DMA_START_PULSE} - PA1 = ~{DMA_START_SHORT_PULSE} - PA2 = GDMA_CHAN_RST - PA3 = NEXT_CHAN_CLK - PA4 = HDMA_EMPTY_SCANLINE_COUNTER - PA5 = HDMA_CHAN_RST - PA6 = DISABLE_HDMA_CHANNEL - PA7 = ~{DMA_RAM_WR}"
- note added: "POSI_Q always 0 when HDMA is not enabled. Set to 1 when HDMA becomes activa POSD_Q is the equivalent for GDMA. We can see that HDMA takes priority over GDMA but also that HDMA cannot be started when GDMA is on-going. Perhaps a safety feature? OORF goes low for 8 cycles whenever HDMA or GDMA become active"
- note added: "SKDK is 0 when the end of HDMA table is reached: i.e. HDMA Line counter and Repeat flag are all set to 0"
- note added: "SODT (~{GDMA_CHAN_RST} ~{wYOOX} On for 2 XIN cycles when GDMA length becomes 0 ~{wYOOX} On for 2 XIN cycles when GDMA length becomes 0 ~{wXOPA} On at the end of the transfer pattern ~{wZOGY}"
- note added: "SOJJ: Negative pulse at the start of a GDMA or HDMA series of transfer SOGW: Negative pulse at the end of GDMA or HDMA transfer ROMP: Negative pulse only when all HDMA channels have been serviced"
- note added: "UOCE & UOFY can only be "00", "10" or "01" but never "11" "00" during GDMA"
- note added: "negative pulse on rising edge"
- note added: "positive pulse on rising edge"
- note added: "wZOGE: Get HDMA line counter value from data bus following VBLANK falling edge or when line counter reaches 0"
- note removed: "SODT (~{GDMA_CHAN_RST} ~{wYOOX} On for 2 XIN cycles when GDMA length becomes 0 ~{wYOOX} On for 2 XIN cycles when GDMA length becomes 0 ~{wXOPA} ~{wYOGY}"
- note removed: "UOCE & UOFY can only be "00", "10" or "01" but never "11""
- moved on the sheet: FMKL, LNZS, OBEE, ODNR, OOLO, ROBA, RODU, ROHL, ROMP, RONY, SBRW, SOGW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
