File: S-CPU_kicad/DMAothers.kicad_sch (KiCad schematic)
At the start: 208 parts

Commit message: Schematics update.
Parts:
- added NBIE, OBEQ: AND_2, symbol Ricoh_Cells:AND_2
- added NBIV, NBIZ, OBHN, OBIW: DFFR_B, symbol Ricoh_Cells:DFFR_B
- added OAOU: DFFR_A, symbol Ricoh_Cells:DFFR_A
Connections:
- net LONG_FALLING_VBLANK: now also OAOU.2 (D)
- net wMAGR_wMAGV: now also NBIV.3 (CLK), NBIV.4 (~{CLK}), NBIZ.3 (CLK), NBIZ.4 (~{CLK}), OBHN.3 (CLK), OBHN.4 (~{CLK}), OBIW.3 (CLK), OBIW.4 (~{CLK})
- net wNBEB_wNBEG_XIN/8: now also OAOU.3 (CLK), OAOU.4 (~{CLK})
- net DMA_CLK renamed CPU_CLK
- net DMA_FALLING_VBLANK: no longer names the net of SOQC.2
- net DMA_FALLING_VBLANK: now also NBIE.3
- net DMA_RISING_HBLANK: no longer names the net of SOUV.2
- net DMA_RISING_HBLANK: now also OBEQ.3
- new net: OBIW.1 (~{RESET}), OBIW.5 (~{RESET})
- new net: OBEQ.1, OBHN.2 (D), OBIW.7 (Q)
- new net: NBIE.1, NBIV.2 (D), NBIZ.7 (Q)
- new net: NBIE.2, NBIV.6 (~{Q})
- new net: OAOU.1 (~{RESET}), OAOU.5 (~{RESET})
- new net: NBIZ.2 (D), OAOU.6 (Q)
- new net: NBIZ.1 (~{RESET}), NBIZ.5 (~{RESET})
- new net: OBHN.1 (~{RESET}), OBHN.5 (~{RESET})
- new net: OBEQ.2, OBHN.6 (~{Q})
- new net: NBIV.1 (~{RESET}), NBIV.5 (~{RESET})
- new net HBLANK: OBIW.2 (D)
- no-connect marks 87 -> 96
Other:
- note added: "SODT (~{GDMA_CHAN_RST} ~{wYOOX} On for 2 XIN cycles when GDMA length becomes 0 ~{wYOOX} On for 2 XIN cycles when GDMA length becomes 0 ~{wXOPA} On at the end of the transfer pattern ~{wZOGY} At the end of each HDMA channel"
- note added: "UOCE & UOFY can only be "00", "10" or "01" but never "11" "00" during GDMA "10" while HDMA channel is transferring data "01" at the end of each HDMA channel"
- note removed: "SODT (~{GDMA_CHAN_RST} ~{wYOOX} On for 2 XIN cycles when GDMA length becomes 0 ~{wYOOX} On for 2 XIN cycles when GDMA length becomes 0 ~{wXOPA} On at the end of the transfer pattern ~{wZOGY}"
- note removed: "UOCE & UOFY can only be "00", "10" or "01" but never "11" "00" during GDMA"
- company: (none) -> Author: Regis Galland
- title: (none) -> SNES S-CPU Schematics 

Commit message: Schematics tidying in progress.
Connections:
- net wDBJW_wHASI_RST renamed wDBJW_wHASI_~{RST}
Changed lines of the file:
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@@
   (title_block
     (title "SNES S-CPU Schematics ")
-    (date "2023-06-14")
+    (date "2023-10-19")
     (rev "0.1")
     (company "Author: Regis Galland")
@@
     (effects (font (size 1.27 1.27)) (justify right))
   )
-  (hierarchical_label "wDBJW_wHASI_RST" (shape input) (at 374.65 243.84 180) (fields_autoplaced)
+  (hierarchical_label "wDBJW_wHASI_~{RST}" (shape input) (at 374.65 243.84 180) (fields_autoplaced)
     (effects (font (size 1.27 1.27)) (justify right))
   )
@@
     (effects (font (size 1.27 1.27)) (justify left))
   )
-  (hierarchical_label "wDBJW_wHASI_RST" (shape input) (at 88.265 384.81 180) (fields_autoplaced)
+  (hierarchical_label "wDBJW_wHASI_~{RST}" (shape input) (at 88.265 384.81 180) (fields_autoplaced)
     (effects (font (size 1.27 1.27)) (justify right))
   )
@@
     (effects (font (size 1.27 1.27)) (justify right))
   )
-  (hierarchical_label "wDBJW_wHASI_RST" (shape input) (at 63.5 71.12 180) (fields_autoplaced)
+  (hierarchical_label "wDBJW_wHASI_~{RST}" (shape input) (at 63.5 71.12 180) (fields_autoplaced)
     (effects (font (size 1.27 1.27)) (justify right))
   )
@@
     (effects (font (size 1.27 1.27)) (justify left))
   )
-  (hierarchical_label "wDBJW_wHASI_RST" (shape input) (at -76.835 -100.33 180) (fields_autoplaced)
+  (hierarchical_label "wDBJW_wHASI_~{RST}" (shape input) (at -76.835 -100.33 180) (fields_autoplaced)
     (effects (font (size 1.27 1.27)) (justify right))
   )
@@
     (effects (font (size 1.27 1.27)) (justify left))
   )
-  (hierarchical_label "wDBJW_wHASI_RST" (shape input) (at 63.5 226.695 180) (fields_autoplaced)
+  (hierarchical_label "wDBJW_wHASI_~{RST}" (shape input) (at 63.5 226.695 180) (fields_autoplaced)
     (effects (font (size 1.27 1.27)) (justify right))
   )
@@
     (effects (font (size 1.27 1.27)) (justify right))
   )
-  (hierarchical_label "wDBJW_wHASI_RST" (shape input) (at 457.2 104.14 180) (fields_autoplaced)
+  (hierarchical_label "wDBJW_wHASI_~{RST}" (shape input) (at 457.2 104.14 180) (fields_autoplaced)
     (effects (font (size 1.27 1.27)) (justify right))
   )
@@
     (effects (font (size 1.27 1.27)) (justify right))
   )
-  (hierarchical_label "wDBJW_wHASI_RST" (shape input) (at -95.25 7.62 180) (fields_autoplaced)
+  (hierarchical_label "wDBJW_wHASI_~{RST}" (shape input) (at -95.25 7.62 180) (fields_autoplaced)
     (effects (font (size 1.27 1.27)) (justify right))
   )
@@
     (effects (font (size 1.27 1.27)) (justify right))
   )
-  (hierarchical_label "wDBJW_wHASI_RST" (shape input) (at 538.48 514.35 180) (fields_autoplaced)
+  (hierarchical_label "wDBJW_wHASI_~{RST}" (shape input) (at 538.48 514.35 180) (fields_autoplaced)
     (effects (font (size 1.27 1.27)) (justify right))
   )
@@
     (effects (font (size 1.27 1.27)) (justify right))
   )
-  (hierarchical_label "wDBJW_wHASI_RST" (shape input) (at 577.85 182.88 180) (fields_autoplaced)
+  (hierarchical_label "wDBJW_wHASI_~{RST}" (shape input) (at 577.85 182.88 180) (fields_autoplaced)
     (effects (font (size 1.27 1.27)) (justify right))
   )
@@
     (effects (font (size 1.27 1.27)) (justify right))
   )
-  (hierarchical_label "wDBJW_wHASI_RST" (shape input) (at 577.215 212.09 180) (fields_autoplaced)
+  (hierarchical_label "wDBJW_wHASI_~{RST}" (shape input) (at 577.215 212.09 180) (fields_autoplaced)
     (effects (font (size 1.27 1.27)) (justify right))
   )
