File: S-CPU_kicad/DMAothers.kicad_sch (KiCad schematic)
At the start: 215 parts

Commit message: Big update on the hierarchical sheet. DMA section update too.
Parts:
- added OCLC, OCLX: DFFR_A, symbol Ricoh_Cells:DFFR_A
- added OMRS: INVERTER_A, symbol Ricoh_Cells:INVERTER_A
- added ZOOJ: DFFR_B, symbol Ricoh_Cells:DFFR_B
Connections:
- net wUOGG: now also OCLX.2 (D)
- net wXOWO: now also ZOOJ.3 (CLK), ZOOJ.4 (~{CLK})
- net HBLANK renamed wHBLANK
- net JPO0 renamed wJPOUT0
- net JPO1 renamed wJPOUT1
- net JPO2 renamed wJPOUT2
- net VBLANK renamed wVBLANK
- net wQKAG5 renamed INDIRECT_HDMA_FLAG
- net wSKDK renamed ~{DATA_IS_ZERO}
- net wWOVT renamed CYCLE_COUNTER0
- net wWOWE renamed CYCLE_COUNTER1
- new net: OCLC.1 (~{RESET}), OCLC.5 (~{RESET})
- new net: OCLC.2 (D), OMRS.2
- new net: OCLX.1 (~{RESET}), OCLX.5 (~{RESET})
- new net: ZOOJ.1 (~{RESET}), ZOOJ.5 (~{RESET})
- new net: OMRS.1, ZOOJ.6 (~{Q})
- new net BUS_DIRECTION_FLAG: ZOOJ.2 (D)
- new net DMA_B->A: OCLC.6 (Q)
- new net wNBHJ_wNBHM_XIN/2: OCLC.3 (CLK), OCLC.4 (~{CLK}), OCLX.3 (CLK), OCLX.4 (~{CLK})
- new net ~{DMA_BUS_ON}: OCLX.6 (Q)
- no-connect marks 96 -> 100
Other:
- note added: "Valid on cycle 0-1 and 6-7"
- note added: "Valid on cycle 0-3"
- note added: "Valid on cycle 2-3"
- note added: "Valid on cycle 4-5"
- note added: "Valid on cycle 4-7"
- note added: "Valid on cycle 6-7"
- note removed: "Indirect HDMA transfer when set to 1"

Commit message: DMA section update. Fixed gate related to INC/DEC and BORROW/CARRY FLAG
Connections:
- net DMA_STEP5: now reaches FMKL.2 (D), FMKL.2 (D), FMKL.7 (Q), ZOQW.2
- net at FMKL.1 (~{RESET}), FMKL.5 (~{RESET}): no longer FMKL.7 (Q), OBEE.1
- net DMA_STEP7: now reaches FMKL.2 (D), FMKL.7 (Q)
- net DMA_STEP6: now reaches ASIK.2, BSHU.1, FMKL.2 (D), FMKL.7 (Q)
- net wVOLG renamed DMA_STEP1
- net wWPAI renamed DMA_STEP2
- net wXOWO renamed ~{DMA_STEP2}
- net wXPHM renamed DMA_STEP3
- net wYOYP renamed DMA_SYSCLK_EN
- new net: FMKL.7 (Q), OBEE.1
Other:
- moved on the sheet: ASAK, ASBC, ASBG, ASCU, ASDD, ASDM, ASFK, ASGB, ASIK, BSBOA, BSBOB, BSBOC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

Commit message: DMA section update. Found errors between some MUX and MUXI gates.
Connections:
- net BSBO_0_A1: now also BSBO.24; no longer BSBO.29
- net BSBO_1_A0: now also BSBO.29; no longer BSBO.24
- net at FMKL.1 (~{RESET}), FMKL.5 (~{RESET}): now also FMKL.7 (Q), OBEE.1
- net ~{DMA_BUS_ON} renamed HDMA_TABLE_RD
Other:
- note added: "UOCE & UOFY can only be "00", "10" or "01" but never "11" "00" during GDMA "01" during HDMA table read "10" during HDMA data transfer"
- note removed: "UOCE & UOFY can only be "00", "10" or "01" but never "11" "00" during GDMA "10" while HDMA channel is transferring data "01" at the end of each HDMA channel"
- moved on the sheet: BSBOA, BSBOB, BSBOC, FMKL, OBEE, OCLC, OCLX, ODNR, OMRS, PAWC, RONY, SOXY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

Commit message: Found issue in the HDMA section. No seems to make sense. HDMA has 2 ways to start depending on whether GDMA is currently running.
Connections:
- net at OBEE.3: now also FMKL.1 (~{RESET}), FMKL.2 (D), FMKL.5 (~{RESET}); no longer OBEE.2
- net START_HDMA: now reaches FMKL.2 (D), SONJ.1, SOPE.3
- net at SOZA.1: now also FMKL.7 (Q), SOXY.3; no longer SOXY.4
- net END_OF_TABLE: now reaches BSEK.1, FMKL.7 (Q)
- net END_HDMA renamed ~{END_HDMA}
- net wQOXN: no longer names the net of FMKL.2 (D), FMKL.7 (Q), OOLO.2
- net wROLX: no longer names the net of FMKL.3 (CLK), FMKL.4 (~{CLK}), FMKL.7 (Q)
- removed net wSOXO: FMKL.1 (~{RESET}), FMKL.2 (D), FMKL.5 (~{RESET}), FMKL.7 (Q), SOXY.3
- net wSOZA: no longer names the net of OBEE.1
- net wSOZA: now also SOXY.4; no longer SOZA.4
- new net: OBEE.2, SOZA.4
Other:
- note added: "HDMA END detection, but also stop HDMA if 420C register content is changed to 0"
- note added: "If HDMA starts when GDMA is running, it will wait for the end of the current pattern HDMA to take over. GDMA will resume at the end of HDMA."
- note removed: "HDMA won't actually start if 420C register content is changed to 0"
- moved on the sheet: FMKL, NBIE, NBIV, NBIZ, OAOU, OBEE, OBEQ, OBHN, OBIW, POGD, QOHV, QOUI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

Commit message: Further tidying of the DMA section. New sheet added dedicated to GDMA/ HDMA Start and Stop signals.
Parts:
- removed FMKL (x29), NBIV, NBIZ, OBHN, OBIW, OOBX: DFFR_B, symbol Ricoh_Cells:DFFR_B
- removed NBIE, OBEE (x3), OBEQ, POPB, POSD, SONJ, SOPE, SOUV: AND_2, symbol Ricoh_Cells:AND_2
- removed OAOU: DFFR_A, symbol Ricoh_Cells:DFFR_A
- removed OOIW, OOLO, QOUI: NOR_2, symbol Ricoh_Cells:NOR_2
- removed POGD, PORZ, RONY, SOOS, SOVA: INVERTER_A, symbol Ricoh_Cells:INVERTER_A
- removed POOO, PORE, QOHV, ROKI, SOQC: OR_2, symbol Ricoh_Cells:OR_2
- removed POUL: OR_3, symbol Ricoh_Cells:OR_3
- removed ROHW, ROME: AND_3, symbol Ricoh_Cells:AND_3
- removed SBRW (x3): DFFSR, symbol Ricoh_Cells:DFFSR
- removed SOXY, SOZA: NAND_3, symbol Ricoh_Cells:NAND_3
- added FMKL (x3): DFFR_B, symbol Ricoh_Cells:DFFR_B
Connections:
- net CYCLE_COUNTER0: now also FMKL.7 (Q)
- net CYCLE_COUNTER1: now also FMKL.7 (Q)
- net wNBEB_wNBEG_XIN/8: now also FMKL.2 (D)
- net wOBXZ_wOCHV_~{XIN/2}: now also FMKL.3 (CLK), FMKL.4 (~{CLK})
- net at WOWY.4: now also FMKL.1 (~{RESET}), FMKL.1 (~{RESET}), FMKL.5 (~{RESET}), FMKL.5 (~{RESET})
- net wVOJF renamed GDMA_PATTERN_END
- new net: FMKL.2 (D), FMKL.3 (CLK), FMKL.4 (~{CLK}), FMKL.6 (~{Q})
- new net: FMKL.3 (CLK), FMKL.4 (~{CLK}), FMKL.7 (Q)
- new net: FMKL.1 (~{RESET}), FMKL.5 (~{RESET})
- new net: FMKL.2 (D), FMKL.6 (~{Q})
- no-connect marks 100 -> 59
Other:
- note added: "DMA RAM ADDRESS AND WRITES SIGNALS"
- note added: "OORF goes low for 8 cycles whenever HDMA or GDMA become active"
- note added: "WOVT and WOWE is a 2 bit counter for DMA transfers that deals with different patterns It gets reset at the end of each transfer pattern during GDMA and on STEP 2 during HDMA"
- note removed: "HDMA END detection, but also stop HDMA if 420C register content is changed to 0"
- note removed: "If HDMA starts when GDMA is running, it will wait for the end of the current pattern HDMA to take over. GDMA will resume at the end of HDMA."
- note removed: "POSI_Q always 0 when HDMA is not enabled. Set to 1 when HDMA becomes activa POSD_Q is the equivalent for GDMA. We can see that HDMA takes priority over GDMA but also that HDMA cannot be started when GDMA is on-going. Perhaps a safety feature? OORF goes low for 8 cycles whenever HDMA or GDMA become active"
- note removed: "SOPE goes high for a few cycles when HDMA is enabled at: - the end of VBLANK (falling edge) - the rising edge of HBLANK when VBLANK is low (i.e. during rendering)"
- note removed: "WOVT and WOWE is a 2 bit counter for DMA transfers that deals with different patterns"
- moved on the sheet: ASAK, ASCU, ASDD, ASDM, BSBOA, BSBOB, BSBOC, BSQD, BSSO, CSZL, CTBB, DTBB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

Commit message: General update a
Parts:
- removed RKUL4: TRI_BUF_IF1, symbol Ricoh_Cells:TRI_BUF_IF1
- added ODNR: TRI_BUF_IF0, symbol Ricoh_Cells:TRI_BUF_IF0
Connections:
- net DMA_STEP2: now also PAWC.4 (RESET)
- net HDMA_EMPTY_SCANLINE_COUNTER: now also ODNR.1 (IN), ODNR.3 (IN)
- net PA4: now also ODNR.4
- net ~{DMA_STEP2}: no longer PAWC.4 (RESET)
- net ~{MODE5}: now also ODNR.2 (~{ENA})
- net at ZOBY.2: now also YOXF.3; no longer YOXF.3
- net at ZOBY.3: now also YOXF.3; no longer YOXF.3
- net GET_SCANLINE_COUNTER: now reaches XOTJ.5 (Q)
- net GET_SCANLINE_COUNTER: now also FMKL.2 (D), ZOJK.3, ZONY.1
- net ~{UPDATE_SCANLINE_COUNTER}: now reaches ZOAA.2, ZOAV.2
- net wASLJ: no longer names the net of PAWC.3 (Q), ZOAV.1
- removed net wXOTJ: FMKL.2 (D), XOTJ.6 (~{Q}), ZOJK.3, ZONY.1
- net ~{GDMA_CHAN_RST} renamed ~{DMA_CHAN_RST}
Other:
- note added: "Also valid on cycle 0-2 and 7"
- note added: "OORF goes low for 4 cycles whenever HDMA or GDMA become active"
- note added: "SODT (~{DMA_CHAN_RST} ~{wYOOX} On for 2 XIN cycles when GDMA length becomes 0 ~{wYOOX} On for 2 XIN cycles when GDMA length becomes 0 ~{wXOPA} On at the end of the transfer pattern (HDMA) ~{wZOGY} At the end of each HDMA channel (end of table read?)"
- note added: "SOJJ: Negative pulse at the start of a GDMA or HDMA series of transfer This occurs because the start pulse resets SOKC and then clocks SOKC. SOGW: Negative pulse at the end of GDMA or HDMA transfer ROMP: Negative pulse only when all HDMA channels have been serviced"
- note added: "STEPS: - step 1: - read DMA RAM at address "00" i.e. DMA config, B-BUS and HDMA scanline counter - latch B-bus and DMA config registers - step 2: reset cycle counter - step 3 (second half) : latching of DMA address buses to A-BUS and B-BUS - step 3- 4: wite new HDMA scanline counter value - step 5: disable HDMA channel if counter not zero and reload flag not set"
- note added: "Text to be pasted in https://wavedrom.com/editor.html {signal: [ {name: 'xin', wave: 'n..................|....'}, {name: 'xin/2', wave: '0101010101010101010|.101'}, {name: 'xin/4', wave: '0.1.0.1.0.1.0.1.0.1|0.1.'}, {name: 'xin/8', wave: '0...1...0...1...0..|....'}, {name: 'cycle', wave: '2345678923456789234|....', data: ['0', '1', '2', '3', '4', '5', '6', '7', '0', '1', '2', '3', '4', '5', '6', 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"
- note added: "UOCE & UOFY can only be "00", "10" or "01" but never "11" "00" during GDMA "10" during HDMA table read "01" during HDMA data transfer"
- note added: "Valid on cycle 0-2 and 7"
- note added: "Valid on cycle 6-7 synchronised with step 2"
- note added: "Valid when pattern cycle = "00" or when pattern cycle /= "00" and dma cycle is 0-2 or 7"
- note added: "Write decremented HDMA scanline counter during step 3-4 ouside of VBLANK falling edge or when scanline is not 0."
- note removed: "OORF goes low for 8 cycles whenever HDMA or GDMA become active"
- note removed: "SODT (~{GDMA_CHAN_RST} ~{wYOOX} On for 2 XIN cycles when GDMA length becomes 0 ~{wYOOX} On for 2 XIN cycles when GDMA length becomes 0 ~{wXOPA} On at the end of the transfer pattern ~{wZOGY} At the end of each HDMA channel"
- note removed: "SOJJ: Negative pulse at the start of a GDMA or HDMA series of transfer SOGW: Negative pulse at the end of GDMA or HDMA transfer ROMP: Negative pulse only when all HDMA channels have been serviced"
- note removed: "UOCE & UOFY can only be "00", "10" or "01" but never "11" "00" during GDMA "01" during HDMA table read "10" during HDMA data transfer"
- note removed: "Valid on cycle 6-7"
- moved on the sheet: ASAK, ASBC, ASBG, ASCU, ASDD, ASDM, ASFK, ASGB, ASIK, BSBOA, BSBOB, BSBOC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

Commit message: HDMA section seems correct after all. More notes added.
Connections:
- net DMA_STEP2: now also PAWC.1 (SET); no longer PAWC.4 (RESET)
- net at PAWC.1 (SET): now also PAWC.4 (RESET), ZOQW.3; no longer ZONY.3
- net GET_SCANLINE_COUNTER renamed FETCH_SCANLINE_COUNTER
- net wUOGG renamed READ_HDMA_TABLE
- net wYOWZ renamed FETCH_IND_ADDR
- net wZOGE: no longer names the net of ASIK.1, BSEK.3, FMKL.7 (Q)
- net ~{DMA_CHAN_RST} renamed ~{RESET_GDMA_CHAN_STOP_DMA_CHAN}
- new net: PAWC.4 (RESET), ZONY.3
Other:
- note added: "CSVJ_Q = '1' on pattern cycle 0 or 2 and connected to ZOGY. This signal is used to end HDMA table data transfer rather than stopping normal data transfer as this is handled by XOPA. Ending on pattern cycle 0 would correspond to direct mode and cycle 2 to indirect mode."
- note added: "SODT (~{RESET_GDMA_CHAN_STOP_DMA_CHAN}) ~{wYOOX} On for 2 XIN cycles when GDMA length becomes 0 ~{wYOOX} On for 2 XIN cycles when GDMA length becomes 0 ~{wXOPA} On at the end of the data transfer pattern (HDMA) ~{wZOGY} On at the end of each table read (HDMA)"
- note added: "SOJJ: Negative pulse at the start of a GDMA or HDMA series of transfer This occurs because the start pulse resets SOKC and then clocks SOKC. SOGW: Negative pulse at the end of GDMA or HDMA transfer ROMP: Negative pulse only when all HDMA channels have been serviced Simulation shows that when VBLANK ends, HDMA will enable HDMA channels and fetch the scanline values (and the indirect 16-bit address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"
- note added: "STEPS: - step 1: - read DMA RAM at address "00" i.e. DMA config, B-BUS and HDMA scanline counter - latch B-bus and DMA config registers - step 2: - reset cycle counter - - step 3 (second half) : latching of DMA address buses to A-BUS and B-BUS - step 3- 4: wite new HDMA scanline counter value - step 5: disable HDMA channel if counter not zero and reload flag not set"
- note added: "Write decremented HDMA scanline counter during step 3-4 ouside of VBLANK falling edge or when scanline is not 0. Logic issue at the moment but perhaps ZOAV is not really there"
- note removed: "CSVJ_Q = 1 on cycle 1 or 3 during patterns that are 2 or 4 cycles long for 2 clock cycles"
- note removed: "SODT (~{DMA_CHAN_RST} ~{wYOOX} On for 2 XIN cycles when GDMA length becomes 0 ~{wYOOX} On for 2 XIN cycles when GDMA length becomes 0 ~{wXOPA} On at the end of the transfer pattern (HDMA) ~{wZOGY} At the end of each HDMA channel (end of table read?)"
- note removed: "SOJJ: Negative pulse at the start of a GDMA or HDMA series of transfer This occurs because the start pulse resets SOKC and then clocks SOKC. SOGW: Negative pulse at the end of GDMA or HDMA transfer ROMP: Negative pulse only when all HDMA channels have been serviced"
- note removed: "STEPS: - step 1: - read DMA RAM at address "00" i.e. DMA config, B-BUS and HDMA scanline counter - latch B-bus and DMA config registers - step 2: reset cycle counter - step 3 (second half) : latching of DMA address buses to A-BUS and B-BUS - step 3- 4: wite new HDMA scanline counter value - step 5: disable HDMA channel if counter not zero and reload flag not set"
- note removed: "Write decremented HDMA scanline counter during step 3-4 ouside of VBLANK falling edge or when scanline is not 0."
- moved on the sheet: ASDD, ASDM, FMKL, LNZS, ODNR, OORC, OORF, OOSR, OOZO, PAWC, POUO, RKMU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

Commit message: More DMA updates - extra notes regarding behaviour
Parts:
- YOJQ: value DFFR_B -> DFFR_C; symbol Ricoh_Cells:DFFR_B -> Ricoh_Cells:DFFR_C
Other:
- note added: "BSBO A0 0 1 0 1"
- note added: "BSBO A1 0 0 1 1"
- note added: "DMA Registers Number of Lines to Transfer (HDMA) (B0) + B Address (B2) + Parameters for DMA Transfer (B1) A Address (Low Byte) (B0) + A Address (High Byte) (B2) + A Address Bank (B1) Number Bytes to Transfer (Low Byte) (DMA) (B0) + Number Bytes to Transfer (High Byte) (DMA) (B2) + Data Bank (H-DMA) (B1) A2 Table Address (Low Byte) (B0) + A2 Table Address (High Byte) (B2) + Fast Access memory (B1)"
- note added: "HDMA STEPS: - step 1: - read DMA RAM at address "00" i.e. DMA config, B-BUS and HDMA scanline counter - latch B-bus and DMA config registers - step 2: - reset cycle counter - - step 3 (second half) : latching of DMA address buses to A-BUS and B-BUS - step 3- 4: wite new HDMA scanline counter value - step 5: disable HDMA channel if counter not zero and reload flag not set"
- note added: "Text to be pasted in https://wavedrom.com/editor.html {signal: [ {name: 'xin', wave: 'n..................|....'}, {name: 'xin/2', wave: '0101010101010101010|.101'}, {name: 'xin/4', wave: '0.1.0.1.0.1.0.1.0.1|0.1.'}, {name: 'xin/8', wave: '0...1...0...1...0..|....'}, {name: 'cycle', wave: '2345678923456789234|67x.', data: ['0', '1', '2', '3', '4', '5', '6', '7', '0', '1', '2', '3', '4', '5', '6', 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"
- note added: "UOCE & UOFY can only be "00", "10" or "01" but never "11" "00" during GDMA data transfer "10" during HDMA table read and during GDMA initialisation to acquire DMA settings "01" during HDMA data transfer"
- note added: "WOCA ~{BANK0_WR} Not allowed Allowed Allowed Allowed"
- note added: "When GDMA starts, YOJQ is set to '1' via its set input (might be the only cell in the whole chip) which will force DMA RAM address to "00" for 8 cycles from cycle 0-7. During this time, it will read the DMA settings as well as the B-bus. GMDA does not use bank 0 data as it is only used by HDMA. It will then the A-bus address during cycle 0-3 and then the length counter during cycle 4-7 until the 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"
- note added: "Write can only occur on cycle 3 and 7"
- note added: "XOAO ~{BANK2_WR} Allowed Allowed Allowed Allowed"
- note added: "YOJQ is not the right type of gate"
- note removed: "STEPS: - step 1: - read DMA RAM at address "00" i.e. DMA config, B-BUS and HDMA scanline counter - latch B-bus and DMA config registers - step 2: - reset cycle counter - - step 3 (second half) : latching of DMA address buses to A-BUS and B-BUS - step 3- 4: wite new HDMA scanline counter value - step 5: disable HDMA channel if counter not zero and reload flag not set"
- note removed: "Text to be pasted in https://wavedrom.com/editor.html {signal: [ {name: 'xin', wave: 'n..................|....'}, {name: 'xin/2', wave: '0101010101010101010|.101'}, {name: 'xin/4', wave: '0.1.0.1.0.1.0.1.0.1|0.1.'}, {name: 'xin/8', wave: '0...1...0...1...0..|....'}, {name: 'cycle', wave: '2345678923456789234|....', data: ['0', '1', '2', '3', '4', '5', '6', '7', '0', '1', '2', '3', '4', '5', '6', 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"
- note removed: "UOCE & UOFY can only be "00", "10" or "01" but never "11" "00" during GDMA "10" during HDMA table read "01" during HDMA data transfer"
- moved on the sheet: ASAK, ASBC, ASBG, ASCU, ASDD, ASDM, ASFK, ASGB, ASIK, BSBOA, BSBOB, BSBOC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
