File: S-CPU_kicad/DMAothers.kicad_sch (KiCad schematic)
At the start: 156 parts

Commit message: Identified some DFFs as being DFFs with SET input rather than RESET input. It helps explaining a lot of beahiour in the MUL/DIV section and in the DMA section.
Parts:
- ASDM, FMKL, ZOOJ: value DFFR_B -> DFFR_D; symbol Ricoh_Cells:DFFR_B -> Ricoh_Cells:DFFR_D
Connections:
- net DMA_SYSCLK_EN: now also FMKL.8 (Q); no longer FMKL.7 (Q)
- net END_OF_TABLE: now also FMKL.8 (Q); no longer FMKL.7 (Q)
- net FETCH_IND_ADDR: now also FMKL.8 (Q); no longer FMKL.7 (Q)
- net wNAQE_wNBBM_XIN/2: now also FMKL.1 (CLK), FMKL.1 (CLK), FMKL.1 (CLK), FMKL.1 (CLK); no longer FMKL.3 (CLK), FMKL.3 (CLK), FMKL.3 (CLK), FMKL.3 (CLK), FMKL.4 (~{CLK}), FMKL.4 (~{CLK}), FMKL.4 (~{CLK}), FMKL.4 (~{CLK})
- net wNBEB_wNBEG_XIN/8: now also FMKL.1 (CLK), FMKL.1 (CLK), FMKL.1 (CLK); no longer FMKL.3 (CLK), FMKL.3 (CLK), FMKL.3 (CLK), FMKL.4 (~{CLK}), FMKL.4 (~{CLK}), FMKL.4 (~{CLK})
- net wNBKW_wNBPG_~{XIN/4}: now also FMKL.1 (CLK); no longer FMKL.3 (CLK), FMKL.4 (~{CLK})
- net wOACU_wOAFI_XIN/4: now also FMKL.1 (CLK), FMKL.1 (CLK), FMKL.1 (CLK); no longer FMKL.3 (CLK), FMKL.3 (CLK), FMKL.3 (CLK), FMKL.4 (~{CLK}), FMKL.4 (~{CLK}), FMKL.4 (~{CLK})
- net wOBXZ_wOCHV_~{XIN/2}: now also ASDM.1 (CLK), FMKL.1 (CLK), FMKL.1 (CLK); no longer ASDM.3 (CLK), ASDM.4 (~{CLK}), FMKL.3 (CLK), FMKL.3 (CLK), FMKL.4 (~{CLK}), FMKL.4 (~{CLK})
- net ~{DMA_STEP2}: now also ZOOJ.1 (CLK); no longer ZOOJ.3 (CLK), ZOOJ.4 (~{CLK})
- net ~{INDIRECT_HDMA}: now also ASDM.8 (Q); no longer ASDM.7 (Q)
- net at ASDM.7 (~{Q}): no longer YOLV.1
- net at FMKL.7 (~{Q}): no longer XOIL.1
- net at XOMS.1, XONF.1: now also FMKL.8 (Q); no longer FMKL.7 (Q)
- net at ASDD.2, BSBO.11, XPDE.2: now also ASDM.1 (CLK); no longer ASDM.3 (CLK), ASDM.4 (~{CLK})
- net at UOGG.1: now also FMKL.8 (Q); no longer FMKL.7 (Q)
- net at FMKL.3 (CLK), FMKL.4 (~{CLK}): now also FMKL.8 (Q); no longer FMKL.7 (Q)
- net at FMKL.7 (~{Q}): no longer BSEK.2
- net at ASIK.1, BSEK.3: now also FMKL.8 (Q); no longer FMKL.7 (Q)
- net at OOSR.2: now also FMKL.7 (~{Q}); no longer FMKL.6 (~{Q})
- net at UOKI.1: now also FMKL.8 (Q); no longer FMKL.7 (Q)
- net at FMKL.1 (CLK): now also BSHU.2; no longer FMKL.5 (~{RESET})
- net at ROBA.1: now also FMKL.7 (~{Q}); no longer FMKL.6 (~{Q})
- net at OMRS.1: now also ZOOJ.7 (~{Q}); no longer ZOOJ.6 (~{Q})
- net at OORC.1: now also FMKL.7 (~{Q}); no longer FMKL.6 (~{Q})
- net at ASGB.2: now also FMKL.7 (~{Q}); no longer FMKL.6 (~{Q})
- net at ASGB.3: now also FMKL.8 (Q); no longer FMKL.7 (Q)
- new net: ASDM.8 (Q), YOLV.1
- new net: FMKL.8 (Q), XOIL.1
- new net: BSEK.2, FMKL.8 (Q)
- no-connect marks 59 -> 42
Other:
- note added: "POSI (HDMA transfer) 0 0 1 1"
- note added: "SODT (~{RESET_GDMA_CHAN_STOP_DMA_CHAN}) wYOOX On for 2 XIN cycles when GDMA length becomes 0 wYOOX On for 2 XIN cycles when GDMA length becomes 0 wXOPA On at the end of the data transfer pattern (HDMA) wZOGY On at the end of each table read (HDMA)"
- note added: "UOCE & UOFY "00" "00" "01" "10""
- note added: "WOCA ~{BANK0_WR} Allowed Allowed Allowed Allowed"
- note added: "XOAO ~{BANK2_WR} Not allowed Allowed Allowed Allowed"
- note removed: "POSI 0 0 1 1"
- note removed: "SODT (~{RESET_GDMA_CHAN_STOP_DMA_CHAN}) ~{wYOOX} On for 2 XIN cycles when GDMA length becomes 0 ~{wYOOX} On for 2 XIN cycles when GDMA length becomes 0 ~{wXOPA} On at the end of the data transfer pattern (HDMA) ~{wZOGY} On at the end of each table read (HDMA)"
- note removed: "UOCE & UOFY can only be "00", "10" or "01" but never "11" "00" during GDMA data transfer "10" during HDMA table read and during GDMA initialisation to acquire DMA settings "01" during HDMA data transfer"
- note removed: "WOCA ~{BANK0_WR} Not allowed Allowed Allowed Allowed"
- note removed: "XOAO ~{BANK2_WR} Allowed Allowed Allowed Allowed"
- note removed: "YOJQ is not the right type of gate"

Commit message: Fix ERC errors in schematics.
Connections:
- net CYCLE_COUNTER0 renamed PATTERN_COUNTER0
- net CYCLE_COUNTER1 renamed PATTERN_COUNTER1
Other:
- note added: "HDMA STEPS: - step 1: - read DMA RAM at address "00" i.e. DMA config, B-BUS and HDMA scanline counter - latch B-bus and DMA config registers - step 2: - reset pattern counter - - step 3 (second half) : latching of DMA address buses to A-BUS and B-BUS - step 3- 4: wite new HDMA scanline counter value - step 5: disable HDMA channel if counter not zero and reload flag not set"
- note removed: "HDMA STEPS: - step 1: - read DMA RAM at address "00" i.e. DMA config, B-BUS and HDMA scanline counter - latch B-bus and DMA config registers - step 2: - reset cycle counter - - step 3 (second half) : latching of DMA address buses to A-BUS and B-BUS - step 3- 4: wite new HDMA scanline counter value - step 5: disable HDMA channel if counter not zero and reload flag not set"
- title: SNES S-CPU Schematics  -> Reverse Engineered SNES S-CPU Schematics 
- moved on the sheet: FMKL, ODNR, OOZO, POUO, SODT, UOKI, UONJ, XOIL, XOKS, XOMS, XONF

Commit message: More notes added to detail HDMA steps
Connections:
- net DMA_STEP5: no longer ZOQW.2
- net FETCH_SCANLINE_COUNTER: now also ZOQW.2
- net ~{DMA_STEP1}: now reaches ASDD.2, ASDM.1 (CLK), BSBO.11, XPDE.2
- net at PAWC.4 (RESET), ZOQW.3: now also PAWC.4 (RESET); no longer PAWC.1 (SET)
- net at ZONY.3: now also PAWC.1 (SET); no longer PAWC.4 (RESET)
Other:
- note added: "HDMA STEPS GENERATOR"
- note added: "In MODE5 DMA bedugging mode: - PA0 = ~{DMA_START_PULSE} - PA1 = ~{DMA_START_SHORT_PULSE} - PA2 = GDMA_CHAN_RST - PA3 = NEXT_CHAN_CLK - PA4 = HDMA_EMPTY_SCANLINE_COUNTER - PA5 = HDMA_CHAN_RST - PA6 = DISABLE_HDMA_CHANNEL - PA7 = ~{DMA_RAM_WR} - JPOUT0 = DMA_CLK_EN - JPOUT1 = DMA RAM A0 - JPOUT2 = DMA RAM A1"
- note added: "On NEXT_CHAN_CLK rising edge, a 2 Xin pulse is generated and goes through a shift register clocked at XIN/2 which defines HDMA steps to sequence its behaviour. From current findings, the DMA steps are: - step 1: - read DMA RAM at address "00" i.e. DMA config (Bank 1), B-BUS (Bank 2) and HDMA scanline counter (Bank 0) - latch B-bus and DMA config registers - step 2: - reset pattern counter - latch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"
- note added: "PA0"
- note added: "PA1"
- note added: "PA2"
- note added: "PA3"
- note added: "PA4"
- note added: "PA5"
- note added: "PA6"
- note added: "PA7"
- note added: "When GDMA starts, YOJQ is set to '1' via its set input (might be the only cell in the whole chip) which will force DMA RAM address to "00" for 8 cycles from cycle 0-7. During this time, it will read the DMA settings as well as the B-bus. GMDA does not use bank 0 data as it is only used by HDMA. It will then read the A-bus address during cycle 0-3 and then the length counter during cycle 4-7 until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"
- note added: "Write decremented HDMA scanline counter during step 3-4 ouside of VBLANK falling edge or when scanline is not 0."
- note added: "wZOGE: Get HDMA line counter value from data bus following VBLANK falling edge or when line counter reaches 0 during cycle 4-7 wCSGZ and wCSDS will be 0 during HDMA transfer which will update the incremented indirect address saved in DMA RAM (indirect HDMA?)."
- note removed: "HDMA STEPS: - step 1: - read DMA RAM at address "00" i.e. DMA config, B-BUS and HDMA scanline counter - latch B-bus and DMA config registers - step 2: - reset pattern counter - - step 3 (second half) : latching of DMA address buses to A-BUS and B-BUS - step 3- 4: wite new HDMA scanline counter value - step 5: disable HDMA channel if counter not zero and reload flag not set"
- note removed: "In MODE5 DMA bedugging mode: - PA0 = ~{DMA_START_PULSE} - PA1 = ~{DMA_START_SHORT_PULSE} - PA2 = GDMA_CHAN_RST - PA3 = NEXT_CHAN_CLK - PA4 = HDMA_EMPTY_SCANLINE_COUNTER - PA5 = HDMA_CHAN_RST - PA6 = DISABLE_HDMA_CHANNEL - PA7 = ~{DMA_RAM_WR}"
- note removed: "When GDMA starts, YOJQ is set to '1' via its set input (might be the only cell in the whole chip) which will force DMA RAM address to "00" for 8 cycles from cycle 0-7. During this time, it will read the DMA settings as well as the B-bus. GMDA does not use bank 0 data as it is only used by HDMA. It will then the A-bus address during cycle 0-3 and then the length counter during cycle 4-7 until the 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"
- note removed: "Write decremented HDMA scanline counter during step 3-4 ouside of VBLANK falling edge or when scanline is not 0. Logic issue at the moment but perhaps ZOAV is not really there"
- note removed: "wZOGE: Get HDMA line counter value from data bus following VBLANK falling edge or when line counter reaches 0"
- moved on the sheet: ASAK, ASBC, ASBG, ASCU, ASDD, ASDM, ASFK, ASGB, ASIK, BSBOA, BSBOB, BSBOC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

Commit message: Big rework on the hierachical sheet to make thigs a bit clearer. PDF exported for Rev 0.1.
Parts:
- renumbered ASAK to ASAR, XPDE to ASEA, PAWC to ASLJ, FMKL to ASMG, FMKL to ASMP, CSZL to ASMS, CTBB to ASNP, YOLV to BSCX, ODNR to BSDK, FMKL to BSGB, FMKL to BSKW, FMKL to BSOQ, ODNR to CSAH, ODNR to CSBF, YOXF to CSCY, ASDM to CSMN, ASDM to CSMX, ASDM to CSMZ, ASDM to CSQI, ASDM to CSVJ, ASDD to DTEU, ZODY to DTIH, ZODY to DTJZ, ASDD to DTNW, YOLV to DTQU, ASDD to DTRS, ODNR to DTTS, FMKL to OONQ, FMKL to OOXS, FMKL to ROAW, FMKL to ROBL, FMKL to ROEI, SBRW to SOKC, FMKL to VOAT, FMKL to VOBM, FMKL to VODK, FMKL to VOEX, FMKL to VOGQ, FMKL to VOKG, ODNR to VONZ, ODNR to WOEU, YOLV to WOIX, ODNR to WOJX, ODNR to WOKW, ODNR to WOME, ODNR to WOML, ODNR to WOSL, FMKL to WOVT, FMKL to WOWE, FMKL to WPAI, FMKL to XOFC, YOLV to XOPA, PAWC to XOVF, ASAK to XPDO, ODNR to XPGS, FMKL to XPHM, ODNR to YOAC, YOXF to YOEH, YOXF to YOFK, ODNR to YOQY, FMKL to YOWZ, FMKL to YOYP, FMKL to YOZV, FMKL to ZOGE, YOLV to ZOGY, FMKL to ZORH, BSQD to ZOSP, BSSO to ZOYR
Connections:
- net DMA_B->A: now also OCLC.9 (Q); no longer OCLC.6 (Q)
- net DMA_ON: now also XOFC.6 (~{RESET}); no longer XOFC.1 (~{RESET}), XOFC.5 (~{RESET})
- net DMA_STEP2: now also WPAI.9 (Q); no longer WPAI.7 (Q)
- net DMA_STEP3: now also XPHM.9 (Q); no longer XPHM.7 (Q)
- net DMA_STEP5: now also ZORH.9 (Q); no longer ZORH.7 (Q)
- net DMA_STEP6: now also ASMP.9 (Q); no longer ASMP.7 (Q)
- net DMA_STEP7: now also BSOQ.9 (Q); no longer BSOQ.7 (Q)
- net GDMA_LENGTH_IS_ZERO_PULSE: now also YOJQ.9 (Q); no longer YOJQ.7 (Q)
- net HDMA_TABLE_RD: now also OCLX.9 (Q); no longer OCLX.6 (Q)
- net PATTERN_COUNTER0: now also WOVT.9 (Q); no longer WOVT.7 (Q)
- net PATTERN_COUNTER1: now also WOWE.9 (Q); no longer WOWE.7 (Q)
- net ~{DMA_ON}: now also XOGA.8 (~{Q}); no longer XOGA.6 (~{Q})
- net ~{wCSMZ}: now also CSMZ.8 (~{Q}); no longer CSMZ.6 (~{Q})
- net ~{wCSQI}: now also CSQI.8 (~{Q}); no longer CSQI.6 (~{Q})
- net at VOLG.1: now also VOKG.8 (~{Q}); no longer VOKG.6 (~{Q})
- net at ZORH.2 (D): now also YOZV.9 (Q); no longer YOZV.7 (Q)
- net ~{MRST}: now reaches ZORH.6 (~{RESET})
- net ~{MRST}: now also ASMP.6 (~{RESET}), BSOQ.6 (~{RESET}), ROBL.6 (~{RESET}), ROEI.6 (~{RESET}), SOGE.2, SOKC.4 (~{SET}), VOKG.6 (~{RESET}), WOWY.1, WPAI.6 (~{RESET}), XOFV.1, XOTJ.4 (~{RESET}), XPHM.6 (~{RESET}), YOZV.6 (~{RESET}), ZORE.1
- net at ASCU.6 (~{RESET}): now also TODR.3, YOJQ.6 (~{SET})
- net at YOOX.2: now also ASCU.9 (Q); no longer ASCU.7 (Q)
- net DMA_~{XIN/2}: now reaches CSMZ.1 (CLK)
- net DMA_~{XIN/2}: now also ASMP.1 (CLK), BSOQ.1 (CLK), CSMN.1 (CLK), CSMX.1 (CLK), CSQI.1 (CLK), CSVJ.1 (CLK), ROAW.1 (CLK), ROBL.1 (CLK), ROEI.1 (CLK), VOGQ.1 (CLK), VOKG.1 (CLK), WPAI.1 (CLK), XOFC.1 (CLK), XPHM.1 (CLK), YOCE.3, YOZV.1 (CLK), ZORH.1 (CLK); no longer CSMZ.5 (~{RESET})
- net XIN/2: now reaches OCLC.1 (CLK)
- net XIN/2: now also OCLX.1 (CLK); no longer OCLC.5 (~{RESET})
- net at ROHL.1: now also ROEI.8 (~{Q}); no longer ROEI.6 (~{Q})
- net at ZOGY.2: now also CSVJ.9 (Q); no longer CSVJ.7 (Q)
- net at OOZO.1, POUO.2, SOJJ.1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: now also SOKC.11 (Q); no longer SOKC.5 (Q)
- net at WODN.2: now also XOFC.8 (~{Q}); no longer XOFC.6 (~{Q})
- net at ZODY.1: now also ZOED.9 (Q); no longer ZOED.7 (Q)
- net at TODR.2, XOFV.3: now also XOGA.6 (~{RESET}); no longer XOGA.1 (~{RESET}), XOGA.5 (~{RESET})
- net at RODU.1: now also ROBL.9 (Q); no longer ROBL.7 (Q)
- net at SOGW.1: now also SOKC.9 (~{Q}); no longer SOKC.4 (~{Q})
- net at SOLZ.2: now also SOKC.7 (~{RESET}); no longer SOKC.6 (~{RESET})
- net at ROHL.3, SOGW.2, SOJJ.2: now also SOKC.1 (CLK); no longer SOKC.7 (CLK)
- net DMA_XIN/8: now reaches ZOED.1 (CLK)
- net DMA_XIN/8: now also ASAK.2, DTEU.1, DTSJ.3 (2), OONQ.1 (CLK), OOXS.1 (CLK), VOGQ.2 (D), VOJL.1, YOEH.2, ZOGE.1 (CLK); no longer ZOED.5 (~{RESET})
- net at BSSO.1: now also CSMX.9 (Q); no longer CSMX.7 (Q)
- net at WOWE.6 (~{RESET}): now also WOVT.6 (~{RESET}), WOWY.4; no longer WOWE.2 (D)
- removed net wDBJW_wHASI_~{RST}: ASMP.1 (~{RESET}), ASMP.5 (~{RESET}), BSOQ.1 (~{RESET}), BSOQ.5 (~{RESET}), ROBL.1 (~{RESET}), ROBL.5 (~{RESET}), ROEI.1 (~{RESET}), ROEI.5 (~{RESET}), SOGE.2, SOKC.1 (~{SET}), SOKC.3 (~{SET}), VOKG.1 (~{RESET}), VOKG.5 (~{RESET}), WOWY.1, WPAI.1 (~{RESET}), WPAI.5 (~{RESET}), XOFV.1, XOTJ.4 (~{RESET}), XPHM.1 (~{RESET}), XPHM.5 (~{RESET}), YOZV.1 (~{RESET}), YOZV.5 (~{RESET}), ZORE.1, ZORH.1 (~{RESET}), ZORH.5 (~{RESET})
- net wNAQE_wNBBM_XIN/2 renamed DMA_XIN/2
- removed net wNBEB_wNBEG_XIN/8: ASAK.2, DTEU.1, DTSJ.3 (2), OONQ.1 (CLK), OOXS.1 (CLK), VOGQ.2 (D), VOJL.1, YOEH.2, ZOED.3 (CLK), ZOED.4 (~{CLK}), ZOGE.1 (CLK)
- removed net wNBHJ_wNBHM_XIN/2: OCLC.3 (CLK), OCLC.4 (~{CLK}), OCLX.3 (CLK), OCLX.4 (~{CLK})
- net wNBKW_wNBPG_~{XIN/4} renamed DMA_~{XIN/4}
- net wOACU_wOAFI_XIN/4 renamed DMA_XIN/4
- removed net wOBXZ_wOCHV_~{XIN/2}: ASMP.3 (CLK), ASMP.4 (~{CLK}), BSOQ.3 (CLK), BSOQ.4 (~{CLK}), CSMN.1 (CLK), CSMX.3 (CLK), CSMX.4 (~{CLK}), CSMZ.3 (CLK), CSMZ.4 (~{CLK}), CSQI.3 (CLK), CSQI.4 (~{CLK}), CSVJ.3 (CLK), CSVJ.4 (~{CLK}), ROAW.1 (CLK), ROBL.3 (CLK), ROBL.4 (~{CLK}), ROEI.3 (CLK), ROEI.4 (~{CLK}), VOGQ.1 (CLK), VOKG.3 (CLK), VOKG.4 (~{CLK}), WPAI.3 (CLK), WPAI.4 (~{CLK}), XOFC.3 (CLK), XOFC.4 (~{CLK}), XPHM.3 (CLK), XPHM.4 (~{CLK}), YOCE.3, YOZV.3 (CLK), YOZV.4 (~{CLK}), ZORH.3 (CLK), ZORH.4 (~{CLK})
- net wOCRQ_wOCRS_~{XIN/8} renamed DMA_~{XIN/8}
- new net: ASCU.1 (CLK), XOGA.1 (CLK), YOJQ.1 (CLK), YOLV.3
- new net: VOGQ.8 (Q), WOVT.1 (CLK)
- new net: WOVT.2 (D), WOVT.8 (~{Q}), WOWE.1 (CLK)
- new net: WOWE.2 (D), WOWE.8 (~{Q})

Commit message: Fixed VAWR which should have been an SR DFF (to fix issue #3 raised in github)
Parts:
- BSEK, WOWY: value AND_2 -> AND_3
Connections:
- net DISABLE_HDMA_CHANNEL renamed PAUSE_HDMA_CHAN
- net HDMA_CHAN_RST renamed STOP_HDMA_CHAN
Other:
- note added: "HDMA is paused when no data transfer is needed which occurs on step 5 when scanline counter is greater than 0 and reload flag is off."
- note added: "In MODE5 DMA bedugging mode: - PA0 = ~{DMA_START_PULSE} - PA1 = ~{DMA_START_SHORT_PULSE} - PA2 = GDMA_CHAN_RST - PA3 = NEXT_CHAN_CLK - PA4 = HDMA_EMPTY_SCANLINE_COUNTER - PA5 = STOP_HDMA_CHAN - PA6 = PAUSE_HDMA_CHAN - PA7 = ~{DMA_RAM_WR} - JPOUT0 = DMA_CLK_EN - JPOUT1 = DMA RAM A0 - JPOUT2 = DMA RAM A1"
- note removed: "In MODE5 DMA bedugging mode: - PA0 = ~{DMA_START_PULSE} - PA1 = ~{DMA_START_SHORT_PULSE} - PA2 = GDMA_CHAN_RST - PA3 = NEXT_CHAN_CLK - PA4 = HDMA_EMPTY_SCANLINE_COUNTER - PA5 = HDMA_CHAN_RST - PA6 = DISABLE_HDMA_CHANNEL - PA7 = ~{DMA_RAM_WR} - JPOUT0 = DMA_CLK_EN - JPOUT1 = DMA RAM A0 - JPOUT2 = DMA RAM A1"
