File: S-CPU_kicad/clocks.kicad_sch (KiCad schematic)
At the start: 138 parts

Commit message: Schematics tidying in progress.
Parts:
- removed GBEG: OR_3, symbol Ricoh_Cells:OR_3
Connections:
- net wDBJW_wHASI_RST renamed wDBJW_wHASI_~{RST}
- net wKBNZ renamed wACLK
Changed lines of the file:
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@@
   (title_block
     (title "SNES S-CPU Schematics ")
-    (date "2023-06-14")
+    (date "2023-10-19")
     (rev "0.1")
     (company "Author: Regis Galland")
@@
   (junction (at 374.65 442.595) (diameter 0) (color 0 0 0 0)
   )
-  (junction (at 192.405 80.645) (diameter 0) (color 0 0 0 0)
-  )
   (junction (at 320.675 514.985) (diameter 0) (color 0 0 0 0)
   )
@@
     (stroke (width 0) (type default))
   )
-  (wire (pts (xy 186.055 80.645) (xy 192.405 80.645))
-    (stroke (width 0) (type default))
-  )
   (wire (pts (xy 490.855 359.41) (xy 490.855 383.54))
     (stroke (width 0) (type default))
@@
     (stroke (width 0) (type default))
   )
-  (wire (pts (xy 170.815 78.105) (xy 149.86 78.105))
-    (stroke (width 0) (type default))
-  )
   (wire (pts (xy 360.68 85.725) (xy 363.22 85.725))
     (stroke (width 0) (type default))
@@
     (stroke (width 0) (type default))
   )
-  (wire (pts (xy 149.86 83.185) (xy 170.815 83.185))
-    (stroke (width 0) (type default))
-  )
   (wire (pts (xy 163.83 158.115) (xy 171.45 158.115))
     (stroke (width 0) (type default))
@@
     (stroke (width 0) (type default))
   )
-  (wire (pts (xy 192.405 80.645) (xy 192.405 73.025))
-    (stroke (width 0) (type default))
-  )
   (wire (pts (xy 600.71 347.98) (xy 609.6 347.98))
     (stroke (width 0) (type default))
@@
     (stroke (width 0) (type default))
   )
-  (wire (pts (xy 192.405 73.025) (xy 205.105 73.025))
-    (stroke (width 0) (type default))
-  )
   (wire (pts (xy 372.11 508.635) (xy 377.19 508.635))
     (stroke (width 0) (type default))
@@
     (stroke (width 0) (type default))
   )
-  (wire (pts (xy 530.86 241.3) (xy 561.975 241.3))
+  (wire (pts (xy 530.86 241.3) (xy 537.21 241.3))
     (stroke (width 0) (type default))
   )
@@
     (stroke (width 0) (type default))
   )
-  (wire (pts (xy 149.86 80.645) (xy 170.815 80.645))
-    (stroke (width 0) (type default))
-  )
   (wire (pts (xy 368.3 287.655) (xy 368.3 277.495))
     (stroke (width 0) (type default))
@@
     (effects (font (size 1.27 1.27)) (justify right bottom))
   )
-  (label "wDBJW_wHASI_RST" (at 228.6 281.94 0) (fields_autoplaced)
+  (label "wDBJW_wHASI_~{RST}" (at 228.6 281.94 0) (fields_autoplaced)
     (effects (font (size 1.27 1.27)) (justify left bottom))
   )
@@
     (effects (font (size 1.27 1.27)) (justify left bottom))
   )
-  (label "wDBJW_wHASI_RST" (at 349.25 553.72 0) (fields_autoplaced)
+  (label "wDBJW_wHASI_~{RST}" (at 349.25 553.72 0) (fields_autoplaced)
     (effects (font (size 1.27 1.27)) (justify left bottom))
   )
@@
     (effects (font (size 1.27 1.27)) (justify right bottom))
   )
-  (label "wDBJW_wHASI_RST" (at 260.35 374.65 180) (fields_autoplaced)
+  (label "wDBJW_wHASI_~{RST}" (at 260.35 374.65 180) (fields_autoplaced)
     (effects (font (size 1.27 1.27)) (justify right bottom))
   )
@@
     (effects (font (size 1.27 1.27)) (justify left bottom))
   )
-  (label "SYNCED_REFRESH_EN" (at 149.86 78.105 0) (fields_autoplaced)
-    (effects (font (size 1.27 1.27)) (justify left bottom))
-  )
   (label "~{420D_WR}" (at 213.36 163.195 0) (fields_autoplaced)
     (effects (font (size 1.27 1.27)) (justify left bottom))
@@
     (effects (font (size 1.27 1.27)) (justify left bottom))
   )
-  (label "wDBJW_wHASI_RST" (at 427.355 203.2 0) (fields_autoplaced)
+  (label "wDBJW_wHASI_~{RST}" (at 427.355 203.2 0) (fields_autoplaced)
     (effects (font (size 1.27 1.27)) (justify left bottom))
   )
@@
     (effects (font (size 1.27 1.27)) (justify left bottom))
   )
-  (label "wDBJW_wHASI_RST" (at 203.2 186.055 0) (fields_autoplaced)
+  (label "wDBJW_wHASI_~{RST}" (at 203.2 186.055 0) (fields_autoplaced)
     (effects (font (size 1.27 1.27)) (justify left bottom))
   )
@@
     (effects (font (size 1.27 1.27)) (justify left bottom))
   )
-  (label "wDBJW_wHASI_RST" (at 407.035 439.42 0) (fields_autoplaced)
+  (label "wDBJW_wHASI_~{RST}" (at 407.035 439.42 0) (fields_autoplaced)
     (effects (font (size 1.27 1.27)) (justify left bottom))
   )
@@
     (effects (font (size 1.27 1.27)) (justify left bottom))
   )
-  (label "wDBJW_wHASI_RST" (at 335.915 121.92 0) (fields_autoplaced)
+  (label "wDBJW_wHASI_~{RST}" (at 335.915 121.92 0) (fields_autoplaced)
     (effects (font (size 1.27 1.27)) (justify left bottom))
   )
@@
     (effects (font (size 1.27 1.27)) (justify left bottom))
   )
-  (label "SYNCED_REFRESH_EN" (at 561.975 241.3 180) (fields_autoplaced)
-    (effects (font (size 1.27 1.27)) (justify right bottom))
-  )
   (label "4000-41FF" (at 296.545 107.315 0) (fields_autoplaced)
     (effects (font (size 1.27 1.27)) (justify left bottom))
@@
     (effects (font (size 1.27 1.27)) (justify left bottom))
   )
-  (label "wDBJW_wHASI_RST" (at 339.725 287.655 0) (fields_autoplaced)
+  (label "wDBJW_wHASI_~{RST}" (at 339.725 287.655 0) (fields_autoplaced)
     (effects (font (size 1.27 1.27)) (justify left bottom))
   )
+  (hierarchical_label "DMA_ON" (shape input) (at 594.36 224.79 180) (fields_autoplaced)
+    (effects (font (size 1.27 1.27)) (justify right))
+  )
   (hierarchical_label "wOACU_wOAFI_XIN{slash}4" (shape output) (at 571.5 356.87 0) (fields_autoplaced)
     (effects (font (size 1.27 1.27)) (justify left))
   )
+  (hierarchical_label "SYNCED_REFRESH_EN" (shape output) (at 537.21 241.3 0) (fields_autoplaced)
+    (effects (font (size 1.27 1.27)) (justify left))
+  )
   (hierarchical_label "wOBXZ_wOCHV_~{XIN{slash}2}" (shape output) (at 571.5 337.82 0) (fields_autoplaced)
     (effects (font (size 1.27 1.27)) (justify left))
@@
     (effects (font (size 1.27 1.27)) (justify left))
   )
-  (hierarchical_label "MODE2_OR_MODE3" (shape input) (at 149.86 83.185 180) (fields_autoplaced)
-    (effects (font (size 1.27 1.27)) (justify right))
-  )
-  (hierarchical_label "wDBJW_wHASI_RST" (shape output) (at 260.35 374.65 0) (fields_autoplaced)
+  (hierarchical_label "wDBJW_wHASI_~{RST}" (shape output) (at 260.35 374.65 0) (fields_autoplaced)
     (effects (font (size 1.27 1.27)) (justify left))
   )
@@
     (effects (font (size 1.27 1.27)) (justify left))
   )
-  (hierarchical_label "~{INTERNAL_CYCLE}" (shape input) (at 149.86 80.645 180) (fields_autoplaced)
-    (effects (font (size 1.27 1.27)) (justify right))
-  )
   (hierarchical_label "wIAYI" (shape output) (at 236.855 358.775 0) (fields_autoplaced)
     (effects (font (size 1.27 1.27)) (justify left))
@@
     (effects (font (size 1.27 1.27)) (justify left))
   )
-  (hierarchical_label "RW_EN" (shape output) (at 205.105 73.025 0) (fields_autoplaced)
-    (effects (font (size 1.27 1.27)) (justify left))
+  (hierarchical_label "RW_EN" (shape input) (at 192.405 80.645 180) (fields_autoplaced)
+    (effects (font (size 1.27 1.27)) (justify right))
   )
   (hierarchical_label "wNBKW_wNBPG_~{XIN{slash}4}" (shape output) (at 571.5 382.27 0) (fields_autoplaced)
     (effects (font (size 1.27 1.27)) (justify left))
   )
-  (hierarchical_label "wKBNZ" (shape output) (at 573.405 83.185 0) (fields_autoplaced)
+  (hierarchical_label "wACLK" (shape output) (at 573.405 83.185 0) (fields_autoplaced)
+    (effects (font (size 1.27 1.27)) (justify left))
+  )
+  (hierarchical_label "~{XIN1}" (shape output) (at 445.77 354.33 0) (fields_autoplaced)
     (effects (font (size 1.27 1.27)) (justify left))
   )
@@
         )
       )
-    )
-  )
-  (symbol (lib_id "Ricoh_Cells:OR_3") (at 178.435 80.645 0) (unit 1)
-    (in_bom yes) (on_board yes) (dnp no) (fields_autoplaced)
-    (property "Reference" "GBEG" (at 178.4348 73.8251 0)
-      (effects (font (size 1.27 1.27)))
-    )
-    (property "Value" "OR_3" (at 178.4348 75.7461 0)
-      (effects (font (size 1.27 1.27)))
-    )
-    (property "Footprint" "" (at 178.181 80.645 0)
-      (effects (font (size 1.27 1.27)) hide)
-    )
-    (property "Datasheet" "http://iceboy.a-singer.de/doc/dmg_cells.html#or3" (at 178.435 88.265 0)
-      (effects (font (size 1.27 1.27)) hide)
-    )
-    (pin "1")
-    (pin "2")
-    (pin "3")
-    (pin "4")
-    (instances
-      (project "S-CPU"
-        (path "/ca9d3ca9-0297-4b98-a109-b7c162ccc5c3"
-          (reference "GBEG") (unit 1)
-        )
-        (path "/ca9d3ca9-0297-4b98-a109-b7c162ccc5c3/07b46eb7-d060-47db-b3fe-ac171637ec19"
-          (reference "GBEG") (unit 1)
-        )
-      )

Commit message: Big update on the hierarchical sheet. DMA section update too.
Parts:
- PBAD, PBEG: value DFFR_A -> DFFR_B; symbol Ricoh_Cells:DFFR_A -> Ricoh_Cells:DFFR_B
Connections:
- net H128-135 renamed ~{H128-135}
- net RW_EN renamed CPU_RW_EN
- net wMBLO renamed wMBLO_~{XIN/256}
- no-connect marks 10 -> 12
Other:
- note added: "DRAM refresh is enabled by setting it on for 32 master cycles from H=128 to H=135 DRAM refresh is disabled whenever H(3 downto 0) = "1x1x" (or "1x11" when accessing 4000-41FF HW registers). It means that DRAM refresh comes on at H128 ("010000000") and gets disabled at H138 ("010001010") and SYSCLK signal is feed to DRAM refresh pin during 10H cycles or 40 Master cycles."
- note added: "SYSCLK and ~{SYSCLK} signals used in the DMA region"
- note removed: "SYSCLK and ~{SYSCLK} signals in the DMA region"
- moved on the sheet: PAWC, PAWH
