File: S-CPU_kicad/joypads.kicad_sch (KiCad schematic)
At the start: 280 parts, among them U33 OR_2, U38 OR_2

Commit message: Identified some DFFs as being DFFs with SET input rather than RESET input. It helps explaining a lot of beahiour in the MUL/DIV section and in the DMA section.
Connections:
- net JPDATA_RST renamed ~{JPDATA_RST}
Changed lines of the file:
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@@
     (effects (font (size 1.27 1.27)) (justify right bottom))
   )
-  (label "JPDATA_RST" (at 365.125 540.385 0) (fields_autoplaced)
+  (label "~{JPDATA_RST}" (at 365.125 540.385 0) (fields_autoplaced)
     (effects (font (size 1.27 1.27)) (justify left bottom))
   )
@@
     (effects (font (size 1.27 1.27)) (justify right bottom))
   )
-  (label "JPDATA_RST" (at 477.52 540.385 0) (fields_autoplaced)
+  (label "~{JPDATA_RST}" (at 477.52 540.385 0) (fields_autoplaced)
     (effects (font (size 1.27 1.27)) (justify left bottom))
   )
@@
     (effects (font (size 1.27 1.27)) (justify right bottom))
   )
-  (label "JPDATA_RST" (at 253.365 540.385 0) (fields_autoplaced)
+  (label "~{JPDATA_RST}" (at 253.365 540.385 0) (fields_autoplaced)
     (effects (font (size 1.27 1.27)) (justify left bottom))
   )
@@
     (effects (font (size 1.27 1.27)) (justify left bottom))
   )
-  (label "JPDATA_RST" (at 588.645 540.385 0) (fields_autoplaced)
+  (label "~{JPDATA_RST}" (at 588.645 540.385 0) (fields_autoplaced)
     (effects (font (size 1.27 1.27)) (justify left bottom))
   )
@@
     (effects (font (size 1.27 1.27)) (justify left bottom))
   )
-  (label "JPDATA_RST" (at 361.95 139.065 180) (fields_autoplaced)
-    (effects (font (size 1.27 1.27)) (justify right bottom))
-  )
+  (label "~{JPDATA_RST}" (at 361.95 139.065 180) (fields_autoplaced)
+    (effects (font (size 1.27 1.27)) (justify right bottom))
+  )

Commit message: Fix ERC errors in schematics.
Parts:
- removed OAXV: AND_2, symbol Ricoh_Cells:AND_2
- removed OAYK: INVERTER_A, symbol Ricoh_Cells:INVERTER_A
- renumbered CGAY to DGLJ, DGLJ to EGGS, U33 to FGJP, U38 to GGMX
Connections:
- net wOAXV: now reaches MBUP.2, WAJJ.1
- removed net 65816_?: ABVA1.1 (IN), ABVA1.3 (IN), ABWF1.1 (IN), ABWF1.3 (IN), ABXH1.1 (IN), ABXH1.3 (IN)
- new net 65816_BE: ABVA1.1 (IN), ABVA1.3 (IN)
- new net 65816_EF: ABWF1.1 (IN), ABWF1.3 (IN)
- new net 65816_WAI: ABXH1.1 (IN), ABXH1.3 (IN)
Other:
- title: SNES S-CPU Schematics  -> Reverse Engineered SNES S-CPU Schematics 

Commit message: Big rework on the hierachical sheet to make thigs a bit clearer. PDF exported for Rev 0.1.
Parts:
- removed ABVA1, ABWF1, ABXH1: TRI_BUF_IF1, symbol Ricoh_Cells:TRI_BUF_IF1
- removed ABVA1 (x10): TRI_BUF_IF0, symbol Ricoh_Cells:TRI_BUF_IF0
- removed FBTA? (x5): BUF, symbol Ricoh_Cells:BUF
- removed FFJW, FFKX, GFEE, GFFG, GGDR, GGWB, GGYE, ODYR, WAJJ, WAOX, WAYX: INVERTER_A, symbol Ricoh_Cells:INVERTER_A
- removed GFAY (x3), OACG, OAMJ: DELAY_BUF, symbol Ricoh_Cells:DELAY_BUF
- removed GFVV, GGKX, VBHG, VBIE, WAXM, WAZZ: OR_2, symbol Ricoh_Cells:OR_2
- removed JP1CLK (x2), JP2CLK (x3): OBUF_A, symbol Ricoh_Cells:OBUF_A
- removed JP2I0 (x7): IBUF, symbol Ricoh_Cells:IBUF
- removed KBKC, KBLJ, KBMV: DFFR_A, symbol Ricoh_Cells:DFFR_A
- removed MBUP: AOI_22, symbol Ricoh_Cells:AOI_22
- removed VBBU, VBCP, WAWQ: AND_2, symbol Ricoh_Cells:AND_2
- gave numbers to parts that had none: 9
- renumbered KAVS to AFGF, ABVA1 to AFHM, KBMV to AFIA, ABWF1 to AFIS, KBLJ to AFLC, ABXH1 to AFNO, KBKC to AFOC, ACBV1 to AFPK, KBIF to AFRH, ACGM1 to AFUM, KBIE to AFWZ, ACHJ1 to AFYN, KBGO to AFZJ, ACJG1 to AGEL, KBGM to AGHW, ACKH1 to AGHX, KBMV to BFDW, ABVA1 to BFIV, KBLJ to BFIZ, ABWF1 to BFKI, KBKC to BFMC, ABXH1 to BFOI, KBIF to BFOL, ACBV1 to BFON, KBIE to BFTZ, ACGM1 to BFXS, KBGO to BFXV, ACHJ1 to BFYW, KBGM to BFZS, ACJG1 to BGAA, KAYP to BGAI, ACKH1 to BGGQ, KAVS to CFGC, ABVA1 to CFGO, KBMV to CFGR, ABWF1 to CFHI, KBLJ to CFKG, ABXH1 to CFKP, KBKC to CFMI, ACBV1 to CFML, KBIF to CFOX, ACGM1 to CFSY, KBIE to CFTE, ACHJ1 to CFTH, KBGO to CFVT, ACJG1 to CFZI, KBGM to CFZK, ACKH1 to CFZS, KBMV to DFHJ, ABVA1 to DFIJ, KBLJ to DFIT, ABWF1 to DFMO, KBKC to DFTG, ABXH1 to DFUW, KBIF to DFXA, ACBV1 to DFXY, KBIE to DFYY, ACGM1 to DFZH, KBGO to DGAA, ACHJ1 to DGBZ, KBGM to DGDN, ACJG1 to DGDX, KAYP to DGER, ACKH1 to DGGV, KAVS to EFMC, ABVA1 to EFNZ, KBMV to EFOX, ABWF1 to EFOZ, KBLJ to EFTN, ABXH1 to EFUK, KBKC to EFUW, ACBV1 to EFVW, KBIF to EFWT, ACGM1 to EFXE, KBIE to EFYF, ACHJ1 to EFYO, KBGO to EGCY, ACJG1 to EGDH, KBGM to EGED, ACKH1 to EGEH, KBMV to FFMK, ABVA1 to FFNO, KBLJ to FFNX, ABWF1 to FFPL, KBKC to FFPO, ABXH1 to FFQL, KBIF to FFQW, ACBV1 to FFUM, KBIE to FFVA, ACGM1 to FFVX, KBGO to FFWB, ACHJ1 to FGBR, KBGM to FGCI, ACJG1 to FGFA, KAYP to FGGD, ACKH1 to FGJE, ABVA1 to GFKZ, ABWF1 to GFOQ, ABXH1 to GFWB, ACBV1 to GGBS, ACGM1 to GGFL, ACHJ1 to GGJH, ACJG1 to GGNF, ACKH1 to GGPL, JP2I0 to JPIO0, JP2I0 to JPIO1, JP2I0 to JPIO2, JP2I0 to JPIO3, JP2I0 to JPIO4, JP2I0 to JPIO5, JP2I0 to JPIO6, JP2I0 to JPIO7, RBTV to VAFH, RBSA to VAGJ, RBTV to VAMM, RBAH to VAWR, RBFP to VAWW, RBPF to VAXI, RBSA to VAYA, RBTV to VAYP, BAOZ to WCFG, BAOZ to WCJB, BAOZ to WCLL, BAOZ to WCNB, KAVS to XABG, KBMV to XACL, KBLJ to XAFJ, KBKC to XAGK, KBIF to XAIJ, KBIE to XAJT, KBGO to XANT, KBGM to XAOI, BAOZ to XAOP, BAOZ to XARF, BAOZ to XBBN, BAOZ to XBBQ, BAOZ to XBDH, BAOZ to XBFC, KAVS to YAPL, ABVA1 to YAPP, KBMV to YARP, ABWF1 to YARY, KBLJ to YATC, ABXH1 to YAUO, KBKC to YAVJ, ACBV1 to YAWL, KBIF to YAWS, ACGM1 to YBBP, KBIE to YBDC, ACHJ1 to YBEH, KBGO to YBHJ, ACJG1 to YBKL, KBGM to YBNR, ACKH1 to YBOB, KBMV to ZAEM, ABVA1 to ZAGK, KBLJ to ZAID, ABWF1 to ZAIR, KBKC to ZAKT, ABXH1 to ZALT, KBIF to ZAPI, ACBV1 to ZAPZ, KBIE to ZAQA, ACGM1 to ZAVO, KBGO to ZAXL, ACHJ1 to ZAYR, KBGM to ZBBY, ACJG1 to ZBEQ, KAYP to ZBFI, ACKH1 to ZBKU
Connections:
- net AUTO_JP0: now also VAYP.9 (Q); no longer VAYP.7 (Q)
- net AUTO_JP1: now also VAYA.9 (Q); no longer VAYA.7 (Q)
- net AUTO_JP2: now also VAXI.9 (Q); no longer VAXI.7 (Q)
- net AUTO_JP3: now also VAWW.9 (Q); no longer VAWW.7 (Q)
- net AUTO_JP_READING: now also VAWR.8 (~{Q}); no longer VAWR.6 (~{Q})
- net JPDATA_CLK: now also VAWR.1 (CLK), VAYP.1 (CLK); no longer VAWR.3 (CLK), VAWR.4 (~{CLK}), VAYP.3 (CLK), VAYP.4 (~{CLK})
- net ~{4201_WR}: now also XABG.1 (CLK), XACL.1 (CLK), XAFJ.1 (CLK), XAGK.1 (CLK), XAIJ.1 (CLK), XAJT.1 (CLK), XANT.1 (CLK), XAOI.1 (CLK); no longer XABG.3 (CLK), XABG.4 (~{CLK}), XACL.3 (CLK), XACL.4 (~{CLK}), XAFJ.3 (CLK), XAFJ.4 (~{CLK}), XAGK.3 (CLK), XAGK.4 (~{CLK}), XAIJ.3 (CLK), XAIJ.4 (~{CLK}), XAJT.3 (CLK), XAJT.4 (~{CLK}), XANT.3 (CLK), XANT.4 (~{CLK}), XAOI.3 (CLK), XAOI.4 (~{CLK})
- net ~{JPDATA_RST}: now also AFGF.6 (~{RESET}), AFIA.6 (~{RESET}), AFLC.6 (~{RESET}), AFOC.6 (~{RESET}), AFRH.6 (~{RESET}), AFWZ.6 (~{RESET}), AFZJ.6 (~{RESET}), AGHW.6 (~{RESET}), BFDW.6 (~{RESET}), BFIZ.6 (~{RESET}), BFMC.6 (~{RESET}), BFOL.6 (~{RESET}), BFTZ.6 (~{RESET}), BFXV.6 (~{RESET}), BFZS.6 (~{RESET}), BGAI.6 (~{RESET}), CFGC.6 (~{RESET}), CFGR.6 (~{RESET}), CFKG.6 (~{RESET}), CFMI.6 (~{RESET}), CFOX.6 (~{RESET}), CFTE.6 (~{RESET}), CFVT.6 (~{RESET}), CFZK.6 (~{RESET}), DFHJ.6 (~{RESET}), DFIT.6 (~{RESET}), DFTG.6 (~{RESET}), DFXA.6 (~{RESET}), DFYY.6 (~{RESET}), DGAA.6 (~{RESET}), DGDN.6 (~{RESET}), DGER.6 (~{RESET}), EFMC.6 (~{RESET}), EFOX.6 (~{RESET}), EFTN.6 (~{RESET}), EFUW.6 (~{RESET}), EFWT.6 (~{RESET}), EFYF.6 (~{RESET}), EGCY.6 (~{RESET}), EGED.6 (~{RESET}), FFMK.6 (~{RESET}), FFNX.6 (~{RESET}), FFPO.6 (~{RESET}), FFQW.6 (~{RESET}), FFVA.6 (~{RESET}), FFWB.6 (~{RESET}), FGCI.6 (~{RESET}), FGGD.6 (~{RESET}), YAPL.6 (~{RESET}), YARP.6 (~{RESET}), YATC.6 (~{RESET}), YAVJ.6 (~{RESET}), YAWS.6 (~{RESET}), YBDC.6 (~{RESET}), YBHJ.6 (~{RESET}), YBNR.6 (~{RESET}), ZAEM.6 (~{RESET}), ZAID.6 (~{RESET}), ZAKT.6 (~{RESET}), ZAPI.6 (~{RESET}), ZAQA.6 (~{RESET}), ZAXL.6 (~{RESET}), ZBBY.6 (~{RESET}), ZBFI.6 (~{RESET}); no longer AFGF.1 (~{RESET}), AFGF.5 (~{RESET}), AFIA.1 (~{RESET}), AFIA.5 (~{RESET}), AFLC.1 (~{RESET}), AFLC.5 (~{RESET}), AFOC.1 (~{RESET}), AFOC.5 (~{RESET}), AFRH.1 (~{RESET}), AFRH.5 (~{RESET}), AFWZ.1 (~{RESET}), AFWZ.5 (~{RESET}), AFZJ.1 (~{RESET}), AFZJ.5 (~{RESET}), AGHW.1 (~{RESET}), AGHW.5 (~{RESET}), BFDW.1 (~{RESET}), BFDW.5 (~{RESET}), BFIZ.1 (~{RESET}), BFIZ.5 (~{RESET}), BFMC.1 (~{RESET}), BFMC.5 (~{RESET}), BFOL.1 (~{RESET}), BFOL.5 (~{RESET}), BFTZ.1 (~{RESET}), BFTZ.5 (~{RESET}), BFXV.1 (~{RESET}), BFXV.5 (~{RESET}), BFZS.1 (~{RESET}), BFZS.5 (~{RESET}), BGAI.1 (~{RESET}), BGAI.5 (~{RESET}), CFGC.1 (~{RESET}), CFGC.5 (~{RESET}), CFGR.1 (~{RESET}), CFGR.5 (~{RESET}), CFKG.1 (~{RESET}), CFKG.5 (~{RESET}), CFMI.1 (~{RESET}), CFMI.5 (~{RESET}), CFOX.1 (~{RESET}), CFOX.5 (~{RESET}), CFTE.1 (~{RESET}), CFTE.5 (~{RESET}), CFVT.1 (~{RESET}), CFVT.5 (~{RESET}), CFZK.1 (~{RESET}), CFZK.5 (~{RESET}), DFHJ.1 (~{RESET}), DFHJ.5 (~{RESET}), DFIT.1 (~{RESET}), DFIT.5 (~{RESET}), DFTG.1 (~{RESET}), DFTG.5 (~{RESET}), DFXA.1 (~{RESET}), DFXA.5 (~{RESET}), DFYY.1 (~{RESET}), DFYY.5 (~{RESET}), DGAA.1 (~{RESET}), DGAA.5 (~{RESET}), DGDN.1 (~{RESET}), DGDN.5 (~{RESET}), DGER.1 (~{RESET}), DGER.5 (~{RESET}), EFMC.1 (~{RESET}), EFMC.5 (~{RESET}), EFOX.1 (~{RESET}), EFOX.5 (~{RESET}), EFTN.1 (~{RESET}), EFTN.5 (~{RESET}), EFUW.1 (~{RESET}), EFUW.5 (~{RESET}), EFWT.1 (~{RESET}), EFWT.5 (~{RESET}), EFYF.1 (~{RESET}), EFYF.5 (~{RESET}), EGCY.1 (~{RESET}), EGCY.5 (~{RESET}), EGED.1 (~{RESET}), EGED.5 (~{RESET}), FFMK.1 (~{RESET}), FFMK.5 (~{RESET}), FFNX.1 (~{RESET}), FFNX.5 (~{RESET}), FFPO.1 (~{RESET}), FFPO.5 (~{RESET}), FFQW.1 (~{RESET}), FFQW.5 (~{RESET}), FFVA.1 (~{RESET}), FFVA.5 (~{RESET}), FFWB.1 (~{RESET}), FFWB.5 (~{RESET}), FGCI.1 (~{RESET}), FGCI.5 (~{RESET}), FGGD.1 (~{RESET}), FGGD.5 (~{RESET}), YAPL.1 (~{RESET}), YAPL.5 (~{RESET}), YARP.1 (~{RESET}), YARP.5 (~{RESET}), YATC.1 (~{RESET}), YATC.5 (~{RESET}), YAVJ.1 (~{RESET}), YAVJ.5 (~{RESET}), YAWS.1 (~{RESET}), YAWS.5 (~{RESET}), YBDC.1 (~{RESET}), YBDC.5 (~{RESET}), YBHJ.1 (~{RESET}), YBHJ.5 (~{RESET}), YBNR.1 (~{RESET}), YBNR.5 (~{RESET}), ZAEM.1 (~{RESET}), ZAEM.5 (~{RESET}), ZAID.1 (~{RESET}), ZAID.5 (~{RESET}), ZAKT.1 (~{RESET}), ZAKT.5 (~{RESET}), ZAPI.1 (~{RESET}), ZAPI.5 (~{RESET}), ZAQA.1 (~{RESET}), ZAQA.5 (~{RESET}), ZAXL.1 (~{RESET}), ZAXL.5 (~{RESET}), ZBBY.1 (~{RESET}), ZBBY.5 (~{RESET}), ZBFI.1 (~{RESET}), ZBFI.5 (~{RESET})
- net at ZAGK.1 (IN), ZAGK.3 (IN), ZAID.2 (D): now also ZAEM.9 (Q); no longer ZAEM.6 (Q)
- net at ZAPZ.1 (IN), ZAPZ.3 (IN), ZAQA.2 (D): now also ZAPI.9 (Q); no longer ZAPI.6 (Q)
- net at BGAA.1 (IN), BGAA.3 (IN), BGAI.2 (D): now also BFZS.9 (Q); no longer BFZS.6 (Q)
- net at FGBR.1 (IN), FGBR.3 (IN), FGCI.2 (D): now also FFWB.9 (Q); no longer FFWB.6 (Q)
- net at FGFA.1 (IN), FGFA.3 (IN), FGGD.2 (D): now also FGCI.9 (Q); no longer FGCI.6 (Q)
- net at YAWL.1 (IN), YAWL.3 (IN), YAWS.2 (D): now also YAVJ.9 (Q); no longer YAVJ.6 (Q)
- net at DFXY.1 (IN), DFXY.3 (IN), DFYY.2 (D): now also DFXA.9 (Q); no longer DFXA.6 (Q)
- net at DFZH.1 (IN), DFZH.3 (IN), DGAA.2 (D): now also DFYY.9 (Q); no longer DFYY.6 (Q)
- net at YBEH.1 (IN), YBEH.3 (IN), YBHJ.2 (D): now also YBDC.9 (Q); no longer YBDC.6 (Q)
- net at YBKL.1 (IN), YBKL.3 (IN), YBNR.2 (D): now also YBHJ.9 (Q); no longer YBHJ.6 (Q)
- net at BFXS.1 (IN), BFXS.3 (IN), BFXV.2 (D): now also BFTZ.9 (Q); no longer BFTZ.6 (Q)
- net at BFYW.1 (IN), BFYW.3 (IN), BFZS.2 (D): now also BFXV.9 (Q); no longer BFXV.6 (Q)
- net at EFOZ.1 (IN), EFOZ.3 (IN), EFTN.2 (D): now also EFOX.9 (Q); no longer EFOX.6 (Q)
- net at EFUK.1 (IN), EFUK.3 (IN), EFUW.2 (D): now also EFTN.9 (Q); no longer EFTN.6 (Q)
- net at EGDH.1 (IN), EGDH.3 (IN), EGED.2 (D): now also EGCY.9 (Q); no longer EGCY.6 (Q)
- net at EGEH.1 (IN), EGEH.3 (IN): now also EGED.9 (Q); no longer EGED.6 (Q)
- net at BFON.1 (IN), BFON.3 (IN), BFTZ.2 (D): now also BFOL.9 (Q); no longer BFOL.6 (Q)
- net at AGEL.1 (IN), AGEL.3 (IN), AGHW.2 (D): now also AFZJ.9 (Q); no longer AFZJ.6 (Q)
- net at AGHX.1 (IN), AGHX.3 (IN): now also AGHW.9 (Q); no longer AGHW.6 (Q)
- net at DGDX.1 (IN), DGDX.3 (IN), DGER.2 (D): now also DGDN.9 (Q); no longer DGDN.6 (Q)
- net at ZBEQ.1 (IN), ZBEQ.3 (IN), ZBFI.2 (D): now also ZBBY.9 (Q); no longer ZBBY.6 (Q)
- net at YAPL.2 (D), ZBKU.1 (IN), ZBKU.3 (IN): now also ZBFI.9 (Q); no longer ZBFI.6 (Q)
- net at FFNO.1 (IN), FFNO.3 (IN), FFNX.2 (D): now also FFMK.9 (Q); no longer FFMK.6 (Q)
- net at EFXE.1 (IN), EFXE.3 (IN), EFYF.2 (D): now also EFWT.9 (Q); no longer EFWT.6 (Q)
- net at DFBW.1: now also XANT.9 (Q); no longer XANT.6 (Q)
- net at CFGC.2 (D), DGGV.1 (IN), DGGV.3 (IN): now also DGER.9 (Q); no longer DGER.6 (Q)
- net at CFGO.1 (IN), CFGO.3 (IN), CFGR.2 (D): now also CFGC.9 (Q); no longer CFGC.6 (Q)
- net at FFPL.1 (IN), FFPL.3 (IN), FFPO.2 (D): now also FFNX.9 (Q); no longer FFNX.6 (Q)
- net at FFQL.1 (IN), FFQL.3 (IN), FFQW.2 (D): now also FFPO.9 (Q); no longer FFPO.6 (Q)
- net at EFMC.2 (D), FGJE.1 (IN), FGJE.3 (IN): now also FGGD.9 (Q); no longer FGGD.6 (Q)
- net JPOUT0_CLK: now reaches VAAA.3, VAMM.2 (D)
- net at CFHI.1 (IN), CFHI.3 (IN), CFKG.2 (D): now also CFGR.9 (Q); no longer CFGR.6 (Q)
- net at YBBP.1 (IN), YBBP.3 (IN), YBDC.2 (D): now also YAWS.9 (Q); no longer YAWS.6 (Q)
- net at AFIS.1 (IN), AFIS.3 (IN), AFLC.2 (D): now also AFIA.9 (Q); no longer AFIA.6 (Q)
- net at AFNO.1 (IN), AFNO.3 (IN), AFOC.2 (D): now also AFLC.9 (Q); no longer AFLC.6 (Q)
- net at BFIV.1 (IN), BFIV.3 (IN), BFIZ.2 (D): now also BFDW.9 (Q); no longer BFDW.6 (Q)
- net at EFGJ.1: now also XAOI.9 (Q); no longer XAOI.6 (Q)
- net at AFHM.1 (IN), AFHM.3 (IN), AFIA.2 (D): now also AFGF.9 (Q); no longer AFGF.6 (Q)
- net at DGBZ.1 (IN), DGBZ.3 (IN), DGDN.2 (D): now also DGAA.9 (Q); no longer DGAA.6 (Q)
- net at YARY.1 (IN), YARY.3 (IN), YATC.2 (D): now also YARP.9 (Q); no longer YARP.6 (Q)
- net at YBOB.1 (IN), YBOB.3 (IN): now also YBNR.9 (Q); no longer YBNR.6 (Q)
- net at YAPP.1 (IN), YAPP.3 (IN), YARP.2 (D): now also YAPL.9 (Q); no longer YAPL.6 (Q)
- net at BFOI.1 (IN), BFOI.3 (IN), BFOL.2 (D): now also BFMC.9 (Q); no longer BFMC.6 (Q)
- net at DFUW.1 (IN), DFUW.3 (IN), DFXA.2 (D): now also DFTG.9 (Q); no longer DFTG.6 (Q)
- net at VAWW.6 (~{RESET}): now also VAMM.9 (Q), VASJ.1, VAWR.6 (~{RESET}), VAXI.6 (~{RESET}), VAYA.6 (~{RESET}), VAYP.6 (~{RESET}), VAYR.1; no longer VAWW.2 (D)
- net at CFDM.1: now also XAJT.9 (Q); no longer XAJT.6 (Q)
- net at CFKP.1 (IN), CFKP.3 (IN), CFMI.2 (D): now also CFKG.9 (Q); no longer CFKG.6 (Q)
- net at CFML.1 (IN), CFML.3 (IN), CFOX.2 (D): now also CFMI.9 (Q); no longer CFMI.6 (Q)
- net at EFYO.1 (IN), EFYO.3 (IN), EGCY.2 (D): now also EFYF.9 (Q); no longer EFYF.6 (Q)
- net at AFUM.1 (IN), AFUM.3 (IN), AFWZ.2 (D): now also AFRH.9 (Q); no longer AFRH.6 (Q)
- net at BFKI.1 (IN), BFKI.3 (IN), BFMC.2 (D): now also BFIZ.9 (Q); no longer BFIZ.6 (Q)
- net at ZAIR.1 (IN), ZAIR.3 (IN), ZAKT.2 (D): now also ZAID.9 (Q); no longer ZAID.6 (Q)
- net at ZALT.1 (IN), ZALT.3 (IN), ZAPI.2 (D): now also ZAKT.9 (Q); no longer ZAKT.6 (Q)
- net at XAAX.1: now also XABG.9 (Q); no longer XABG.6 (Q)
- net at EFVW.1 (IN), EFVW.3 (IN), EFWT.2 (D): now also EFUW.9 (Q); no longer EFUW.6 (Q)
- net at ZAAT.1: now also XAFJ.9 (Q); no longer XAFJ.6 (Q)
- net at ZAVO.1 (IN), ZAVO.3 (IN), ZAXL.2 (D): now also ZAQA.9 (Q); no longer ZAQA.6 (Q)
- net at ZAYR.1 (IN), ZAYR.3 (IN), ZBBY.2 (D): now also ZAXL.9 (Q); no longer ZAXL.6 (Q)
- net at VAGJ.2 (D), VAGU.2: now also VAFH.8 (~{Q}); no longer VAFH.6 (~{Q})
- net at VAGU.1: now also VAGJ.8 (~{Q}); no longer VAGJ.6 (~{Q})
- net at YAUO.1 (IN), YAUO.3 (IN), YAVJ.2 (D): now also YATC.9 (Q); no longer YATC.6 (Q)
- net at FFUM.1 (IN), FFUM.3 (IN), FFVA.2 (D): now also FFQW.9 (Q); no longer FFQW.6 (Q)
- net at FFVX.1 (IN), FFVX.3 (IN), FFWB.2 (D): now also FFVA.9 (Q); no longer FFVA.6 (Q)
- net at AFPK.1 (IN), AFPK.3 (IN), AFRH.2 (D): now also AFOC.9 (Q); no longer AFOC.6 (Q)
- net AUTO_JP_CLK: now reaches VAYV.3
- net at CFZS.1 (IN), CFZS.3 (IN): now also CFZK.9 (Q); no longer CFZK.6 (Q)
- net at AFDJ.1: now also XAGK.9 (Q); no longer XAGK.6 (Q)
- net at CFSY.1 (IN), CFSY.3 (IN), CFTE.2 (D): now also CFOX.9 (Q); no longer CFOX.6 (Q)
- net at EFNZ.1 (IN), EFNZ.3 (IN), EFOX.2 (D): now also EFMC.9 (Q); no longer EFMC.6 (Q)
- net at AFGF.2 (D), BGGQ.1 (IN), BGGQ.3 (IN): now also BGAI.9 (Q); no longer BGAI.6 (Q)
- net at BFAR.1: now also XAIJ.9 (Q); no longer XAIJ.6 (Q)
- net at AFYN.1 (IN), AFYN.3 (IN), AFZJ.2 (D): now also AFWZ.9 (Q); no longer AFWZ.6 (Q)
- net JP_CLK: now reaches VACD.1, VASU.1
- net JP_CLK: now also VAMM.1 (CLK); no longer VAMM.3 (CLK), VAMM.4 (~{CLK})
- net at YAAV.1: now also XACL.9 (Q); no longer XACL.6 (Q)
- net at CFTH.1 (IN), CFTH.3 (IN), CFVT.2 (D): now also CFTE.9 (Q); no longer CFTE.6 (Q)
- net at DFMO.1 (IN), DFMO.3 (IN), DFTG.2 (D): now also DFIT.9 (Q); no longer DFIT.6 (Q)
- net at CFZI.1 (IN), CFZI.3 (IN), CFZK.2 (D): now also CFVT.9 (Q); no longer CFVT.6 (Q)
- net ~{JP_RST}: now reaches VAMM.6 (~{RESET})
- net ~{JP_RST}: now also VAFH.6 (~{RESET}), VAGJ.6 (~{RESET}), XABG.6 (~{RESET}), XACL.6 (~{RESET}), XAFJ.6 (~{RESET}), XAGK.6 (~{RESET}), XAIJ.6 (~{RESET}), XAJT.6 (~{RESET}), XANT.6 (~{RESET}), XAOI.6 (~{RESET})
- net at DFIJ.1 (IN), DFIJ.3 (IN), DFIT.2 (D): now also DFHJ.9 (Q); no longer DFHJ.6 (Q)
- removed net wMASS_~{JP_RST}: VAFH.1 (~{RESET}), VAFH.5 (~{RESET}), VAGJ.1 (~{RESET}), VAGJ.5 (~{RESET}), VAMM.1 (~{RESET}), VAMM.5 (~{RESET}), XABG.1 (~{RESET}), XABG.5 (~{RESET}), XACL.1 (~{RESET}), XACL.5 (~{RESET}), XAFJ.1 (~{RESET}), XAFJ.5 (~{RESET}), XAGK.1 (~{RESET}), XAGK.5 (~{RESET}), XAIJ.1 (~{RESET}), XAIJ.5 (~{RESET}), XAJT.1 (~{RESET}), XAJT.5 (~{RESET}), XANT.1 (~{RESET}), XANT.5 (~{RESET}), XAOI.1 (~{RESET}), XAOI.5 (~{RESET})
- new net: ZAEM.1 (CLK), ZAGC.2, ZAID.1 (CLK), ZAKT.1 (CLK), ZAPI.1 (CLK), ZAQA.1 (CLK), ZAXL.1 (CLK), ZBBY.1 (CLK), ZBFI.1 (CLK)
- new net: FFLE.2, FFMK.1 (CLK), FFNX.1 (CLK), FFPO.1 (CLK), FFQW.1 (CLK), FFVA.1 (CLK), FFWB.1 (CLK), FGCI.1 (CLK), FGGD.1 (CLK)
- new net: DFFR.2, DFHJ.1 (CLK), DFIT.1 (CLK), DFTG.1 (CLK), DFXA.1 (CLK), DFYY.1 (CLK), DGAA.1 (CLK), DGDN.1 (CLK), DGER.1 (CLK)
- new net: YAOH.2, YAPL.1 (CLK), YARP.1 (CLK), YATC.1 (CLK), YAVJ.1 (CLK), YAWS.1 (CLK), YBDC.1 (CLK), YBHJ.1 (CLK), YBNR.1 (CLK)
- new net: BFCS.2, BFDW.1 (CLK), BFIZ.1 (CLK), BFMC.1 (CLK), BFOL.1 (CLK), BFTZ.1 (CLK), BFXV.1 (CLK), BFZS.1 (CLK), BGAI.1 (CLK)
- new net: EFHT.2, EFMC.1 (CLK), EFOX.1 (CLK), EFTN.1 (CLK), EFUW.1 (CLK), EFWT.1 (CLK), EFYF.1 (CLK), EGCY.1 (CLK), EGED.1 (CLK)
- new net: AFFY.2, AFGF.1 (CLK), AFIA.1 (CLK), AFLC.1 (CLK), AFOC.1 (CLK), AFRH.1 (CLK), AFWZ.1 (CLK), AFZJ.1 (CLK), AGHW.1 (CLK)
- new net: CFEE.2, CFGC.1 (CLK), CFGR.1 (CLK), CFKG.1 (CLK), CFMI.1 (CLK), CFOX.1 (CLK), CFTE.1 (CLK), CFVT.1 (CLK), CFZK.1 (CLK)
- new net: VAXI.1 (CLK), VAYA.2 (D), VAYA.8 (~{Q})
- new net: VAWW.1 (CLK), VAXI.2 (D), VAXI.8 (~{Q})
- new net: VAWW.2 (D), VAWW.8 (~{Q})
- new net: VACD.2, VAFH.1 (CLK), VAGJ.1 (CLK)
- new net: VAYA.1 (CLK), VAYP.2 (D), VAYP.8 (~{Q})
- no-connect marks 5 -> 4
Other:
- note removed: "4016 WRITE"
- note removed: "4016/4017 READ"
- note removed: "Normal clock is XIN/256 which will take 3 scamline lines to fill in jp shift registers. In MODE6, XIN/4 clock is used instead when RDY = 0."
- note removed: "Unconnected ??"
- moved on the sheet: AFDJ, AFFY, AFHM, AFIS, AFNO, AFPK, AFUM, AFYN, AGEL, AGHX, AGJS, BFAR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

Commit message: Fixed VAWR which should have been an SR DFF (to fix issue #3 raised in github)
Parts:
- removed VAWR: DFFR_B, symbol Ricoh_Cells:DFFR_B
- added VAWR: DFFSR, symbol Ricoh_Cells:DFFSR
Connections:
- net AUTO_JP_EN: now also VAWR.4 (~{SET})
- net AUTO_JP_READING: now also VAWR.9 (~{Q})
- net JPDATA_CLK: now also VAWR.1 (CLK)
- net at VAMM.9 (Q), VASJ.1, VAWW.6 (~{RESET})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: now also VAWR.7 (~{RESET})
- net at WBNN.5: now also VAWR.2 (D)
Other:
- note added: "JP counter is reset when entering VBLANK and counts up to 16 for 16 JP clock cycles to shift data into JP registers providing AUTO_JP_EN is set to 1"
- note added: "Vblank rising edge detection"
- note removed: "JP counter is reset outside of VBLANK and count up to 16 for 16 JP clock cycles to shift data into JP registers at the start of VBLANK."
- moved on the sheet: AFDJ, AFFY, AFGF, AFHM, AFIA, AFIS, AFLC, AFNO, AFOC, AFPK, AFRH, AFUM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
