File: S-CPU_kicad/rw_decoding.kicad_sch (KiCad schematic)
At the start: 131 parts

Commit message: Fix ERC errors in schematics.
Parts:
- removed AABC, DBIS, DBVA, FBTA: BUF, symbol Ricoh_Cells:BUF
- removed ABORT: IBUF, symbol Ricoh_Cells:IBUF
- removed VP: OBUF_A, symbol Ricoh_Cells:OBUF_A
- added BAAG, GAJP: BUF, symbol Ricoh_Cells:BUF
- added DFAA: DELAY_BUF, symbol Ricoh_Cells:DELAY_BUF
- added OAXV: AND_2, symbol Ricoh_Cells:AND_2
- added OAYK: INVERTER_A, symbol Ricoh_Cells:INVERTER_A
Connections:
- net ~{MODE6}: now also OAYK.1
- net ~{ROM_SEL}: now also BAAG.2
- net ~{wRDY}: now also OAXV.1
- net at AAFD.3: now also BAAG.1
- net at GAJP.2: now also DFAA.1
- net at ~{CPU_WR}.1 (OUTPUT): now also GAJP.2
- net 65816_IRQ renamed 65816_~{IRQ}
- net 65816_ML renamed 65816_MLB
- net 65816_NMI renamed 65816_~{NMI}
- new net: OAXV.2, OAYK.2
- new net: DFAA.2, GAJP.1
- new net wOAXV: OAXV.3
Other:
- title: SNES S-CPU Schematics  -> Reverse Engineered SNES S-CPU Schematics 

Commit message: Big rework on the hierachical sheet to make thigs a bit clearer. PDF exported for Rev 0.1.
Parts:
- removed AAFD, BALC, LBQM: OR_2, symbol Ricoh_Cells:OR_2
- removed BAAG (x2), CACL, CAFH: BUF, symbol Ricoh_Cells:BUF
- removed BABW, BAUV, CADW, CAEI, CAWE, EAHW, EARJ, EASO, EBMJ, EBMQ, EBOS, FBBC, OAYK: INVERTER_A, symbol Ricoh_Cells:INVERTER_A
- removed BAEH: NOR_2, symbol Ricoh_Cells:NOR_2
- removed BAGU, EBQY, OAXV: AND_2, symbol Ricoh_Cells:AND_2
- removed BAIS: OR_4, symbol Ricoh_Cells:OR_4
- removed BASL, BATZ, EBCS, GBEV: NAND_3, symbol Ricoh_Cells:NAND_3
- removed CACT, CACW, CAHN: AND_3, symbol Ricoh_Cells:AND_3
- removed CAEO: NAND_4, symbol Ricoh_Cells:NAND_4
- removed CAJX: NOR_3, symbol Ricoh_Cells:NOR_3
- removed CARY, EAOI: NOR_6, symbol Ricoh_Cells:NOR_6
- removed EAMV, EANE: NOR_5, symbol Ricoh_Cells:NOR_5
- removed EAPY: NOR_8, symbol Ricoh_Cells:NOR_8
- removed FBAC: AOI_14, symbol Ricoh_Cells:AOI_14
- removed ~{RAM_SEL}, ~{ROM_SEL}: OBUF_A, symbol Ricoh_Cells:OBUF_A
- added DCEG, FBSI: TRI_INV_IF2, symbol Ricoh_Cells:TRI_INV_IF2
- added GBEG2, IARF: OR_3, symbol Ricoh_Cells:OR_3
- added HAKW, IBEP, JBQK, MBSK: BUF, symbol Ricoh_Cells:BUF
- added HALC, HBCT, HBGA, IAQU, IBGG, KBVA: OR_2, symbol Ricoh_Cells:OR_2
- added HAMT, LBXR: D_LATCH_A2, symbol Ricoh_Cells:D_LATCH_A2
- added HANA, HAZL, HBQJ, IAQS, IBNJ, JAXB, JBDE, MBUB, ZOZP: INVERTER_A, symbol Ricoh_Cells:INVERTER_A
- added HBCA, HBEP: TRI_INV_IF0, symbol Ricoh_Cells:TRI_INV_IF0
- added IAQD, IAQV, JAXC, ROLZ: AND_2, symbol Ricoh_Cells:AND_2
- added IARB, IOAW: TRI_BUF_IF0, symbol Ricoh_Cells:TRI_BUF_IF0
- added JBNA: OAI_112, symbol Ricoh_Cells:OAI_112
- added JBND, JBPY, KBUP, ROMA: NAND_2, symbol Ricoh_Cells:NAND_2
- added MBUP: AOI_22, symbol Ricoh_Cells:AOI_22
- added RDY: IBUF, symbol Ricoh_Cells:IBUF
- added VDA, VPA: IOBUF_B, symbol Ricoh_Cells:IOBUF_B
- renumbered GAJP to DBIS, DFAA to FAAN
Connections:
- net CPU_RW_EN: now also GBEG2.4
- net DMA_OFF: now also JBDE.1, JBPY.2
- net DMA_ON: now also LBXR.3 (D)
- net MODE2_OR_MODE3: now also GBEG2.3
- net MODE4-6: now also JBNA.3, MBUP.1
- net MODE4_OR_MODE5: now also ROMA.2
- net SYNCED_REFRESH_EN: now also GBEG2.1
- net ~{DMA_BUS_EN}: now also JBQK.2, MBUP.2
- net ~{DMA_RW_EN}: now also JBNA.5, JBQK.1
- net ~{MODE0_OR_MODE6}: now also ROLZ.2
- net ~{MODE1}: now also KBVA.2, MBUB.1
- net ~{wRDY}: now also HBQJ.2, KBVA.1, MBUP.3, ZOZP.1
- net at BBER.3: now also BBNW.9 (Q); no longer BBNW.6 (Q)
- net ~{XIN}: now reaches BBNW.1 (CLK)
- net ~{XIN}: no longer BBNW.5 (~{RESET})
- net wIBPY: no longer names the net of IBKU.1, IBPY.3, IBUA.2, JBSU.2, KBWT.2, NBZA.2, NCAN.2
- net wIBPY: now also HBCT.2, HBGA.2
- net wOATI_~{XIN/256} renamed ~{XIN/256}
- removed net ~{XIN1}: BBNW.3 (CLK), BBNW.4 (~{CLK})
- new net: MBSK.1, MBUP.3
- new net: HBGA.1, VDA.2 (~{INPUT})
- new net: HBEP.2, HBGA.3
- new net: MBUB.2, MBUP.4
- new net: JBND.2, JBPY.3
- new net: DCEG.3, VPA.1 (DRV_LOW)
- new net: HBCT.1, VPA.2 (~{INPUT})
- new net: DCEG.3, VPA.4 (~{DRV}_HIGH)
- new net: ROMA.1, ZOZP.2
- new net: ROLZ.1, ROMA.3
- new net: KBUP.2, KBVA.3
- new net: HAZL.2, HBCA.1 (~{ENA}), HBEP.1 (~{ENA})
- new net: JAXB.2, JAXC.1
- new net: DCEG.1 (~{ENA}), FBSI.1 (~{ENA}), HAZL.1, IARB.2 (~{ENA}), IOAW.2 (~{ENA}), JAXC.3
- new net: IBGG.2, IBNJ.2
- new net: IBEP.1, IBGG.3
- new net: IAQV.3, IARB.1 (IN), IARB.3 (IN)
- new net: IAQD.3, IOAW.1 (IN), IOAW.3 (IN)
- new net: HAKW.1, HALC.3
- new net: HBQJ.1, RDY.1 (INPUT)
- new net: HALC.1, HAMT.5 (Q)
- new net: HALC.2, HAMT.3 (D), HANA.2
- new net: IARF.1, JBDE.2
- new net: FBSI.3, VDA.1 (DRV_LOW)
- new net: FBSI.3, VDA.4 (~{DRV}_HIGH)
- new net: HBCA.2, HBCT.3
- new net: JBNA.1, LBXR.5 (Q)
- new net: IAQS.2, IAQU.2
- new net: IAQD.1, IAQU.3, IAQV.1
- new net 65816_ADDR_LATCH: HAMT.1 (ENA)
- new net 65816_RDY: HANA.1, JBND.3
- new net 65816_VDA: IAQD.2
- new net 65816_VPA: IAQV.2
- new net MODE0_OR_MODE1_AND_RDY: JAXB.1, JBNA.4, JBPY.1, KBUP.3
- new net XIN/2: LBXR.1 (ENA)
- new net wIARB_or_wHBCA: DCEG.2, HBCA.3, IARB.4, IARF.3
- new net wIOAW_or_wHBEP: FBSI.2, HBEP.3, IARF.2, IOAW.4
- new net ~{65816_ADDR_EN}: HAKW.2
- new net ~{65816_ADDR_RST}: IBEP.2
- new net ~{CPU_RST}: IAQU.1, IBGG.1, JBNA.2
- new net ~{EXTERNAL_BUS_EN}: MBSK.2
- new net ~{INTERNAL_CYCLE}: GBEG2.2, IARF.4
- new net ~{MODE0}: KBUP.1
- new net ~{MODE7}: IAQS.1, IBNJ.1, JAXC.2, JBND.1
- no-connect marks 1 -> 4
Other:
- note added: "Cells in DMA section but not connected. Change of design or test in early prototypes?"
- note added: "Disconnects 65816 in MODE7, in MODE1 when RDY is low and during DMA"
- note added: "IARF Goes low during internal CPU cycles VDA and VPA are low and DMA is not running"
- note added: "JBNA = JBQK set to '1' when in MODE2-3, in MODE7, in MODE1 + RDY = 0 or DMA is OFF"
- note added: "Low when RDY = 0 in mode 1 or when DMA is on in mode 4-6"
- note added: "One of the conditions for ~{PAWR} to be asserted: - CPU write when CPU_RW_EN = '1' and ADDR = 21XX and CPU_RW_EN = '0' and R~{W} = '0' and SYSCLK = '1' - DMA write when ~{DMA_RW_EN} = '0' and DMA_B->A = '0' and SYSCLK = '1' and HDMA_TABLE_RD = '0' One of the conditions for ~{PARD} to be asserted: - CPU read when CPU_RW_EN = '1' and ADDR = 21XX and ~{DMA_RW_EN} = '1' and R~{W} = '1' and SYSCLK = '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"
- note removed: "Address decoding"
- note removed: "B-BUS select (21XX) when not in MODE2 or 3"
- note removed: "DMA registers 4300-437F active low select"
- note removed: "Internal registers only In NES mode (MODE2-3), only 4016 and 4017 will set CPU_REG_RD to 1."
- note removed: "RAM and RAM Selection"
- note removed: "~{ROMSEL} = ~{A23}.A22.A21.A20.A19.A18.A17 + ~{A22}.~{A15} Consistent with access to: - 00-3F/80-BF:8000-FFFF or - 40-7D/C0-FF:0000-FFFF ~{RAMSEL} = not (~{/A23}.A22.A21.A20.A19.A18.A17 + ~{A22}.~{A15}.~{A14}.~{A13}) Consistent with access to: - 00-3F/80-BF:0000-1FFF or - 7E-7F:0000-FFFF"
- moved on the sheet: AABZ, AAHT, AAJX, AAKO, AALV, AAMX, ACPQ, BAAO, BABK, BABL, BBER, BBQF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

Commit message: Fixed VAWR which should have been an SR DFF (to fix issue #3 raised in github)
Connections:
- net at MBSK.1: now also MBUP.5; no longer MBUP.3
- net at VPA.4 (~{DRV}_HIGH): now also DCEG.4; no longer DCEG.3
- net at SYSCLK.3 (~{DRV}_HIGH): now also IBTS.4; no longer IBTS.3
- net at VDA.4 (~{DRV}_HIGH): now also FBSI.4; no longer FBSI.3
Other:
- moved on the sheet: BABL, CPUCK, DBPI, DCDY, HAKW, HALC, HAMT, HANA, HBCA, HBCT, HBEP, HBFW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
